File: doc/Power Regulator PCB/Power Regulator PCB.kicad_pcb (KiCad board)
At the start: 2 copper layers, 92 x 43 mm, 13 parts, among them U1 LM2596S-3.3, U2 LM2596S-5

Commit message: Updated Power Reg PCB Commit
Parts:
- moved C2 18.7 mm to (148.5, 81.2)
- moved C3 18.3 mm to (148.5, 99.2)
- moved L2 9.71 mm to (135.5, 101.5)
- moved L1 9.62 mm to (135.5, 79.0)
- moved E3 9.00 mm to (157.5, 105.5)
- moved E2 8.25 mm to (158.0, 76.0)
- moved D2 6.95 mm to (124.0, 91.0)
- moved D1 3.88 mm to (132.5, 91.0), turned to 180 degrees
- moved E1 1.12 mm to (89.0, 106.0)
Connections:
- C2 pad 2: <NO NET> -> GND
- C3 pad 2: <NO NET> -> GND
- D1 pad 2: <NO NET> -> GND
- D2 pad 2: <NO NET> -> GND
- E1 pad 1: (no net) -> GND
- U1 pad 5: <NO NET> -> GND
- U2 pad 5: <NO NET> -> GND
Routing:
- net GND: track 0.00 -> 130.3 mm, vias 0 -> 4
- net Net-(U1-FB): track 0.00 -> 70.3 mm
- net Net-(U2-FB): track 0.00 -> 69.7 mm, vias 0 -> 2
- net Net-(D1-K): track 0.00 -> 66.1 mm, vias 0 -> 4
- net Net-(D2-K): track 0.00 -> 41.4 mm, vias 0 -> 2
- net <NO NET>: track 23.8 -> 0.00 mm, vias 1 -> 0
- net Net-(U1-VIN): track 44.2 -> 43.2 mm, vias 0 -> 2
Other:
- board size 92 x 43 mm -> 82 x 43 mm
- board text added: "+12V"
- board text added: "+3V"
- board text added: "+5V"
- board text added: "BAJA SAE"
- board text added: "GND"
- board text added: "IN"
- board text added: "OUT"
