File: doc/Power Regulator PCB (LT8608)/Power Regulator PCB (LT8608).kicad_sch (KiCad schematic)
At the start: 29 parts

Commit message: Completed LT8606 Schematic
Parts:
- added C12: 10nF, Capacitor_SMD:C_0805_2012Metric, symbol Device:C
- added C13: 270uF, Capacitor_SMD:CP_Elec_6.3x9.9, symbol Device:C_Polarized
- added C14: 1uF, Capacitor_SMD:C_0805_2012Metric, symbol Device:C
- added C15: 10uF, Capacitor_SMD:C_1206_3216Metric, symbol Device:C_Polarized
- added C16: 47uF, Capacitor_SMD:C_1210_3225Metric, symbol Device:C_Polarized
- added D1: D, Diode_SMD:D_2114_3652Metric, symbol Device:D
- added E5: +5V (Pi Power), MountingHole:MountingHole_4.5mm_Pad_TopOnly, symbol Mechanical:MountingHole_Pad
- added L3: 3.3uH, Inductor_SMD:L_Coilcraft_XAL7030-332, symbol Device:L
- added U3: LM22678TJ-5, Package_TO_SOT_SMD:TO-263-7_TabPin8, symbol Regulator_Switching:LM22678TJ-5
- C10, C11, C2, C5, C6, C9: footprint (none) -> Capacitor_SMD:C_0805_2012Metric
- C3: footprint (none) -> Capacitor_SMD:C_0201_0603Metric
- C4, C8: footprint (none) -> Capacitor_SMD:C_1206_3216Metric
- C7: footprint (none) -> Mounting_Wuerth:Mounting_Wuerth_WA-SMSE-ExternalM3_H6mm_9771060360
- L1, L2: footprint (none) -> Inductor_SMD:L_Coilcraft_XAL7030-222
- R1, R2, R3, R4, R5, R6, R7, R8: footprint (none) -> Resistor_SMD:R_0805_2012Metric
Connections:
- net 0: now also C13.2, C14.2, C15.2, C16.2, D1.2 (A), U3.4 (GND), U3.8 (GND)
- net at C1.1, E1.1, U1.10 (EN/UV)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: now also C14.1, C15.1, C16.1, U3.2 (VIN)
- new net: C13.1, E5.1, L3.2, U3.6 (FB)
- new net: C12.1, D1.1 (K), L3.1, U3.3 (BOOT)
- new net: C12.2, U3.1 (SW)
Other:
- moved on the sheet: C1, E1, E4
