File: doc/Power Regulator PCB (LT8608)/Power Regulator PCB (LT8608).kicad_pcb (KiCad board)
At the start: 2 copper layers, 77.5 x 70.5 mm, 38 parts, among them U3 LM22678TJ-5

Commit message: Work on PCB layout
Parts:
- C7: footprint Mounting_Wuerth:Mounting_Wuerth_WA-SMSE-ExternalM3_H6mm_9771060360 -> Capacitor_SMD:C_0201_0603Metric
- moved L1 45.5 mm to (141.0, 59.6), turned to 90 degrees
- moved R8 45.4 mm to (152.2, 77.1)
- moved U1 42.0 mm to (147.6, 70.1)
- moved R1 38.6 mm to (135.0, 101.0)
- moved C3 38.3 mm to (157.2, 69.1)
- moved C8 38.2 mm to (135.0, 103.5)
- moved C1 37.7 mm to (152.5, 67.9), turned to 90 degrees
- moved TP1 33.4 mm to (147.8, 75.1)
- moved C10 33.3 mm to (152.8, 72.6), turned to -90 degrees
- moved R5 31.2 mm to (157.3, 74.1)
- moved C15 30.8 mm to (141.5, 104.0), turned to 180 degrees
- moved R2 30.3 mm to (140.5, 97.5)
- moved C6 29.6 mm to (153.9, 104.0)
- moved C4 26.5 mm to (149.0, 59.7), turned to -90 degrees
- moved C7 25.5 mm to (134.8, 98.5)
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Connections:
- U1 pad 11: (no net) -> 0
- U1 pad 9: 0 -> Net-(U1-EN/UV)
- U2 pad 11: (no net) -> 0
- U2 pad 9: 0 -> Net-(U1-EN/UV)
Routing:
- net Net-(U2-FB): track 0.00 -> 19.6 mm
- net 0: track 0.00 -> 17.6 mm, vias 0 -> 4
- net Net-(U2-PG): track 0.00 -> 15.0 mm, vias 0 -> 2
- net Net-(U2-SW): track 0.00 -> 13.5 mm
- net Net-(C7-Pad1): track 0.00 -> 10.7 mm
- net Net-(U1-EN/UV): track 0.00 -> 7.53 mm
- net Net-(U2-RT): track 0.00 -> 6.18 mm
- net Net-(U2-TR/SS): track 0.00 -> 5.51 mm
- net Net-(U2-INTV): track 0.00 -> 5.03 mm
- net Net-(U2-BST): track 0.00 -> 3.27 mm
- added copper zone on B.Cu, net 0
