File: doc/Schematics and PCBs/ESP32 IMU/ESP32 IMU.kicad_sch (KiCad schematic)
At the start: 3 parts

Commit message: Updated IMU PCB/Uploaded custom symbology
Parts:
- added J1: +5V, Connector_PinHeader_1.00mm:PinHeader_1x02_P1.00mm_Vertical, symbol Connector_Generic:Conn_01x02
Connections:
- net GND: now also UNIT_2.6 (GND), J1.2 (Pin_2)
- no-connect marks 1 -> 8
Other:
- moved on the sheet: UNIT_3

Commit message: Updated IMU PCB
Parts:
- added C1: .33u, Capacitor_THT:C_Axial_L3.8mm_D2.6mm_P7.50mm_Horizontal, symbol Device:C
- added C2: 22u, Capacitor_THT:CP_Axial_L11.0mm_D8.0mm_P15.00mm_Horizontal, symbol Device:C_Polarized
- added U1: BA50JC5T, Package_TO_SOT_THT:TO-220-3_Horizontal_TabDown, symbol Regulator_Linear:LF80_TO220
Connections:
- net GND: now also C1.2, C2.2, U1.2 (GND)
- net at J1.1 (Pin_1): now also C1.1, U1.1 (VI)
- net +5V renamed +5v
- net +5v: now also C2.1, U1.3 (VO)
Other:
- moved on the sheet: J1, UNIT_2, UNIT_3

Commit message: Final Touches on IMU
Other:
- moved on the sheet: C1, C2, J1, U1, UNIT_1, UNIT_2, UNIT_3
