File: doc/Schematics and PCBs/ESP32 IMU/ESP32 IMU.kicad_pcb (KiCad board)
At the start: 2 copper layers, 74 x 67.5 mm, 3 parts

Commit message: Updated IMU PCB/Uploaded custom symbology
Parts:
- added J1: +5V, Connector_PinHeader_1.00mm:PinHeader_1x02_P1.00mm_Vertical, F.Cu at (117.5, 61.0)
- added REF**: MountingHole_4.5mm, MountingHole:MountingHole_4.5mm, F.Cu at (108.0, 42.5)
- added REF**: MountingHole_4.5mm, MountingHole:MountingHole_4.5mm, F.Cu at (182.5, 112.0)
- added REF**: MountingHole_4.5mm, MountingHole:MountingHole_4.5mm, F.Cu at (182.5, 42.5)
- added REF**: MountingHole_4.5mm, MountingHole:MountingHole_4.5mm, F.Cu at (108.0, 112.0)
- moved UNIT_3 40.4 mm to (160.5, 65.0)
- moved UNIT_2 21.3 mm to (161.0, 95.0), turned to 90 degrees
- moved UNIT_1 4.73 mm to (129.2, 86.3)
Connections:
- UNIT_2 pad 6: unconnected-(UNIT_2-GND-Pad6) -> GND
Routing:
- net +5V: track 48.6 -> 6.63 mm
- net Net-(UNIT_1-IO5): track 0.00 -> 28.1 mm
- net Net-(UNIT_1-IO19): track 0.00 -> 23.5 mm, vias 0 -> 1
- net Net-(UNIT_1-IO18): track 0.00 -> 19.4 mm
Other:
- board size 74 x 67.5 mm -> 86.5 x 83.5 mm
- board text added: "BNO055 IMU"
- board text added: "CAN BUS"
- board text added: "ESP 32"
- board text added: "GND"
- board text added: "IMU SENSOR"
- board text added: "PN: IMU1"
- board text added: "SN:"
- board text added: "UNIVERSITY OF ARIZONA BAJA SAE"

Commit message: Updated IMU PCB
Parts:
- added C1: .33u, Capacitor_THT:C_Axial_L3.8mm_D2.6mm_P7.50mm_Horizontal, F.Cu at (114.2, 62.2)
- added C2: 22u, Capacitor_THT:CP_Axial_L11.0mm_D8.0mm_P15.00mm_Horizontal, F.Cu at (109.0, 88.5)
- added U1: BA50JC5T, Package_TO_SOT_THT:TO-220-3_Horizontal_TabDown, F.Cu at (111.5, 66.3)
- moved REF** 16.7 mm to (180.0, 59.0)
- moved REF** 16.5 mm to (107.5, 59.0)
- moved UNIT_1 4.96 mm to (130.5, 81.5)
- moved J1 4.19 mm to (118.8, 57.0)
- moved REF** 2.00 mm to (180.5, 112.0)
- moved UNIT_2 0.08 mm to (160.9, 95.0)
Connections:
- J1 pad 1: +5V -> Net-(J1-Pin_1)
- UNIT_1 pad J2-19: +5V -> +5v
- UNIT_2 pad 7: +5V -> +5v
- UNIT_3 pad 1: +5V -> +5v
Routing:
- net GND: track 0.00 -> 141.3 mm, vias 0 -> 2
- net +5v: track 0.00 -> 140.8 mm
- net Net-(UNIT_1-IO23): track 0.00 -> 26.7 mm
- net Net-(UNIT_1-IO22): track 0.00 -> 25.2 mm, vias 0 -> 1
- net Net-(UNIT_1-IO21): track 0.00 -> 25.0 mm, vias 0 -> 1
- net Net-(J1-Pin_1): track 0.00 -> 12.3 mm
- net +5V: track 6.63 -> 0.00 mm
- net Net-(UNIT_1-IO18): track 19.4 -> 16.1 mm
- net Net-(UNIT_1-IO5): track 28.1 -> 24.8 mm
- net Net-(UNIT_1-IO19): track 23.5 -> 20.2 mm
Other:
- board size 86.5 x 83.5 mm -> 84 x 65 mm
- board text added: "+-"
- board text added: "UNIVERSITY OF ARIZONA BAJA SAE Connor Larson Nov, 2024"
- board text removed: "GND"
- board text removed: "UNIVERSITY OF ARIZONA BAJA SAE"

Commit message: Updated IMU PCB and CANbus footprint
CAN bus footprint was not explicit in facing up or facing down. Updated to be explicit and edited PCB to match.
Parts:
- UNIT_2: value HiLetgo CAN Bus -> HiLetgo CAN Bus (Facing Up); footprint BAJA SAE:HiLetgo CAN Bus -> BAJA SAE:HiLetgo CAN Bus (Facing Up)
- moved UNIT_2 2.54 mm to (160.5, 97.5), turned to -90 degrees
Routing:
- net +5v: track 140.8 -> 124.3 mm
- net Net-(UNIT_1-IO18): track 16.1 -> 28.2 mm, vias 0 -> 3
- net GND: track 141.3 -> 130.2 mm, vias 2 -> 1
- net Net-(UNIT_1-IO23): track 26.7 -> 31.9 mm
- net Net-(UNIT_1-IO5): track 24.8 -> 20.0 mm
- net Net-(UNIT_1-IO19): track 20.2 -> 21.1 mm, vias 1 -> 0

Commit message: Updated IMU PCB
Updated silkscreen
Parts:
- CAN Bus (Facing UP): renamed from UNIT_2
Routing:
- net GND: track 130.2 -> 143.9 mm
- net +5v: track 124.3 -> 117.1 mm
Other:
- board text added: "+5V"
- board text added: "BNO055"
- board text added: "ESP-32"
- board text added: "GND"
Changed lines of the file:
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@@
 		(tags "C Axial series Axial Horizontal pin pitch 7.5mm  length 3.8mm diameter 2.6mm")
 		(property "Reference" "C1"
-			(at 3.5 2.5 0)
+			(at 4 2.25 -90)
+			(unlocked yes)
 			(layer "F.SilkS")
 			(effects
@@
 		)
 		(property "Value" ".33u"
-			(at 3.75 2.42 90)
+			(at 3.75 0.5 -90)
+			(unlocked yes)
 			(layer "F.Fab")
 			(effects
@@
 		(tags "Through hole pin header THT 1x02 1.00mm single row")
 		(property "Reference" "J1"
-			(at -3.5 0 0)
+			(at -3 0.5 270)
+			(unlocked yes)
 			(layer "F.SilkS")
 			(effects
@@
 		(layer "F.Cu")
 		(at 160.5 97.5 -90)
-		(property "Reference" "UNIT_2"
-			(at 0 -0.5 -90)
+		(property "Reference" "CAN Bus (Facing UP)"
+			(at 0 -1 270)
 			(unlocked yes)
 			(layer "F.SilkS")
@@
 		(property "Reference" "C2"
 			(at 7.5 -5.12 -90)
+			(unlocked yes)
 			(layer "F.SilkS")
 			(effects
@@
 		(tags "TO-220-3 Horizontal RM 2.54mm")
 		(property "Reference" "U1"
-			(at -1.96 2.27 0)
+			(at -3.71 -4.98 -90)
+			(unlocked yes)
 			(layer "F.SilkS")
 			(effects
@@
 		(layer "Edge.Cuts")
 	)
+	(gr_text "+5V"
+		(at 120.75 108 270)
+		(layer "F.SilkS")
+		(effects
+			(font
+				(size 1 1)
+				(thickness 0.1)
+			)
+		)
+	)
 	(gr_text "SN:"
 		(at 178 94.5 -90)
@@
 		)
 	)
+	(gr_text "ESP-32"
+		(at 131.5 85.75 270)
+		(layer "F.SilkS")
+		(effects
+			(font
+				(size 1 1)
+				(thickness 0.1)
+			)
+		)
+	)
+	(gr_text "BNO055"
+		(at 160.5 65 270)
+		(layer "F.SilkS")
+		(effects
+			(font
+				(size 1 1)
+				(thickness 0.1)
+			)
+		)
+	)
+	(gr_text "GND"
+		(at 139.75 62.5 270)
+		(layer "F.SilkS")
+		(effects
+			(font
+				(size 1 1)
+				(thickness 0.1)
+			)
+		)
+	)
 	(gr_text "BNO055 IMU"
-		(at 145 65.5 -90)
+		(at 174.75 66 -90)
 		(layer "F.SilkS")
 		(effects
@@
 	)
 	(gr_text "CAN BUS"
-		(at 145.5 109.5 -90)
+		(at 175 76.75 -90)
 		(layer "F.SilkS")
 		(effects
@@
 	)
 	(segment
+		(start 109 66.27)
+		(end 109 65.165)
+		(width 0.2)
+		(layer "B.Cu")
+		(net 8)
+	)
+	(segment
 		(start 132.93 89.07)
 		(end 145.93 89.07)
@@
 	)
 	(segment
+		(start 109 65.165)
+		(end 114.25 59.915)
+		(width 0.2)
+		(layer "B.Cu")
+		(net 8)
+	)
+	(segment
 		(start 132.5 89.5)
 		(end 132.93 89.07)
@@
 	)
 	(segment
+		(start 114.25 59.915)
+		(end 114.25 54.75)
+		(width 0.2)
+		(layer "B.Cu")
+		(net 8)
+	)
+	(segment
 		(start 151.5 86.5)
 		(end 149 86.5)
@@
 	)
 	(segment
-		(start 156.26 76)
-		(end 154.15 73.89)
-		(width 0.2)
-		(layer "F.Cu")
-		(net 45)
-	)
-	(segment
 		(start 140.75 114)
 		(end 124.45 114)
@@
 	)
 	(segment
-		(start 166.54 76)
-		(end 156.26 76)
-		(width 0.2)
-		(layer "F.Cu")
-		(net 45)
-	)
-	(segment
 		(start 152.85 98.767351)
 		(end 144 107.617351)
@@
 	)
 	(segment
+		(start 154.15 78.16)
+		(end 152.85 79.46)
+		(width 0.2)
+		(layer "B.Cu")
+		(net 45)
+	)
+	(segment
 		(start 109 88.5)
 		(end 109 98.55)
 		(width 0.2)
 		(layer "B.Cu")
+		(net 45)
+	)
+	(segment
+		(start 154.15 73.89)
+		(end 154.15 78.16)
+		(width 0.2)
+		(layer "B.Cu")

Commit message: Final Touches on IMU
Parts:
- added G***: LOGO, BAJA SAE:Baja Logo, F.Cu at (181.2, 79.5)
Other:
- board text added: "UNIVERSITY OF ARIZONA Connor Larson Nov, 2024"
- board text removed: "BNO055 IMU"
- board text removed: "CAN BUS"
- board text removed: "UNIVERSITY OF ARIZONA BAJA SAE Connor Larson Nov, 2024"

Commit message: Updated ESP-32 IMU PCB
Added J2 as a bypass for the power regulator
Parts:
- added J2: +5V, Connector_PinHeader_1.00mm:PinHeader_1x02_P1.00mm_Vertical, F.Cu at (114.8, 115.2)
Routing:
- net GND: track 143.9 -> 157.0 mm
- net +5v: track 117.1 -> 126.1 mm
