File: hardware/KICAD Projects/BAJE SAE/Sensor Projects/ESP32 IMU/ESP32 IMU.kicad_pcb (KiCad board)
At the start: 2 copper layers, 84 x 65 mm, 13 parts, among them J1 +5V, J2 +5V, U1 BA50JC5T

Commit message: Updated IMU PCB to Revision 2
sectioned off schematic
changed schematic from wires to flags
edited PCB to be much smaller
updated J1 to be correct size
increased ESP 32 pad size
updated CAN Bus to hang off board
flipped power reg to other side
updated on board graphics
added to do list on schem
Parts:
- removed J2: +5V, Connector_PinHeader_1.00mm:PinHeader_1x02_P1.00mm_Vertical
- C1, C2, G***, U1: moved to B.Cu
- moved REF** 72.5 mm to (180.0, 60.0)
- moved REF** 70.0 mm to (110.0, 60.0)
- moved J1 69.7 mm to (177.5, 94.5), turned to -90 degrees
- moved U1 65.0 mm to (176.5, 68.2), turned to -90 degrees
- moved C2 47.0 mm to (155.5, 82.0), turned to 0 degrees
- moved UNIT_3 39.0 mm to (159.5, 104.0), turned to 180 degrees
- moved C1 38.3 mm to (150.5, 74.8)
- moved G*** 30.1 mm to (160.5, 101.2), turned to 180 degrees
- moved CAN Bus (Facing UP) 26.8 mm to (159.5, 70.8), turned to 90 degrees
- moved REF** 3.61 mm to (110.0, 115.0)
- moved REF** 3.04 mm to (180.0, 115.0)
- moved UNIT_1 1.92 mm to (130.0, 83.3)
Connections:
- net Net-(UNIT_1-IO21) renamed SDA
- net Net-(UNIT_1-IO22) renamed SCL
- UNIT_1 pad J3-10: Net-(UNIT_1-IO5) -> CS
- UNIT_1 pad J3-2: Net-(UNIT_1-IO23) -> SI
- UNIT_1 pad J3-8: Net-(UNIT_1-IO19) -> SO
- UNIT_1 pad J3-9: Net-(UNIT_1-IO18) -> SCK
Routing:
- net GND: track 157.0 -> 0.00 mm, vias 1 -> 0
- net +5v: track 126.1 -> 0.00 mm
- net Net-(UNIT_1-IO23): track 31.9 -> 0.00 mm
- net Net-(UNIT_1-IO18): track 28.2 -> 0.00 mm, vias 3 -> 0
- net SCL: track 25.2 -> 0.00 mm, vias 1 -> 0
- net SDA: track 25.0 -> 0.00 mm, vias 1 -> 0
- net Net-(UNIT_1-IO19): track 21.1 -> 0.00 mm
- net Net-(UNIT_1-IO5): track 20.0 -> 0.00 mm
- net Net-(J1-Pin_1): track 12.3 -> 0.00 mm
Other:
- board size 84 x 65 mm -> 82 x 67 mm
- board text added: "+"
- board text added: "IMU"
- board text removed: "+-"
- board text removed: "+5V"
- board text removed: "BNO055"
- board text removed: "ESP 32"
- board text removed: "ESP-32"
- board text removed: "GND"
- board text removed: "IMU SENSOR"
- board text removed: "PN: IMU1"
- board text removed: "SN:"

Commit message: fixed issue that causes the whole pcb not to work
Parts:
- removed C1: .33u, Capacitor_THT:C_Axial_L3.8mm_D2.6mm_P7.50mm_Horizontal
- removed C2: 22u, Capacitor_THT:CP_Axial_L11.0mm_D8.0mm_P15.00mm_Horizontal
- removed REF** (x4): MountingHole_4.5mm, MountingHole:MountingHole_4.5mm
- removed U1: BA50JC5T, Package_TO_SOT_THT:TO-220-3_Horizontal_TabDown
- moved J1 43.4 mm to (141.0, 118.0), turned to 180 degrees
- moved G*** 4.07 mm to (156.5, 102.0)
- moved CAN Bus (Facing UP) 2.50 mm to (157.5, 72.2)
- moved UNIT_3 2.00 mm to (157.5, 104.0)
- moved UNIT_1 1.72 mm to (129.0, 84.8)
Other:
- board size 82 x 67 mm -> 63.9 x 62.2 mm
