File: hardware/KICAD Projects/BAJE SAE/Sensor Projects/ESP32 IMU/ESP32 IMU.kicad_sch (KiCad schematic)
At the start: 7 parts, among them J1 +5V, U1 BA50JC5T

Commit message: Updated IMU PCB to Revision 2
sectioned off schematic
changed schematic from wires to flags
edited PCB to be much smaller
updated J1 to be correct size
increased ESP 32 pad size
updated CAN Bus to hang off board
flipped power reg to other side
updated on board graphics
added to do list on schem
Connections:
- net CS: now reaches UNIT_1.J3-10 (IO5), UNIT_2.5 (CS)
- net SI: now reaches UNIT_1.J3-2 (IO23), UNIT_2.3 (SI)
- net SCL: now reaches UNIT_1.J3-3 (IO22), UNIT_3.5 (SCL)
- net SDA: now reaches UNIT_1.J3-6 (IO21), UNIT_3.4 (SDA)
- net SO: now reaches UNIT_1.J3-8 (IO19), UNIT_2.4 (SO)
- net SCK: now reaches UNIT_1.J3-9 (IO18), UNIT_2.2 (SCK)
- no-connect marks 8 -> 34
Other:
- note added: "CAN Bus"
- note added: "ESP32"
- note added: "IMU"
- note added: "Power Regulation"
- company: (none) -> University of Arizona Baja SAE
- title: (none) -> ESP 32 IMU
- moved on the sheet: C1, C2, J1, U1, UNIT_1, UNIT_2, UNIT_3

Commit message: Updated IMU Rev 2 Schem
Other:
- note added: "TO DO - Measure CAN bus so it hangs off board properly - Make sure IO is all on same side of board - Figure out why power regulation no worky - Add revision to silkscreen"
Changed lines of the file:
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@@
+		)
+	)
+	(text "TO DO\n\n- Measure CAN bus so it hangs off board properly\n- Make sure IO is all on same side of board\n- Figure out why power regulation no worky\n- Add revision to silkscreen"
+		(exclude_from_sim no)
+		(at 60.96 144.78 0)
+		(effects
+			(font
+				(size 1.27 1.27)
+			)
 		)
 	)

Commit message: fixed issue that causes the whole pcb not to work
Parts:
- removed C1: .33u, Capacitor_THT:C_Axial_L3.8mm_D2.6mm_P7.50mm_Horizontal, symbol Device:C
- removed C2: 22u, Capacitor_THT:CP_Axial_L11.0mm_D8.0mm_P15.00mm_Horizontal, symbol Device:C_Polarized
- removed U1: BA50JC5T, Package_TO_SOT_THT:TO-220-3_Horizontal_TabDown, symbol Regulator_Linear:LF80_TO220
Connections:
- net +5v: now also J1.1 (Pin_1)
- net GND: now also UNIT_3.3 (GND)
- no-connect marks 34 -> 33
Other:
- note added: "ESP-32 Socketed with ESS-119-T-03"
- note added: "Power"
- note added: "Socket"
- note removed: "Power Regulation"
- note removed: "TO DO - Measure CAN bus so it hangs off board properly - Make sure IO is all on same side of board - Figure out why power regulation no worky - Add revision to silkscreen"

Commit message: updates to esp32 IMU
Other:
- moved on the sheet: UNIT_1
