File: hardware/KICAD Projects/BAJE SAE/Sensor Projects/ESP32 IMU (Micro)/ESP32 IMU.kicad_pcb (KiCad board)
At the start: 2 copper layers, 57.1 x 72 mm, 12 parts, among them J1 +5V, U1 BA50JC5T

Commit message: Finished rough sketch of the ESP32 IMU Micro
Parts:
- removed C1: .33u, Capacitor_THT:C_Axial_L3.8mm_D2.6mm_P7.50mm_Horizontal
- removed C2: 22u, Capacitor_THT:CP_Axial_L11.0mm_D8.0mm_P15.00mm_Horizontal
- removed REF** (x4): MountingHole_4.5mm, MountingHole:MountingHole_4.5mm
- removed U1: BA50JC5T, Package_TO_SOT_THT:TO-220-3_Horizontal_TabDown
- CAN Bus (Facing UP): moved to B.Cu
- UNIT_3: moved to B.Cu
- moved G*** 41.6 mm to (132.0, 118.0), turned to 0 degrees
- moved CAN Bus (Facing UP) 10.8 mm to (129.8, 80.0), turned to 90 degrees
- moved J1 9.60 mm to (136.4, 65.8)
- moved UNIT_3 9.11 mm to (129.7, 113.2), turned to 0 degrees
- moved UNIT_1 8.12 mm to (129.4, 91.4), turned to 180 degrees
Connections:
- J1 pad 1: Net-(J1-Pin_1) -> +5v
Routing:
- net GND: track 0.00 -> 70.1 mm
- net +5v: track 0.00 -> 55.6 mm
- net SCL: track 0.00 -> 16.7 mm
- net SDA: track 0.00 -> 16.4 mm
Other:
- board size 57.1 x 72 mm -> 30.5 x 66 mm
- board text added: "UNIVERSITY OF ARIZONA Connor Larson Jan, 2025"
- board text removed: "UNIVERSITY OF ARIZONA Connor Larson Nov, 2024"

Commit message: fixed issue that causes the whole pcb not to work
Parts:
- moved J1 2.22 mm to (135.0, 67.5)
- moved UNIT_3 0.99 mm to (129.5, 114.1)
- moved UNIT_1 0.13 mm to (129.3, 91.4)
Routing:
- net +5v: track 55.6 -> 56.7 mm
- net GND: track 70.1 -> 69.2 mm
Other:
- board size 30.5 x 66 mm -> 30.5 x 70.5 mm

Commit message: updates to esp32 IMU
Parts:
- J1: value +5V -> Conn_01x02; footprint Connector_PinHeader_1.00mm:PinHeader_1x02_P1.00mm_Vertical -> Connector_Wire:SolderWire-0.75sqmm_1x02_P4.8mm_D1.25mm_OD2.3mm_Relief2x
- moved J1 25.2 mm to (131.4, 92.4), turned to 180 degrees
Connections:
- UNIT_3 pad 3: unconnected-(UNIT_3-GND-Pad3) -> GND
Routing:
- net +5v: track 56.7 -> 16.9 mm
- net GND: track 69.2 -> 57.7 mm
Other:
- outline, holes or cut-outs redrawn

Commit message: Updates to IMU and Temp PCB
Parts:
- added J2: CAN to outer connector, Connector_Wire:SolderWire-0.1sqmm_1x04_P3.6mm_D0.4mm_OD1mm_Relief, F.Cu at (134.8, 79.3)
- added J3: Conn_01x02, Connector_PinHeader_2.54mm:PinHeader_1x02_P2.54mm_Vertical, B.Cu at (131.7, 66.9)
- added J4: Conn_01x02, Connector_PinHeader_2.54mm:PinHeader_1x02_P2.54mm_Vertical, B.Cu at (127.1, 66.9)
- J1: footprint Connector_Wire:SolderWire-0.75sqmm_1x02_P4.8mm_D1.25mm_OD2.3mm_Relief2x -> Connector_Wire:SolderWire-0.75sqmm_1x02_P4.8mm_D1.25mm_OD2.3mm_Relief
- moved UNIT_1 7.16 mm to (129.3, 98.6)
- moved J1 4.74 mm to (131.5, 97.2)
- moved CAN Bus (Facing UP) 2.61 mm to (129.8, 82.6)
- moved UNIT_3 1.68 mm to (129.5, 115.8)
Routing:
- net GND: track 57.7 -> 0.00 mm
- net +5v: track 16.9 -> 0.00 mm
- net SCL: track 16.7 -> 0.00 mm
- net SDA: track 16.4 -> 0.00 mm
Other:
- board size 30.5 x 70.5 mm -> 30.5 x 73.3 mm
- board text added: "-"

Commit message: finished imu, started others
Parts:
- removed J3, J4: Conn_01x02, Connector_PinHeader_2.54mm:PinHeader_1x02_P2.54mm_Vertical
- J1: footprint Connector_Wire:SolderWire-0.75sqmm_1x02_P4.8mm_D1.25mm_OD2.3mm_Relief -> Connector_Wire:SolderWire-0.75sqmm_1x02_P4.8mm_D1.25mm_OD2.3mm
- J2: footprint Connector_Wire:SolderWire-0.1sqmm_1x04_P3.6mm_D0.4mm_OD1mm_Relief -> Connector_Wire:SolderWire-0.1sqmm_1x04_P3.6mm_D0.4mm_OD1mm
- moved J1 20.7 mm to (131.8, 76.5)
- moved J2 16.8 mm to (134.8, 62.5)
- moved CAN Bus (Facing UP) 8.09 mm to (127.1, 90.2)
- moved G*** 4.96 mm to (129.0, 114.0)
- moved UNIT_3 0.55 mm to (129.5, 115.3)
Connections:
- CAN Bus (Facing UP) pad 2: Net-(UNIT_1-IO18) -> SCK
- CAN Bus (Facing UP) pad 3: Net-(UNIT_1-IO23) -> SI
- CAN Bus (Facing UP) pad 4: Net-(UNIT_1-IO19) -> SO
- CAN Bus (Facing UP) pad 5: Net-(UNIT_1-IO5) -> CS
- J2 pad 1: /Green 1 -> Low
- J2 pad 2: /White 1 -> High
- J2 pad 3: /Green 2 -> Low
- J2 pad 4: /White 2 -> High
Routing:
- net GND: track 0.00 -> 69.8 mm
- net +5v: track 0.00 -> 53.6 mm
- net SI: track 0.00 -> 19.6 mm, vias 0 -> 1
- net SCL: track 0.00 -> 19.2 mm
- net CS: track 0.00 -> 17.4 mm
- net SDA: track 0.00 -> 15.8 mm
- net Low: track 0.00 -> 15.3 mm
- net High: track 0.00 -> 14.2 mm
- net SO: track 0.00 -> 13.0 mm
- net SCK: track 0.00 -> 7.72 mm
Other:
- board text added: "BNO on this side"
- board text added: "CAN BUS on this side"
- board text added: "ESP-32 on this side"
- board text added: "H"
- board text added: "L"
