File: hardware/KICAD Projects/BAJE SAE/Sensor Projects/ESP32 IMU (Micro)/ESP32 IMU.kicad_pcb (KiCad board)
At the start: 2 copper layers, 30.5 x 73.3 mm, 6 parts, among them J1 Conn_01x02, J2 CAN to outer connector

Commit message: finished pcbs yayyyy
Routing:
- net GND: track 69.8 -> 96.9 mm
- net SCK: track 7.72 -> 17.9 mm
- net SI: track 19.6 -> 24.7 mm
- net +5v: track 53.6 -> 49.3 mm, vias 0 -> 2
- net CS: track 17.4 -> 16.9 mm, vias 0 -> 2
Other:
- board text added: "Designed by Connor & Matthew Larson in Tucson, AZ"
- board text removed: "UNIVERSITY OF ARIZONA Connor Larson Jan, 2025"
Changed lines of the file:
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@@
 			(outputformat 1)
 			(mirror no)
-			(drillshape 1)
+			(drillshape 0)
 			(scaleselection 1)
-			(outputdirectory "")
+			(outputdirectory "Gerber Files/")
 		)
 	)
@@
 			(net 7 "unconnected-(UNIT_1-TXD0-PadJ3-4)")
 			(pinfunction "TXD0")
-			(pintype "output")
+			(pintype "output+no_connect")
 			(solder_mask_margin 0.102)
 		)
@@
 			(net 31 "unconnected-(UNIT_1-RXD0-PadJ3-5)")
 			(pinfunction "RXD0")
-			(pintype "input")
+			(pintype "input+no_connect")
 			(solder_mask_margin 0.102)
 		)
@@
 		)
 		(pad "1" thru_hole circle
-			(at -9.95 -5.22 270)
+			(at -9.95 10.02 270)
 			(size 1.8 1.8)
 			(drill 0.9)
@@
 		)
 		(pad "2" thru_hole circle
-			(at -9.95 -2.68 270)
+			(at -9.95 7.48 270)
 			(size 1.8 1.8)
 			(drill 0.9)
@@
 		)
 		(pad "3" thru_hole circle
-			(at -9.95 -0.14 270)
+			(at -9.95 4.94 270)
 			(size 1.8 1.8)
 			(drill 0.9)
@@
 		)
 		(pad "5" thru_hole circle
-			(at -9.95 4.94 270)
+			(at -9.95 -0.14 270)
 			(size 1.8 1.8)
 			(drill 0.9)
@@
 		)
 		(pad "6" thru_hole circle
-			(at -9.95 7.48 270)
+			(at -9.95 -2.68 270)
 			(size 1.8 1.8)
 			(drill 0.9)
@@
 		)
 		(pad "7" thru_hole circle
-			(at -9.95 10.02 270)
+			(at -9.95 -5.22 270)
 			(size 1.8 1.8)
 			(drill 0.9)
@@
 	)
 	(gr_text "CAN BUS on this side"
-		(at 137.5 87 0)
+		(at 121.6 92.6 -90)
 		(layer "B.SilkS")
 		(effects
@@
 		)
 	)
-	(gr_text "-"
-		(at 125.674 80.6484 0)
-		(layer "F.SilkS")
+	(gr_text "Designed by Connor & Matthew Larson \nin Tucson, AZ"
+		(at 135.8 96.5 270)
+		(layer "B.SilkS")
 		(effects
 			(font
-				(size 2 2)
+				(size 1 1)
 				(thickness 0.1)
 			)
-			(justify left bottom)
+			(justify left bottom mirror)
 		)
 	)
-	(gr_text "L"
-		(at 127 60.75 0)
+	(gr_text "-"
+		(at 125.674 80.6484 0)
 		(layer "F.SilkS")
 		(effects
 			(font
-				(size 1 1)
+				(size 2 2)
 				(thickness 0.1)
 			)
@@
 		)
 	)
-	(gr_text "UNIVERSITY OF ARIZONA\nConnor Larson Jan, 2025"
-		(at 120.25 73.25 0)
+	(gr_text "L"
+		(at 127 60.75 0)
 		(layer "F.SilkS")
 		(effects
@@
 	)
 	(gr_text "ESP-32 on this side"
-		(at 121.75 93.25 0)
+		(at 121.2 79.9 -90)
 		(layer "F.SilkS")
 		(effects
@@
 	)
 	(segment
-		(start 134.966 84.516)
-		(end 126.95 76.5)
+		(start 115.9 101.6)
+		(end 115.9 70.7)
 		(width 0.4)
 		(layer "B.Cu")
@@
 	)
 	(segment
-		(start 131.77 103)
-		(end 130.25 103)
+		(start 134.966 84.516)
+		(end 126.95 76.5)
 		(width 0.4)
 		(layer "B.Cu")
@@
 	)
 	(segment
-		(start 134.58 91.08)
-		(end 134.58 100.19)
+		(start 115.9 70.7)
+		(end 116.8 69.8)
 		(width 0.4)
 		(layer "B.Cu")
@@
 	)
 	(segment
-		(start 134.5 84.982)
-		(end 134.5 91)
+		(start 116.8 69.8)
+		(end 120.25 69.8)
 		(width 0.4)
 		(layer "B.Cu")
@@
 	)
 	(segment
-		(start 134.58 100.19)
-		(end 131.77 103)
+		(start 116.576 102.276)
+		(end 115.9 101.6)
 		(width 0.4)
 		(layer "B.Cu")
@@
 	)
 	(segment
-		(start 130.25 103)
-		(end 128.23 105.02)
+		(start 120.25 69.8)
+		(end 126.95 76.5)
 		(width 0.4)
 		(layer "B.Cu")
@@
 	)
 	(segment
+		(start 117.9414 102.276)
+		(end 116.576 102.276)
+		(width 0.4)
+		(layer "B.Cu")
+		(net 6)
+	)
+	(segment
 		(start 140.9814 84.516)
 		(end 134.966 84.516)
@@
 	)
 	(segment
-		(start 134.5 91)
-		(end 134.58 91.08)
+		(start 126.46 102.23)
+		(end 124.42 100.19)
 		(width 0.4)
 		(layer "B.Cu")
@@
 	)
 	(segment
-		(start 134.966 84.516)
-		(end 134.5 84.982)
+		(start 126.46 103.25)
+		(end 126.46 102.23)
 		(width 0.4)
 		(layer "B.Cu")
@@
 	)
 	(segment
-		(start 120.75 104.5)
-		(end 122.65 104.5)
+		(start 125.8 104.4)
+		(end 127.83 104.4)
 		(width 0.2)
 		(layer "F.Cu")
@@
 	)
 	(segment
-		(start 122.65 104.5)
-		(end 126.96 100.19)
+		(start 127.83 104.4)
+		(end 132.04 100.19)
 		(width 0.2)
 		(layer "F.Cu")
@@
 	)
 	(via
-		(at 120.75 104.5)
+		(at 125.8 104.4)
 		(size 0.6)
 		(drill 0.3)
@@
 	)
 	(segment
+		(start 120.75 104.5)
+		(end 120.85 104.4)
+		(width 0.2)
+		(layer "B.Cu")
+		(net 16)
+	)
+	(segment
 		(start 117.9414 114.976)
 		(end 120.75 112.1674)
@@
 	)
 	(segment
-		(start 132.04 100.19)
-		(end 132.04 98.54)
+		(start 120.85 104.4)
+		(end 125.8 104.4)
 		(width 0.2)
-		(layer "F.Cu")
-		(net 26)
+		(layer "B.Cu")
+		(net 16)
 	)
 	(segment
@@
 	)
 	(segment
-		(start 132.04 98.54)
+		(start 128.9 98.25)
+		(end 128.9 98.1)
+		(width 0.2)
+		(layer "F.Cu")
+		(net 26)
+	)
+	(segment
+		(start 126.96 100.19)
+		(end 128.9 98.25)
+		(width 0.2)
+		(layer "F.Cu")
+		(net 26)
+	)
+	(segment
+		(start 128.8 95.3)
 		(end 128.156 94.656)
 		(width 0.2)
@@
 		(net 26)
 	)
+	(via
+		(at 128.9 98.1)
+		(size 0.6)
+		(drill 0.3)
+		(layers "F.Cu" "B.Cu")
+		(net 26)
+	)
+	(via
+		(at 128.8 95.3)
+		(size 0.6)
+		(drill 0.3)
+		(layers "F.Cu" "B.Cu")
+		(net 26)
+	)
 	(segment
-		(start 127.29 102.25)
-		(end 123.15 106.39)
+		(start 128.9 95.4)
+		(end 128.8 95.3)
+		(width 0.2)
+		(layer "B.Cu")
+		(net 26)
+	)
+	(segment
+		(start 128.9 98.1)
+		(end 128.9 95.4)
+		(width 0.2)
+		(layer "B.Cu")
+		(net 26)
+	)
+	(segment
+		(start 131.75 94.82)
+		(end 130.17 96.4)
 		(width 0.2)
 		(layer "F.Cu")
@@
 	)
 	(segment
+		(start 130.17 96.4)
+		(end 123.9 96.4)
+		(width 0.2)
+		(layer "F.Cu")
+		(net 33)
+	)
+	(segment
+		(start 121.88 100.19)
+		(end 121.88 98.42)
+		(width 0.2)
+		(layer "F.Cu")
+		(net 33)
+	)
+	(segment
+		(start 121.88 100.19)
+		(end 121.88 105.12)
+		(width 0.2)
+		(layer "F.Cu")
+		(net 33)
+	)
+	(segment
 		(start 133.25 76.5)
 		(end 137.934 71.816)
@@
 	)
 	(segment
-		(start 131.75 94.82)
-		(end 137.12 100.19)
+		(start 121.88 105.12)
+		(end 123.15 106.39)
 		(width 0.2)
 		(layer "F.Cu")
@@
 	)
 	(segment
-		(start 137.934 71.816)
-		(end 140.9814 71.816)
+		(start 121.88 98.42)
+		(end 122.5 97.8)
 		(width 0.2)
 		(layer "F.Cu")
@@
 	)
 	(segment
-		(start 135.06 102.25)
-		(end 127.29 102.25)
+		(start 137.934 71.816)
+		(end 140.9814 71.816)
 		(width 0.2)
 		(layer "F.Cu")
 		(net 33)
 	)
+	(via
+		(at 122.5 97.8)
+		(size 0.6)
+		(drill 0.3)
+		(layers "F.Cu" "B.Cu")
+		(net 33)
+	)
+	(via
+		(at 123.9 96.4)
+		(size 0.6)
+		(drill 0.3)
+		(layers "F.Cu" "B.Cu")
+		(net 33)
+	)
 	(segment
-		(start 137.12 100.19)
-		(end 135.06 102.25)
+		(start 122.5 97.8)
+		(end 123.9 96.4)
 		(width 0.2)
-		(layer "F.Cu")
+		(layer "B.Cu")
 		(net 33)
 	)
 	(segment
-		(start 124.42 100.19)
-		(end 121.426 97.196)
+		(start 131.586 97.196)
+		(end 117.9414 97.196)
 		(width 0.2)
 		(layer "F.Cu")
@@
 	)
 	(segment
-		(start 121.426 97.196)
-		(end 117.9414 97.196)
+		(start 134.58 100.19)
+		(end 131.586 97.196)
 		(width 0.2)
 		(layer "F.Cu")
@@
 	)
 	(segment
-		(start 120.75 98.25)
-		(end 119.264 99.736)
+		(start 129.5 100.19)
+		(end 128.01 98.7)
 		(width 0.2)
 		(layer "B.Cu")
@@
 	)
 	(segment
-		(start 129.5 100.19)
-		(end 127.56 98.25)
+		(start 120.3 98.7)
+		(end 119.264 99.736)
 		(width 0.2)
 		(layer "B.Cu")
@@
 	)
 	(segment
-		(start 127.56 98.25)
-		(end 120.75 98.25)
+		(start 128.01 98.7)
+		(end 120.3 98.7)
 		(width 0.2)
 		(layer "B.Cu")
