File: hardware/KICAD Projects/BAJE SAE/Sensor Projects/ESP32 IMU (Micro)/ESP32 IMU.kicad_sch (KiCad schematic)
At the start: 7 parts, among them J1 +5V, U1 BA50JC5T

Commit message: Finished rough sketch of the ESP32 IMU Micro
Parts:
- removed C1: .33u, Capacitor_THT:C_Axial_L3.8mm_D2.6mm_P7.50mm_Horizontal, symbol Device:C
- removed C2: 22u, Capacitor_THT:CP_Axial_L11.0mm_D8.0mm_P15.00mm_Horizontal, symbol Device:C_Polarized
- removed U1: BA50JC5T, Package_TO_SOT_THT:TO-220-3_Horizontal_TabDown, symbol Regulator_Linear:LF80_TO220
Connections:
- net +5v: now also J1.1 (Pin_1)

Commit message: fixed issue that causes the whole pcb not to work
Connections:
- net GND: now also UNIT_3.3 (GND)
- no-connect marks 34 -> 33
Other:
- note added: "ESP-32 Socketed with ESS-119-T-03"
- note added: "Power"
- note added: "Socket"
- note removed: "Power Regulation"
- note removed: "TO DO - Measure CAN bus so it hangs off board properly - Make sure IO is all on same side of board - Figure out why power regulation no worky - Add revision to silkscreen"
- moved on the sheet: J1
Changed lines of the file:
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@@
-	)
-	(no_connect
-		(at 158.75 123.19)
 	)
 	(no_connect
@@
 	(wire
 		(pts
-			(xy 226.06 54.61) (xy 236.22 54.61)
+			(xy 194.31 54.61) (xy 196.85 54.61)
 		)
 		(stroke
@@
 	(wire
 		(pts
-			(xy 99.06 106.68) (xy 99.06 109.22)
+			(xy 193.04 52.07) (xy 196.85 52.07)
 		)
 		(stroke
@@
 	(wire
 		(pts
-			(xy 236.22 57.15) (xy 236.22 59.69)
+			(xy 99.06 106.68) (xy 99.06 109.22)
 		)
 		(stroke
@@
 		(pts
 			(xy 142.24 76.2) (xy 142.24 77.47)
+		)
+		(stroke
+			(width 0)
+			(type default)
+		)
+	)
+	(wire
+		(pts
+			(xy 158.75 123.19) (xy 161.29 123.19)
 		)
 		(stroke
@@
 	)
 	(rectangle
+		(start 179.07 67.31)
+		(end 211.76 82.6616)
+		(stroke
+			(width 0)
+			(type dot)
+		)
+		(fill
+			(type none)
+		)
+	)
+	(rectangle
 		(start 179.4 45.6084)
-		(end 253.242 80.7032)
+		(end 212.09 60.96)
 		(stroke
 			(width 0)
@@
 		)
 	)
-	(text "TO DO\n\n- Measure CAN bus so it hangs off board properly\n- Make sure IO is all on same side of board\n- Figure out why power regulation no worky\n- Add revision to silkscreen"
-		(exclude_from_sim no)
-		(at 60.96 144.78 0)
-		(effects
-			(font
-				(size 1.27 1.27)
-			)
-		)
-	)
 	(text "IMU"
 		(exclude_from_sim no)
@@
 		)
 	)
-	(text "Power Regulation"
+	(text "Socket"
 		(exclude_from_sim no)
-		(at 187.96 44.45 0)
+		(at 181.864 66.04 0)
+		(effects
+			(font
+				(size 1.27 1.27)
+			)
+		)
+	)
+	(text "Power"
+		(exclude_from_sim no)
+		(at 182.118 44.196 0)
 		(effects
 			(font
@@
 		)
 	)
+	(text "ESP-32 Socketed with \nESS-119-T-03"
+		(exclude_from_sim no)
+		(at 195.58 75.184 0)
+		(effects
+			(font
+				(size 1.27 1.27)
+			)
+		)
+	)
 	(text "CAN Bus"
 		(exclude_from_sim no)
@@
 	(global_label "+5v"
 		(shape output)
-		(at 226.06 54.61 180)
+		(at 193.04 52.07 180)
 		(fields_autoplaced yes)
 		(effects
@@
 		)
 		(property "Intersheetrefs" "${INTERSHEET_REFS}"
-			(at 219.3253 54.61 0)
+			(at 186.3053 52.07 0)
 			(effects
 				(font
@@
 		)
 	)
+	(global_label "GND"
+		(shape input)
+		(at 194.31 54.61 180)
+		(fields_autoplaced yes)
+		(effects
+			(font
+				(size 1.27 1.27)
+			)
+			(justify right)
+		)
+		(property "Intersheetrefs" "${INTERSHEET_REFS}"
+			(at 187.4543 54.61 0)
+			(effects
+				(font
+					(size 1.27 1.27)
+				)
+				(justify right)
+				(hide yes)
+			)
+		)
+	)
 	(global_label "SCL"
 		(shape input)
@@
 				)
 				(justify right)
+				(hide yes)
+			)
+		)
+	)
+	(global_label "GND"
+		(shape input)
+		(at 161.29 123.19 0)
+		(fields_autoplaced yes)
+		(effects
+			(font
+				(size 1.27 1.27)
+			)
+			(justify left)
+		)
+		(property "Intersheetrefs" "${INTERSHEET_REFS}"
+			(at 168.1457 123.19 0)
+			(effects
+				(font
+					(size 1.27 1.27)
+				)
+				(justify left)
 				(hide yes)
 			)
@@
 	(symbol
 		(lib_id "Connector_Generic:Conn_01x02")
-		(at 241.3 54.61 0)
+		(at 201.93 52.07 0)
 		(unit 1)
 		(exclude_from_sim no)
@@
 		(fields_autoplaced yes)
 		(property "Reference" "J1"
-			(at 243.84 54.6099 0)
+			(at 204.47 52.0699 0)
 			(effects
 				(font
@@
 		)
 		(property "Value" "+5V"
-			(at 243.84 57.1499 0)
+			(at 204.47 54.6099 0)
 			(effects
 				(font
@@
 		)
 		(property "Footprint" "Connector_PinHeader_1.00mm:PinHeader_1x02_P1.00mm_Vertical"
-			(at 241.3 54.61 0)
+			(at 201.93 52.07 0)
 			(effects
 				(font
@@
 		)
 		(property "Datasheet" "~"
-			(at 241.3 54.61 0)
+			(at 201.93 52.07 0)
 			(effects
 				(font
@@
 		)
 		(property "Description" "Generic connector, single row, 01x02, script generated (kicad-library-utils/schlib/autogen/connector/)"
-			(at 241.3 54.61 0)
+			(at 201.93 52.07 0)
 			(effects
 				(font
@@
 					(unit 1)
 				)
-			)
-		)
-	)
-	(symbol
-		(lib_id "power:GND")
-		(at 236.22 59.69 0)
-		(unit 1)
-		(exclude_from_sim no)
-		(in_bom yes)
-		(on_board yes)
-		(dnp no)
-		(fields_autoplaced yes)
-		(property "Reference" "#PWR09"
-			(at 236.22 66.04 0)
-			(effects
-				(font
-					(size 1.27 1.27)
-				)
-				(hide yes)
-			)
-		)
-		(property "Value" "GND"
-			(at 236.22 64.77 0)
-			(effects
-				(font
-					(size 1.27 1.27)
-				)
-			)
-		)
-		(property "Footprint" ""
-			(at 236.22 59.69 0)
-			(effects
-				(font
-					(size 1.27 1.27)
-				)
-				(hide yes)
-			)
-		)
-		(property "Datasheet" ""
-			(at 236.22 59.69 0)
-			(effects
-				(font
-					(size 1.27 1.27)
-				)
-				(hide yes)
-			)
-		)
-		(property "Description" "Power symbol creates a global label with name \"GND\" , ground"
-			(at 236.22 59.69 0)
-			(effects
-				(font
-					(size 1.27 1.27)
-				)
-				(hide yes)
-			)
-		)
-		(pin "1"
-		)
-		(instances
-			(project ""
-				(path "/7db5226c-054a-443a-bdfe-e8f86c4e465d"
-					(reference "#PWR09")
-					(unit 1)
-				)

Commit message: updates to esp32 IMU
Parts:
- J1: value +5V -> Conn_01x02; footprint Connector_PinHeader_1.00mm:PinHeader_1x02_P1.00mm_Vertical -> Connector_Wire:SolderWire-0.75sqmm_1x02_P4.8mm_D1.25mm_OD2.3mm_Relief2x
Changed lines of the file:
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@@
 	(wire
 		(pts
-			(xy 194.31 54.61) (xy 196.85 54.61)
+			(xy 194.31 54.61) (xy 200.66 54.61)
 		)
 		(stroke
@@
 	(wire
 		(pts
-			(xy 193.04 52.07) (xy 196.85 52.07)
+			(xy 193.04 52.07) (xy 200.66 52.07)
 		)
 		(stroke
@@
 				(justify left)
 				(hide yes)
-			)
-		)
-	)
-	(symbol
-		(lib_id "Connector_Generic:Conn_01x02")
-		(at 201.93 52.07 0)
-		(unit 1)
-		(exclude_from_sim no)
-		(in_bom yes)
-		(on_board yes)
-		(dnp no)
-		(fields_autoplaced yes)
-		(property "Reference" "J1"
-			(at 204.47 52.0699 0)
-			(effects
-				(font
-					(size 1.27 1.27)
-				)
-				(justify left)
-			)
-		)
-		(property "Value" "+5V"
-			(at 204.47 54.6099 0)
-			(effects
-				(font
-					(size 1.27 1.27)
-				)
-				(justify left)
-			)
-		)
-		(property "Footprint" "Connector_PinHeader_1.00mm:PinHeader_1x02_P1.00mm_Vertical"
-			(at 201.93 52.07 0)
-			(effects
-				(font
-					(size 1.27 1.27)
-				)
-				(hide yes)
-			)
-		)
-		(property "Datasheet" "~"
-			(at 201.93 52.07 0)
-			(effects
-				(font
-					(size 1.27 1.27)
-				)
-				(hide yes)
-			)
-		)
-		(property "Description" "Generic connector, single row, 01x02, script generated (kicad-library-utils/schlib/autogen/connector/)"
-			(at 201.93 52.07 0)
-			(effects
-				(font
-					(size 1.27 1.27)
-				)
-				(hide yes)
-			)
-		)
-		(pin "1"
-		)
-		(pin "2"
-		)
-		(instances
-			(project ""
-				(path "/7db5226c-054a-443a-bdfe-e8f86c4e465d"
-					(reference "J1")
-					(unit 1)
-				)
 			)
 		)
@@
 					(unit 1)
 				)
+			)
+		)
+	)
+	(symbol
+		(lib_id "Connector_Generic:Conn_01x02")
+		(at 205.74 52.07 0)
+		(unit 1)
+		(exclude_from_sim no)
+		(in_bom yes)
+		(on_board yes)
+		(dnp no)
+		(fields_autoplaced yes)
+		(property "Reference" "J1"
+			(at 208.28 52.0699 0)
+			(effects
+				(font
+					(size 1.27 1.27)
+				)
+				(justify left)
+			)
+		)
+		(property "Value" "Conn_01x02"
+			(at 208.28 54.6099 0)
+			(effects
+				(font
+					(size 1.27 1.27)
+				)
+				(justify left)
+				(hide yes)
+			)
+		)
+		(property "Footprint" "Connector_Wire:SolderWire-0.75sqmm_1x02_P4.8mm_D1.25mm_OD2.3mm_Relief2x"
+			(at 205.74 52.07 0)
+			(effects
+				(font
+					(size 1.27 1.27)
+				)
+				(hide yes)
+			)
+		)
+		(property "Datasheet" "~"
+			(at 205.74 52.07 0)
+			(effects
+				(font
+					(size 1.27 1.27)
+				)
+				(hide yes)
+			)
+		)
+		(property "Description" "Generic connector, single row, 01x02, script generated (kicad-library-utils/schlib/autogen/connector/)"
+			(at 205.74 52.07 0)
+			(effects
+				(font
+					(size 1.27 1.27)
+				)
+				(hide yes)
+			)
+		)
+		(pin "2"
+		)
+		(pin "1"
+		)
+		(instances
+			(project ""
+				(path "/7db5226c-054a-443a-bdfe-e8f86c4e465d"
+					(reference "J1")
+					(unit 1)
+				)

Commit message: Updates to IMU and Temp PCB
Parts:
- added J2: CAN to outer connector, Connector_Wire:SolderWire-0.1sqmm_1x04_P3.6mm_D0.4mm_OD1mm_Relief, symbol Connector_Generic:Conn_01x04
- added J3, J4: Conn_01x02, Connector_PinHeader_2.54mm:PinHeader_1x02_P2.54mm_Vertical, symbol Connector_Generic:Conn_01x02
Connections:
- new net Green 1: J2.1 (Pin_1), J3.1 (Pin_1)
- new net Green 2: J2.3 (Pin_3), J4.1 (Pin_1)
- new net White 1: J2.2 (Pin_2), J3.2 (Pin_2)
- new net White 2: J2.4 (Pin_4), J4.2 (Pin_2)
Other:
- note added: "I/O"
- note removed: "Power"
- moved on the sheet: J1

Commit message: Updates to IMU and Temp.
Other:
- note added: "Connector Pinout"
- moved on the sheet: J1, J2, J3, J4, UNIT_1, UNIT_3

Commit message: finished imu, started others
Parts:
- removed J3, J4: Conn_01x02, Connector_PinHeader_2.54mm:PinHeader_1x02_P2.54mm_Vertical, symbol Connector_Generic:Conn_01x02
- added J3: Conn_01x06, symbol Connector_Generic:Conn_01x06
- J1: footprint Connector_Wire:SolderWire-0.75sqmm_1x02_P4.8mm_D1.25mm_OD2.3mm_Relief2x -> Connector_Wire:SolderWire-0.75sqmm_1x02_P4.8mm_D1.25mm_OD2.3mm
- J2: footprint Connector_Wire:SolderWire-0.1sqmm_1x04_P3.6mm_D0.4mm_OD1mm_Relief -> Connector_Wire:SolderWire-0.1sqmm_1x04_P3.6mm_D0.4mm_OD1mm
- UNIT_2: value HiLetgo CAN Bus -> CAN Bus
Connections:
- net Green 2 is gone; now on net Low: J2.3 (Pin_3)
- net White 2 is gone; now on net High: J2.4 (Pin_4)
- net Green 1 renamed Low
- net Low: now also UNIT_2.9 (Low_CAN)
- net White 1 renamed High
- net High: now also UNIT_2.8 (High_CAN)
- no-connect marks 33 -> 35
Other:
- note added: "+5v"
- note added: "GND"
- note added: "High"
- note added: "Low"
- moved on the sheet: J2
