File: hardware/KICAD Projects/BAJE SAE/Sensor Projects/Temperature Sensor/Temperature Sensor.kicad_sch (KiCad schematic)
At the start: 8 parts, among them J1 +5V, J2 Bypass, U1 BA50JC5T

Commit message: Updates to IMU and Temp PCB
Parts:
- removed C1: 22u, Capacitor_THT:CP_Axial_L11.0mm_D8.0mm_P15.00mm_Horizontal, symbol Device:C_Polarized
- removed C2: .33u, Capacitor_THT:C_Axial_L3.8mm_D2.6mm_P7.50mm_Horizontal, symbol Device:C
- removed J1: +5V, Connector_PinHeader_1.00mm:PinHeader_1x02_P1.00mm_Vertical, symbol Connector_Generic:Conn_01x02
- removed J2: Bypass, Connector_PinHeader_1.00mm:PinHeader_1x02_P1.00mm_Vertical, symbol Connector_Generic:Conn_01x02
- removed U1: BA50JC5T, Package_TO_SOT_THT:TO-220-3_Horizontal_TabDown, symbol Regulator_Linear:LF80_TO220
- added J3, J4: Conn_01x02, Connector_PinHeader_2.54mm:PinHeader_1x02_P2.54mm_Vertical, symbol Connector_Generic:Conn_01x02
- added J5: Conn_01x02, Connector_Wire:SolderWire-0.75sqmm_1x02_P4.8mm_D1.25mm_OD2.3mm_Relief2x, symbol Connector_Generic:Conn_01x02
- added J6: CAN to outer connector, Connector_Wire:SolderWire-0.1sqmm_1x04_P3.6mm_D0.4mm_OD1mm_Relief, symbol Connector_Generic:Conn_01x04
Connections:
- new net +5v: J5.1 (Pin_1)
- new net GND: J5.2 (Pin_2)
- new net Green 1: J3.1 (Pin_1), J6.1 (Pin_1)
- new net Green 2: J4.1 (Pin_1), J6.3 (Pin_3)
- new net White 1: J3.2 (Pin_2), J6.2 (Pin_2)
- new net White 2: J4.2 (Pin_2), J6.4 (Pin_4)
Other:
- note added: "CAN Bus"
- note added: "I/O"
- note added: "Nano"
- note added: "Temp Sensor"
- moved on the sheet: UNIT_1, UNIT_2, UNIT_3

Commit message: finished imu, started others
Parts:
- removed J3, J4: Conn_01x02, Connector_PinHeader_2.54mm:PinHeader_1x02_P2.54mm_Vertical, symbol Connector_Generic:Conn_01x02
- removed J6: CAN to outer connector, Connector_Wire:SolderWire-0.1sqmm_1x04_P3.6mm_D0.4mm_OD1mm_Relief, symbol Connector_Generic:Conn_01x04
- added J2: CAN to outer connector, Connector_Wire:SolderWire-0.1sqmm_1x04_P3.6mm_D0.4mm_OD1mm, symbol Connector_Generic:Conn_01x04
- added J3: Conn_01x06, symbol Connector_Generic:Conn_01x06
- J5: footprint Connector_Wire:SolderWire-0.75sqmm_1x02_P4.8mm_D1.25mm_OD2.3mm_Relief2x -> Connector_Wire:SolderWire-0.75sqmm_1x02_P4.8mm_D1.25mm_OD2.3mm
- UNIT_2: footprint BAJA SAE:HiLetgo CAN Bus (Facing Up) -> BAJA SAE:HiLetgo CAN Bus; symbol BAJA SAE:HiLetgo_CAN_BUS -> 0_Baja_Final:HiLetgo_CAN_BUS
Connections:
- new net High: J2.2 (Pin_2), J2.4 (Pin_4), UNIT_2.8 (High_CAN)
- new net Low: J2.1 (Pin_1), J2.3 (Pin_3), UNIT_2.9 (Low_CAN)
Other:
- note added: "+5v"
- note added: "Connector Pinout"
- note added: "ESP-32 Socketed with ESS-119-T-03"
- note added: "GND"
- note added: "High"
- note added: "Low"
- note added: "Socket"
- moved on the sheet: J5, UNIT_3

Commit message: Removed KICAD Symbol Libraries
Other:
- note added: "Nano socketed with HWS16130 http://www.peconnectors.com/sockets-sip-machined/ hws16130/?utm_source=googleads&vt_keyword=&gad_source= 1&gbraid=0AAAAAD-J6wRIeL1mScc81doEXt4u-oFxN&gclid=Cj0KC QiA4rK8BhD7ARIsAFe5LXJCXX4yoeMSgdYYrUZ8CYCOGg6YWjx-KireWWb9vicOqA-PgvhT3uIaAs8kEALw_wcB"
- note removed: "ESP-32 Socketed with ESS-119-T-03"
Changed lines of the file:
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@@
+	(wire
+		(pts
+			(xy 93.98 143.51) (xy 92.71 143.51)
+		)
+		(stroke
+			(width 0)
+			(type default)
+		)
+	)
 	(wire
 		(pts
@@
 	)
 	(rectangle
-		(start 197.2308 79.6376)
-		(end 229.9208 94.9892)
+		(start 118.2368 108.5936)
+		(end 218.186 123.9452)
 		(stroke
 			(width 0)
@@
 		)
 	)
-	(text "ESP-32 Socketed with \nESS-119-T-03"
-		(exclude_from_sim no)
-		(at 214.376 87.884 0)
+	(text "Nano socketed with \nHWS16130\nhttp://www.peconnectors.com/sockets-sip-machined/\nhws16130/?utm_source=googleads&vt_keyword=&gad_source=\n1&gbraid=0AAAAAD-J6wRIeL1mScc81doEXt4u-oFxN&gclid=Cj0KC\nQiA4rK8BhD7ARIsAFe5LXJCXX4yoeMSgdYYrUZ8CYCOGg6YWjx-KireWWb9vicOqA-PgvhT3uIaAs8kEALw_wcB"
+		(exclude_from_sim no)
+		(at 168.91 116.84 0)
 		(effects
 			(font
@@
 	(text "Socket"
 		(exclude_from_sim no)
-		(at 200.66 78.74 0)
+		(at 121.666 107.696 0)
 		(effects
 			(font
@@
 	(global_label "High"
 		(shape input)
-		(at 92.71 143.51 0)
+		(at 93.98 143.51 0)
 		(fields_autoplaced yes)
 		(effects
@@
 		)
 		(property "Intersheetrefs" "${INTERSHEET_REFS}"
-			(at 99.9285 143.51 0)
-			(effects
-				(font
+			(at 101.1985 143.51 0)
+			(effects
+				(font

Commit message: re-added symbol library
Connections:
- net GND is gone; now on net 0: J5.2 (Pin_2)
Changed lines of the file:
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@@
+	(wire
+		(pts
+			(xy 102.87 71.12) (xy 102.87 67.31)
+		)
+		(stroke
+			(width 0)
+			(type default)
+		)
+	)
 	(wire
 		(pts
@@
 		(pts
 			(xy 148.59 58.42) (xy 148.59 59.69)
+		)
+		(stroke
+			(width 0)
+			(type default)
+		)
+	)
+	(wire
+		(pts
+			(xy 102.87 67.31) (xy 100.33 67.31)
 		)
 		(stroke
@@
 		)
 	)
+	(global_label "GND"
+		(shape input)
+		(at 100.33 67.31 180)
+		(fields_autoplaced yes)
+		(effects
+			(font
+				(size 1.27 1.27)
+			)
+			(justify right)
+		)
+		(property "Intersheetrefs" "${INTERSHEET_REFS}"
+			(at 93.4743 67.31 0)
+			(effects
+				(font
+					(size 1.27 1.27)
+				)
+				(justify right)
+				(hide yes)
+			)
+		)
+	)
 	(global_label "+5v"
 		(shape output)
@@
 					(unit 1)
 				)
+			)
+		)
+	)
+	(symbol
+		(lib_id "Simulation_SPICE:0")
+		(at 102.87 71.12 0)
+		(unit 1)
+		(exclude_from_sim no)
+		(in_bom yes)
+		(on_board yes)
+		(dnp no)
+		(fields_autoplaced yes)
+		(property "Reference" "#GND04"
+			(at 102.87 76.2 0)
+			(effects
+				(font
+					(size 1.27 1.27)
+				)
+				(hide yes)
+			)
+		)
+		(property "Value" "0"
+			(at 102.87 68.58 0)
+			(effects
+				(font
+					(size 1.27 1.27)
+				)
+				(hide yes)
+			)
+		)
+		(property "Footprint" ""
+			(at 102.87 71.12 0)
+			(effects
+				(font
+					(size 1.27 1.27)
+				)
+				(hide yes)
+			)
+		)
+		(property "Datasheet" "https://ngspice.sourceforge.io/docs/ngspice-html-manual/manual.xhtml#subsec_Circuit_elements__device"
+			(at 102.87 81.28 0)
+			(effects
+				(font
+					(size 1.27 1.27)
+				)
+				(hide yes)
+			)
+		)
+		(property "Description" "0V reference potential for simulation"
+			(at 102.87 78.74 0)
+			(effects
+				(font
+					(size 1.27 1.27)
+				)
+				(hide yes)
+			)
+		)
+		(pin "1"
+		)
+		(instances
+			(project "Temperature Sensor"
+				(path "/74467775-d059-4e20-8fe4-b429e963843c"
+					(reference "#GND04")
+					(unit 1)
+				)
