File: hardware/KICAD Projects/BAJE SAE/Sensor Projects/Temperature Sensor/Temperature Sensor.kicad_pcb (KiCad board)
At the start: 2 copper layers, 56.5 x 80.8 mm, 13 parts, among them J1 +5V, J2 Bypass, U1 BA50JC5T

Commit message: Corrected onboard labels from IMU to TEMP on temperature sensor
Other:
- board text added: "CVT TEMP SENSOR"
- board text added: "CVT Temperature Sensor"
- board text removed: "IMU SENSOR"
- board text removed: "Temperature Sensor"
Changed lines of the file:
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@@
 		)
 	)
-	(gr_text "IMU SENSOR"
+	(gr_text "CVT TEMP SENSOR"
 		(at 139.75 71.25 90)
 		(layer "F.SilkS")
@@
 		)
 	)
-	(gr_text "Temperature Sensor"
+	(gr_text "CVT Temperature Sensor"
 		(at 155.75 38.25 0)
 		(layer "F.SilkS")

Commit message: Updates to IMU and Temp PCB
Parts:
- removed C1: 22u, Capacitor_THT:CP_Axial_L11.0mm_D8.0mm_P15.00mm_Horizontal
- removed C2: .33u, Capacitor_THT:C_Axial_L3.8mm_D2.6mm_P7.50mm_Horizontal
- removed J1: +5V, Connector_PinHeader_1.00mm:PinHeader_1x02_P1.00mm_Vertical
- removed J2: Bypass, Connector_PinHeader_1.00mm:PinHeader_1x02_P1.00mm_Vertical
- removed REF** (x4): MountingHole_4.5mm, MountingHole:MountingHole_4.5mm
- removed U1: BA50JC5T, Package_TO_SOT_THT:TO-220-3_Horizontal_TabDown
- removed UNIT_3: ~, BAJA SAE:GY-906 (Facing Down)
- added J3: Conn_01x02, Connector_PinHeader_2.54mm:PinHeader_1x02_P2.54mm_Vertical, F.Cu at (96.1, 61.1)
- added J4: Conn_01x02, Connector_PinHeader_2.54mm:PinHeader_1x02_P2.54mm_Vertical, F.Cu at (100.8, 61.1)
- added J5: Conn_01x02, Connector_Wire:SolderWire-0.75sqmm_1x02_P4.8mm_D1.25mm_OD2.3mm_Relief2x, F.Cu at (135.5, 124.3)
- added J6: CAN to outer connector, Connector_Wire:SolderWire-0.1sqmm_1x04_P3.6mm_D0.4mm_OD1mm_Relief, F.Cu at (95.6, 51.0)
- moved UNIT_1 99.0 mm to (111.0, 129.4), turned to 180 degrees
- moved UNIT_2 84.5 mm to (111.3, 135.5), turned to 90 degrees
Routing:
- net 0: track 133.1 -> 0.00 mm
- net +5V: track 65.5 -> 0.00 mm
- net SO: track 64.3 -> 0.00 mm
- net SI: track 61.1 -> 0.00 mm
- net SCK: track 59.6 -> 0.00 mm
- net SCL: track 17.3 -> 0.00 mm
- net SDA: track 12.2 -> 0.00 mm
- net Net-(J1-Pin_1): track 11.6 -> 0.00 mm
- net +3V: track 5.01 -> 0.00 mm
Other:
- board text removed: "+-"
- board text removed: "CAN Bus"
- board text removed: "Nano"
- board text removed: "SCK"

Commit message: Updates to temperature sensor PCB
Parts:
- added UNIT_3: ~, BAJA SAE:GY-906 (Facing Down), B.Cu at (109.9, 102.6)
- J5: footprint Connector_Wire:SolderWire-0.75sqmm_1x02_P4.8mm_D1.25mm_OD2.3mm_Relief2x -> Connector_Wire:SolderWire-0.75sqmm_1x02_P4.8mm_D1.25mm_OD2.3mm_Relief
- UNIT_2: moved to B.Cu
- moved J6 106.3 mm to (105.9, 156.8)
- moved J3 84.2 mm to (108.9, 144.3)
- moved J4 84.2 mm to (113.5, 144.3)
- moved J5 27.0 mm to (108.5, 122.5)
- moved UNIT_2 6.11 mm to (110.9, 129.4), turned to -90 degrees
- moved UNIT_1 3.04 mm to (111.0, 132.4)
Other:
- board size 56.5 x 80.8 mm -> 28.3 x 68.6 mm

Commit message: finished imu, started others
Parts:
- removed J3, J4: Conn_01x02, Connector_PinHeader_2.54mm:PinHeader_1x02_P2.54mm_Vertical
- removed J6: CAN to outer connector, Connector_Wire:SolderWire-0.1sqmm_1x04_P3.6mm_D0.4mm_OD1mm_Relief
- added G***: LOGO, BAJA SAE:Baja Logo, F.Cu at (143.8, 124.5)
- added J2: CAN to outer connector, Connector_Wire:SolderWire-0.1sqmm_1x04_P3.6mm_D0.4mm_OD1mm, F.Cu at (150.0, 64.5)
- J5: footprint Connector_Wire:SolderWire-0.75sqmm_1x02_P4.8mm_D1.25mm_OD2.3mm_Relief -> Connector_Wire:SolderWire-0.75sqmm_1x02_P4.8mm_D1.25mm_OD2.3mm
- UNIT_2: footprint BAJA SAE:HiLetgo CAN Bus (Facing Up) -> 0_Baja_Final:HiLetgo CAN Bus (Facing Up)
- moved J5 62.9 mm to (141.9, 69.2)
- moved UNIT_1 47.6 mm to (144.6, 98.7)
- moved UNIT_3 43.7 mm to (144.2, 75.5), turned to 0 degrees
- moved G*** 42.0 mm to (143.2, 68.0)
- moved UNIT_2 36.6 mm to (142.1, 110.3), turned to 90 degrees
Other:
- board size 28.3 x 68.6 mm -> 30.5 x 73.3 mm
- board text added: "H"
- board text added: "L"
- board text added: "Temp"
- board text added: "UNIVERSITY OF ARIZONA Connor Larson Jan, 2025"
- board text removed: "UNIVERSITY OF ARIZONA Connor Larson Nov, 2024"

Commit message: Removed KICAD Symbol Libraries
Parts:
- removed the G*** at (143.2, 68.0)
- moved UNIT_3 2.05 mm to (144.2, 73.5)
- moved G*** 1.77 mm to (144.0, 126.2)
- moved J5 0.15 mm to (142.1, 69.2)
- moved J2 0.10 mm to (149.9, 64.5)
- moved UNIT_1 0.08 mm to (144.6, 98.8)
- moved UNIT_2 0.06 mm to (142.1, 110.2)
Connections:
- UNIT_1 pad 29: 0 -> GND
- UNIT_1 pad 4: 0 -> GND
- UNIT_2 pad 8: (no net) -> Low
- UNIT_2 pad 9: (no net) -> High
- UNIT_3 pad 2: 0 -> GND
Routing:
- net GND: track 0.00 -> 61.8 mm
- net SO: track 0.00 -> 43.0 mm, vias 2 -> 1
- net SI: track 0.00 -> 40.9 mm
- net SCK: track 0.00 -> 40.2 mm
- net +5V: track 0.00 -> 35.9 mm
- net Low: track 0.00 -> 35.5 mm
- net High: track 0.00 -> 35.2 mm
- net SDA: track 0.00 -> 25.0 mm, vias 0 -> 2
- net SCL: track 0.00 -> 24.6 mm, vias 0 -> 1
- net +3V: track 0.00 -> 4.13 mm
Other:
- outline, holes or cut-outs redrawn
- board text added: "+"
- board text added: "16 SCK"
- board text added: "NANO THIS SIDE"
- board text removed: "CVT TEMP SENSOR"
- board text removed: "PN: TEMP1"
- board text removed: "SN:"
- board text removed: "Temp"

Commit message: re-added symbol library
Other:
- outline, holes or cut-outs redrawn
Changed lines of the file:
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@@
 	)
 	(gr_arc
-		(start 158.47 59.75)
-		(mid 159.368026 60.121974)
-		(end 159.74 61.02)
+		(start 158.48 59.728026)
+		(mid 159.378026 60.1)
+		(end 159.75 60.998026)
 		(stroke
 			(width 0.05)
@@
 	)
 	(gr_arc
-		(start 129.258026 61.018026)
-		(mid 129.629993 60.119993)
-		(end 130.528026 59.748026)
-		(locked yes)
-		(stroke
-			(width 0.05)
-			(type default)
-		)
-		(layer "Edge.Cuts")
-	)
-	(gr_line
-		(start 130.53 59.75)
-		(end 158.47 59.75)
-		(locked yes)
+		(start 129.25 60.998026)
+		(mid 129.621967 60.099993)
+		(end 130.52 59.728026)
+		(stroke
+			(width 0.05)
+			(type default)
+		)
+		(layer "Edge.Cuts")
+	)
+	(gr_line
+		(start 159.75 60.998026)
+		(end 159.75 61.19)
+		(stroke
+			(width 0.05)
+			(type default)
+		)
+		(layer "Edge.Cuts")
+	)
+	(gr_line
+		(start 130.66 59.728026)
+		(end 158.48 59.728026)
 		(stroke
 			(width 0.05)
@@
 	(gr_line
 		(start 130.52 133.064)
-		(end 158.5 133.064)
+		(end 158.25 133.064)
+		(stroke
+			(width 0.05)
+			(type default)
+		)
+		(layer "Edge.Cuts")
+	)
+	(gr_line
+		(start 130.52 59.728026)
+		(end 130.66 59.728026)
 		(stroke
 			(width 0.05)
@@
 	(gr_line
 		(start 159.75 131.794)
-		(end 159.74 61.02)
-		(stroke
-			(width 0.05)
-			(type default)
-		)
-		(layer "Edge.Cuts")
-	)
-	(gr_line
-		(start 129.26 61.02)
+		(end 159.75 61.19)
+		(stroke
+			(width 0.05)
+			(type default)
+		)
+		(layer "Edge.Cuts")
+	)
+	(gr_line
+		(start 129.25 61)
 		(end 129.25 131.794)
 		(stroke
@@
 		(layer "Edge.Cuts")
 	)
+	(gr_line
+		(start 158.48 133.064)
+		(end 158.25 133.064)
+		(stroke
+			(width 0.05)
+			(type default)
+		)
+		(layer "Edge.Cuts")
+	)
 	(gr_text "16 SCK"
-		(at 134.75 79.5 0)
+		(at 136 79.5 0)
 		(layer "F.SilkS")
 		(effects
@@
 		)
 	)
-	(dimension
-		(type aligned)
-		(layer "F.Fab")
-		(pts
-			(xy 129.25 61.5) (xy 159.74 61.5)
-		)
-		(height -9)
-		(gr_text "30.4900 mm"
-			(at 144.495 51.35 0)
-			(layer "F.Fab")
-			(effects
-				(font
-					(size 1 1)
-					(thickness 0.15)
-				)
-			)
-		)
-		(format
-			(prefix "")
-			(suffix "")
-			(units 3)
-			(units_format 1)
-			(precision 4)
-		)
-		(style
-			(thickness 0.1)
-			(arrow_length 1.27)
-			(text_position_mode 0)
-			(extension_height 0.58642)
-			(extension_offset 0.5) keep_text_aligned)
-	)
 	(segment

Commit message: finished pcbs yayyyy
Connections:
- J5 pad 1: +5v -> +5V
- UNIT_1 pad 13: unconnected-(UNIT_1-D10-Pad13) -> CS
- UNIT_2 pad 6: 0 -> GND
- UNIT_2 pad 8: Low -> High
- UNIT_2 pad 9: High -> Low
Routing:
- net CS: track 0.00 -> 39.8 mm, vias 0 -> 1
- net +5V: track 35.9 -> 60.5 mm
- net GND: track 61.8 -> 69.0 mm
- net SCK: track 40.2 -> 46.8 mm
- net Low: track 35.5 -> 36.8 mm
- net High: track 35.2 -> 36.4 mm
- net SI: track 40.9 -> 40.0 mm, vias 0 -> 1
Other:
- board text added: "Designed by Connor & Matthew Larson in Tucson, AZ"
- board text removed: "UNIVERSITY OF ARIZONA Connor Larson Jan, 2025"
