File: hardware/KICAD Projects/BAJE SAE/Sensor Projects/Temperature Sensor/Temperature Sensor.kicad_pcb (KiCad board)
At the start: 2 copper layers, 30.5 x 73.3 mm, 6 parts, among them J2 CAN to outer connector, J5 Conn_01x02

Commit message: temp sense worky now
Parts:
- UNIT_2: footprint 0_Baja_Final:HiLetgo CAN Bus (Facing Up) -> 0_Baja_2025:CAN Bus (Feb 2025)
- UNIT_3: moved to F.Cu
- moved UNIT_2 9.15 mm to (146.8, 102.4)
- moved UNIT_3 0.56 mm to (144.4, 73.0), turned to 180 degrees
Routing:
- net +3V: track 4.13 -> 15.4 mm
- net SDA: track 25.0 -> 18.8 mm, vias 2 -> 0
- net Low: track 36.8 -> 34.5 mm
- net GND: track 69.0 -> 68.0 mm
- net SCL: track 24.6 -> 25.4 mm
- net High: track 36.4 -> 35.9 mm
Other:
- board text added: "CVT Temperature Sensor Rev 2"
- board text removed: "CVT Temperature Sensor"
