File: hardware/KICAD Projects/BAJE SAE/Sensor Projects/Tachometer/Tachometerkicad.kicad_pcb (KiCad board)
At the start: 2 copper layers, 24 parts, among them J1 Conn_01x02, J3 Conn_01x02, J4 CAN to outer connector, Q1 NPN, U1 NE555P, U2 TL071

Commit message: created tachometer platformio project
Parts:
- removed R8: 430, Resistor_THT:R_Axial_DIN0411_L9.9mm_D3.6mm_P7.62mm_Vertical
- added R4: 430, Resistor_THT:R_Axial_DIN0411_L9.9mm_D3.6mm_P15.24mm_Horizontal, F.Cu at (271.0, 89.1)
- added REF**: MountingHole_3.2mm_M3, MountingHole:MountingHole_3.2mm_M3, F.Cu at (383.5, 98.0)
- C1, C2, C3: value 10microferret -> 10u
- D1: value D_Zener -> ~
- R1, R2, R3: footprint Resistor_THT:R_Axial_DIN0411_L9.9mm_D3.6mm_P12.70mm_Horizontal -> Resistor_THT:R_Axial_DIN0411_L9.9mm_D3.6mm_P15.24mm_Horizontal
- R10, R11, R5, R6, R7: footprint Resistor_THT:R_Axial_DIN0411_L9.9mm_D3.6mm_P7.62mm_Vertical -> Resistor_THT:R_Axial_DIN0411_L9.9mm_D3.6mm_P15.24mm_Horizontal
- U2: value TL071 -> LM311
- UNIT_2: moved to B.Cu
- moved R11 189.8 mm to (256.3, 193.8)
- moved R5 189.8 mm to (256.3, 168.1)
- moved C2 189.8 mm to (268.0, 187.1)
- moved C1 189.6 mm to (267.8, 180.5)
- moved R7 187.9 mm to (279.0, 89.1), turned to 90 degrees
- moved C4 180.1 mm to (257.5, 115.0)
- moved C3 175.0 mm to (277.8, 105.5)
- moved R6 172.4 mm to (263.5, 74.4), turned to -90 degrees
- moved J4 144.6 mm to (148.0, 130.5), turned to 180 degrees
- moved R10 121.0 mm to (211.9, 103.5)
- moved UNIT_1 99.6 mm to (143.1, 103.5)
- moved Q1 97.0 mm to (51.3, 97.5)
- moved UNIT_2 77.8 mm to (145.0, 89.5), turned to -90 degrees
- moved J1 76.3 mm to (141.1, 120.5)
- moved R1 68.5 mm to (40.9, 84.5)
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Connections:
- U2 pad 1: unconnected-(U2-NULL-Pad1) -> GND
- U2 pad 2: Net-(U2--) -> Comparator input
- U2 pad 3: Comparator input -> Net-(U2--)
- U2 pad 6: 555 input -> unconnected-(U2-STRB-Pad6)
- U2 pad 7: +5v -> 555 input
- U2 pad 8: unconnected-(U2-NC-Pad8) -> +5v
Other:
- board outline added: 81 x 89 mm
