File: hardware/KICAD Projects/BAJE SAE/Sensor Projects/Tachometer/Tachometerkicad.kicad_sch (KiCad schematic)
At the start: 25 parts, among them J1 Conn_01x02, J2 Conn_01x06, J3 Conn_01x02, J4 CAN to outer connector, Q1 NPN, U1 NE555P, U2 TL071

Commit message: the last struggle
Parts:
- removed U2: TL071, Package_DIP:DIP-8_W7.62mm, symbol Amplifier_Operational:TL071
- added U2: LM311, Package_DIP:DIP-8_W7.62mm, symbol Comparator:LM311
- C1, C2, C3: value 10microferret -> 10u
- D1: value D_Zener -> ~
Connections:
- net +5v: now also U2.8 (V+)
- net 0: now also U2.1 (GND), U2.4 (V-)
- net 555 input: now also U2.7
- net Comparator input: now also U2.2 (+)
- net at VR1.3: now also U2.3 (-)
Other:
- moved on the sheet: C3, J1, R10, R6, R7, R8, VR1

Commit message: created tachometer platformio project
Parts:
- removed R8: 430, Resistor_THT:R_Axial_DIN0411_L9.9mm_D3.6mm_P7.62mm_Vertical, symbol Device:R
- added R4: 430, Resistor_THT:R_Axial_DIN0411_L9.9mm_D3.6mm_P15.24mm_Horizontal, symbol Device:R
- C1, C2: symbol Device:C -> Device:C_Polarized
- R1, R2, R3: footprint Resistor_THT:R_Axial_DIN0411_L9.9mm_D3.6mm_P12.70mm_Horizontal -> Resistor_THT:R_Axial_DIN0411_L9.9mm_D3.6mm_P15.24mm_Horizontal
- R10, R11, R5, R6, R7: footprint Resistor_THT:R_Axial_DIN0411_L9.9mm_D3.6mm_P7.62mm_Vertical -> Resistor_THT:R_Axial_DIN0411_L9.9mm_D3.6mm_P15.24mm_Horizontal
Connections:
- net at R6.1: now also R4.2
- net at R7.2: now also R4.1
Changed lines of the file:
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@@
 			)
 		)
-		(property "Footprint" "Resistor_THT:R_Axial_DIN0411_L9.9mm_D3.6mm_P7.62mm_Vertical"
+		(property "Footprint" "Resistor_THT:R_Axial_DIN0411_L9.9mm_D3.6mm_P15.24mm_Horizontal"
 			(at 208.28 90.678 90)
 			(effects
@@
 	)
 	(symbol
-		(lib_id "Device:C")
+		(lib_id "Device:C_Polarized")
 		(at 198.12 92.71 0)
 		(unit 1)
@@
 		(fields_autoplaced yes)
 		(property "Reference" "C1"
-			(at 201.93 91.4399 0)
+			(at 201.93 90.5509 0)
 			(effects
 				(font
@@
 		)
 		(property "Value" "10u"
-			(at 201.93 93.9799 0)
+			(at 201.93 93.0909 0)
 			(effects
 				(font
@@
 			)
 		)
-		(property "Description" "Unpolarized capacitor"
+		(property "Description" "Polarized capacitor"
 			(at 198.12 92.71 0)
 			(effects
@@
 				(path "/d32b6a5f-c7f0-4229-a4f9-b1dde9133fa5"
 					(reference "C1")
+					(unit 1)
+				)
+			)
+		)
+	)
+	(symbol
+		(lib_id "Device:R")
+		(at 228.6 72.39 90)
+		(unit 1)
+		(exclude_from_sim no)
+		(in_bom yes)
+		(on_board yes)
+		(dnp no)
+		(fields_autoplaced yes)
+		(property "Reference" "R4"
+			(at 228.6 66.04 90)
+			(effects
+				(font
+					(size 1.27 1.27)
+				)
+			)
+		)
+		(property "Value" "430"
+			(at 228.6 68.58 90)
+			(effects
+				(font
+					(size 1.27 1.27)
+				)
+			)
+		)
+		(property "Footprint" "Resistor_THT:R_Axial_DIN0411_L9.9mm_D3.6mm_P15.24mm_Horizontal"
+			(at 228.6 74.168 90)
+			(effects
+				(font
+					(size 1.27 1.27)
+				)
+				(hide yes)
+			)
+		)
+		(property "Datasheet" "~"
+			(at 228.6 72.39 0)
+			(effects
+				(font
+					(size 1.27 1.27)
+				)
+				(hide yes)
+			)
+		)
+		(property "Description" "Resistor"
+			(at 228.6 72.39 0)
+			(effects
+				(font
+					(size 1.27 1.27)
+				)
+				(hide yes)
+			)
+		)
+		(pin "1"
+		)
+		(pin "2"
+		)
+		(instances
+			(project "Tachometerkicad"
+				(path "/d32b6a5f-c7f0-4229-a4f9-b1dde9133fa5"
+					(reference "R4")
 					(unit 1)
 				)
@@
 	)
 	(symbol
-		(lib_id "Device:C")
+		(lib_id "Device:C_Polarized")
 		(at 215.9 92.71 0)
 		(unit 1)
@@
 		(fields_autoplaced yes)
 		(property "Reference" "C2"
-			(at 219.71 91.4399 0)
+			(at 219.71 90.5509 0)
 			(effects
 				(font
@@
 		)
 		(property "Value" "10u"
-			(at 219.71 93.9799 0)
+			(at 219.71 93.0909 0)
 			(effects
 				(font
@@
 			)
 		)
-		(property "Description" "Unpolarized capacitor"
+		(property "Description" "Polarized capacitor"
 			(at 215.9 92.71 0)
 			(effects
@@
 			)
 		)
-		(property "Footprint" "Resistor_THT:R_Axial_DIN0411_L9.9mm_D3.6mm_P7.62mm_Vertical"
+		(property "Footprint" "Resistor_THT:R_Axial_DIN0411_L9.9mm_D3.6mm_P15.24mm_Horizontal"
 			(at 190.5 90.678 90)
 			(effects
@@
 			)
 		)
-		(property "Footprint" "Resistor_THT:R_Axial_DIN0411_L9.9mm_D3.6mm_P12.70mm_Horizontal"
+		(property "Footprint" "Resistor_THT:R_Axial_DIN0411_L9.9mm_D3.6mm_P15.24mm_Horizontal"
 			(at 95.25 36.068 90)
 			(effects
@@
 			)
 		)
-		(property "Footprint" "Resistor_THT:R_Axial_DIN0411_L9.9mm_D3.6mm_P7.62mm_Vertical"
+		(property "Footprint" "Resistor_THT:R_Axial_DIN0411_L9.9mm_D3.6mm_P15.24mm_Horizontal"
 			(at 238.76 74.168 90)
 			(effects
@@
 	)
 	(symbol
-		(lib_id "Device:R")
-		(at 228.6 72.39 90)
-		(unit 1)
-		(exclude_from_sim no)
-		(in_bom yes)
-		(on_board yes)
-		(dnp no)
-		(fields_autoplaced yes)
-		(property "Reference" "R8"
-			(at 228.6 66.04 90)
-			(effects
-				(font
-					(size 1.27 1.27)
-				)
-			)
-		)
-		(property "Value" "430"
-			(at 228.6 68.58 90)
-			(effects
-				(font
-					(size 1.27 1.27)
-				)
-			)
-		)
-		(property "Footprint" "Resistor_THT:R_Axial_DIN0411_L9.9mm_D3.6mm_P7.62mm_Vertical"
-			(at 228.6 74.168 90)
-			(effects
-				(font
-					(size 1.27 1.27)
-				)
-				(hide yes)
-			)
-		)
-		(property "Datasheet" "~"
-			(at 228.6 72.39 0)
-			(effects
-				(font
-					(size 1.27 1.27)
-				)
-				(hide yes)
-			)
-		)
-		(property "Description" "Resistor"
-			(at 228.6 72.39 0)
-			(effects
-				(font
-					(size 1.27 1.27)
-				)
-				(hide yes)
-			)
-		)
-		(pin "1"
-		)
-		(pin "2"
-		)
-		(instances
-			(project "Tachometerkicad"
-				(path "/d32b6a5f-c7f0-4229-a4f9-b1dde9133fa5"
-					(reference "R8")
-					(unit 1)
-				)
-			)
-		)
-	)
-	(symbol
 		(lib_id "Timer:NE555P")
 		(at 214.63 38.1 270)
@@
 			)
 		)
-		(property "Footprint" "Resistor_THT:R_Axial_DIN0411_L9.9mm_D3.6mm_P7.62mm_Vertical"
+		(property "Footprint" "Resistor_THT:R_Axial_DIN0411_L9.9mm_D3.6mm_P15.24mm_Horizontal"
 			(at 109.982 82.55 90)
 			(effects
@@
 			)
 		)
-		(property "Footprint" "Resistor_THT:R_Axial_DIN0411_L9.9mm_D3.6mm_P7.62mm_Vertical"
+		(property "Footprint" "Resistor_THT:R_Axial_DIN0411_L9.9mm_D3.6mm_P15.24mm_Horizontal"
 			(at 218.44 74.168 90)
 			(effects
@@
 			)
 		)
-		(property "Footprint" "Resistor_THT:R_Axial_DIN0411_L9.9mm_D3.6mm_P12.70mm_Horizontal"
+		(property "Footprint" "Resistor_THT:R_Axial_DIN0411_L9.9mm_D3.6mm_P15.24mm_Horizontal"
 			(at 63.5 36.068 90)
 			(effects
@@
 			)
 		)
-		(property "Footprint" "Resistor_THT:R_Axial_DIN0411_L9.9mm_D3.6mm_P12.70mm_Horizontal"
+		(property "Footprint" "Resistor_THT:R_Axial_DIN0411_L9.9mm_D3.6mm_P15.24mm_Horizontal"
 			(at 108.712 22.86 90)
 			(effects

Commit message: tach updat :P
Parts:
- D1, D2: footprint Diode_THT:D_A-405_P5.08mm_Vertical_AnodeUp -> Diode_THT:D_A-405_P7.62mm_Horizontal
- R1, R10, R11, R2, R3, R4, R5, R6, R7: symbol Device:R -> Device:R_US
Connections:
- net Negative is gone; now on net 0: J1.1 (Pin_1)
- net arduino input: now also UNIT_1.19 (A0); no longer UNIT_1.2 (D0/RX)
Changed lines of the file:
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@@
 	)
 	(no_connect
+		(at 107.95 158.75)
+	)
+	(no_connect
 		(at 107.95 123.19)
 	)
@@
 	)
 	(no_connect
-		(at 85.09 158.75)
-	)
-	(no_connect
 		(at 80.01 158.75)
 	)
@@
 	(wire
 		(pts
+			(xy 85.09 158.75) (xy 85.09 162.56)
+		)
+		(stroke
+			(width 0)
+			(type default)
+		)
+	)
+	(wire
+		(pts
 			(xy 96.52 85.09) (xy 96.52 86.36)
 		)
@@
 	(wire
 		(pts
-			(xy 107.95 158.75) (xy 107.95 166.37)
-		)
-		(stroke
-			(width 0)
-			(type default)
-		)
-	)
-	(wire
-		(pts
 			(xy 212.09 88.9) (xy 215.9 88.9)
 		)
@@
 	(wire
 		(pts
-			(xy 31.75 57.15) (xy 27.94 57.15)
+			(xy 27.94 57.15) (xy 35.56 57.15)
 		)
 		(stroke
@@
 	)
 	(rectangle
-		(start 54.7776 169.2124)
-		(end 141.8 108.392)
+		(start 54.7776 108.392)
+		(end 141.8 169.2124)
 		(stroke
 			(width 0)
@@
 	(global_label "arduino input"
 		(shape input)
-		(at 107.95 166.37 0)
+		(at 85.09 162.56 270)
+		(fields_autoplaced yes)
+		(effects
+			(font
+				(size 1.27 1.27)
+			)
+			(justify right)
+		)
+		(property "Intersheetrefs" "${INTERSHEET_REFS}"
+			(at 85.09 178.4263 90)
+			(effects
+				(font
+					(size 1.27 1.27)
+				)
+				(justify right)
+				(hide yes)
+			)
+		)
+	)
+	(global_label "GND"
+		(shape input)
+		(at 35.56 57.15 0)
 		(fields_autoplaced yes)
 		(effects
@@
 		)
 		(property "Intersheetrefs" "${INTERSHEET_REFS}"
-			(at 123.8163 166.37 0)
+			(at 42.4157 57.15 0)
 			(effects
 				(font
@@
 		)
 	)
-	(global_label "Negative"
-		(shape input)
-		(at 31.75 57.15 0)
-		(fields_autoplaced yes)
-		(effects
-			(font
-				(size 1.27 1.27)
-			)
-			(justify left)
-		)
-		(property "Intersheetrefs" "${INTERSHEET_REFS}"
-			(at 42.839 57.15 0)
-			(effects
-				(font
-					(size 1.27 1.27)
-				)
-				(justify left)
-				(hide yes)
-			)
-		)
-	)
 	(global_label "SI"
 		(shape input)
@@
 			)
 		)
-		(property "Footprint" "Diode_THT:D_A-405_P5.08mm_Vertical_AnodeUp"
+		(property "Footprint" "Diode_THT:D_A-405_P7.62mm_Horizontal"
 			(at 73.66 38.1 0)
 			(effects
@@
 	)
 	(symbol
-		(lib_id "Device:R")
+		(lib_id "Device:R_US")
 		(at 208.28 88.9 90)
 		(unit 1)
@@
 		)
 		(property "Footprint" "Resistor_THT:R_Axial_DIN0411_L9.9mm_D3.6mm_P15.24mm_Horizontal"
-			(at 208.28 90.678 90)
+			(at 208.534 87.884 90)
 			(effects
 				(font
@@
 			)
 		)
-		(property "Description" "Resistor"
+		(property "Description" "Resistor, US symbol"
 			(at 208.28 88.9 0)
 			(effects
@@
 	)
 	(symbol
-		(lib_id "Device:R")
+		(lib_id "Device:R_US")
 		(at 228.6 72.39 90)
 		(unit 1)
@@
 		)
 		(property "Footprint" "Resistor_THT:R_Axial_DIN0411_L9.9mm_D3.6mm_P15.24mm_Horizontal"
-			(at 228.6 74.168 90)
+			(at 228.854 71.374 90)
 			(effects
 				(font
@@
 			)
 		)
-		(property "Description" "Resistor"
+		(property "Description" "Resistor, US symbol"
 			(at 228.6 72.39 0)
 			(effects
@@
 	)
 	(symbol
-		(lib_id "Device:R")
+		(lib_id "Device:R_US")
 		(at 190.5 88.9 90)
 		(unit 1)
@@
 		)
 		(property "Footprint" "Resistor_THT:R_Axial_DIN0411_L9.9mm_D3.6mm_P15.24mm_Horizontal"
-			(at 190.5 90.678 90)
+			(at 190.754 87.884 90)
 			(effects
 				(font
@@
 			)
 		)
-		(property "Description" "Resistor"
+		(property "Description" "Resistor, US symbol"
 			(at 190.5 88.9 0)
 			(effects
@@
 			)
 		)
-		(property "Footprint" "Diode_THT:D_A-405_P5.08mm_Vertical_AnodeUp"
+		(property "Footprint" "Diode_THT:D_A-405_P7.62mm_Horizontal"
 			(at 86.36 38.1 0)
 			(effects
@@
 	)
 	(symbol
-		(lib_id "Device:R")
+		(lib_id "Device:R_US")
 		(at 95.25 34.29 90)
 		(unit 1)
@@
 		)
 		(property "Footprint" "Resistor_THT:R_Axial_DIN0411_L9.9mm_D3.6mm_P15.24mm_Horizontal"
-			(at 95.25 36.068 90)
+			(at 95.504 33.274 90)
 			(effects
 				(font
@@
 			)
 		)
-		(property "Description" "Resistor"
+		(property "Description" "Resistor, US symbol"
 			(at 95.25 34.29 0)
 			(effects
@@
 	)
 	(symbol
-		(lib_id "Device:R")
+		(lib_id "Device:R_US")
 		(at 238.76 72.39 90)
 		(unit 1)
@@
 		)
 		(property "Footprint" "Resistor_THT:R_Axial_DIN0411_L9.9mm_D3.6mm_P15.24mm_Horizontal"
-			(at 238.76 74.168 90)
+			(at 239.014 71.374 90)
 			(effects
 				(font
@@
 			)
 		)
-		(property "Description" "Resistor"
+		(property "Description" "Resistor, US symbol"
 			(at 238.76 72.39 0)
 			(effects
@@
 	)
 	(symbol
-		(lib_id "Device:R")
+		(lib_id "Device:R_US")
 		(at 111.76 82.55 0)
 		(unit 1)
@@
 		)
 		(property "Footprint" "Resistor_THT:R_Axial_DIN0411_L9.9mm_D3.6mm_P15.24mm_Horizontal"
-			(at 109.982 82.55 90)
+			(at 112.776 82.804 90)
 			(effects
 				(font
@@
 			)
 		)
-		(property "Description" "Resistor"
+		(property "Description" "Resistor, US symbol"
 			(at 111.76 82.55 0)
 			(effects
@@
 	)
 	(symbol
-		(lib_id "Device:R")
+		(lib_id "Device:R_US")
 		(at 218.44 72.39 90)
 		(unit 1)
@@
 		)
 		(property "Footprint" "Resistor_THT:R_Axial_DIN0411_L9.9mm_D3.6mm_P15.24mm_Horizontal"
-			(at 218.44 74.168 90)
+			(at 218.694 71.374 90)
 			(effects
 				(font
@@
 			)
 		)
-		(property "Description" "Resistor"
+		(property "Description" "Resistor, US symbol"
 			(at 218.44 72.39 0)
 			(effects
@@
 	)
 	(symbol
-		(lib_id "Device:R")
+		(lib_id "Device:R_US")
 		(at 63.5 34.29 90)
 		(unit 1)
@@
 		)
 		(property "Footprint" "Resistor_THT:R_Axial_DIN0411_L9.9mm_D3.6mm_P15.24mm_Horizontal"
-			(at 63.5 36.068 90)
+			(at 63.754 33.274 90)
 			(effects
 				(font
@@
 			)
 		)
-		(property "Description" "Resistor"
+		(property "Description" "Resistor, US symbol"
 			(at 63.5 34.29 0)
 			(effects
@@
 	)
 	(symbol
-		(lib_id "Device:R")
+		(lib_id "Device:R_US")
 		(at 110.49 22.86 0)
 		(unit 1)
@@
 		)
 		(property "Footprint" "Resistor_THT:R_Axial_DIN0411_L9.9mm_D3.6mm_P15.24mm_Horizontal"
-			(at 108.712 22.86 90)
+			(at 111.506 23.114 90)
 			(effects
 				(font
@@
 			)
 		)
-		(property "Description" "Resistor"
+		(property "Description" "Resistor, US symbol"
 			(at 110.49 22.86 0)
 			(effects
