File: hardware/KICAD Projects/BAJE SAE/Sensor Projects/Tachometer/Tachometerkicad.kicad_sch (KiCad schematic)
At the start: 25 parts, among them J1 Conn_01x02, J2 Conn_01x06, J3 Conn_01x02, J4 CAN to outer connector, Q1 NPN, U1 NE555P, U2 LM311

Commit message: fixed tach
Parts:
- UNIT_2: footprint BAJA SAE:HiLetgo CAN Bus -> 0_Baja_2025:CAN Bus (Feb 2025)
Other:
- moved on the sheet: UNIT_2
Changed lines of the file:
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@@
 	)
 	(no_connect
-		(at -160.02 149.86)
+		(at 200.66 138.43)
 	)
 	(no_connect
@@
 	(wire
 		(pts
-			(xy -125.73 152.4) (xy -127 152.4)
+			(xy 234.95 140.97) (xy 233.68 140.97)
 		)
 		(stroke
@@
 	(wire
 		(pts
-			(xy -143.51 170.18) (xy -143.51 168.91)
+			(xy 217.17 158.75) (xy 217.17 157.48)
 		)
 		(stroke
@@
 	(text "CAN Bus"
 		(exclude_from_sim no)
-		(at -168.91 130.81 0)
+		(at 191.77 119.38 0)
 		(effects
 			(font
@@
 	(global_label "SO"
 		(shape input)
-		(at -160.02 157.48 180)
+		(at 200.66 146.05 180)
 		(fields_autoplaced yes)
 		(effects
@@
 		)
 		(property "Intersheetrefs" "${INTERSHEET_REFS}"
-			(at -165.5452 157.48 0)
+			(at 195.1348 146.05 0)
 			(effects
 				(font
@@
 	(global_label "CS"
 		(shape input)
-		(at -160.02 160.02 180)
+		(at 200.66 148.59 180)
 		(fields_autoplaced yes)
 		(effects
@@
 		)
 		(property "Intersheetrefs" "${INTERSHEET_REFS}"
-			(at -165.4847 160.02 0)
+			(at 195.1953 148.59 0)
 			(effects
 				(font
@@
 	(global_label "High"
 		(shape input)
-		(at -125.73 152.4 0)
+		(at 234.95 140.97 0)
 		(fields_autoplaced yes)
 		(effects
@@
 		)
 		(property "Intersheetrefs" "${INTERSHEET_REFS}"
-			(at -118.5115 152.4 0)
+			(at 242.1685 140.97 0)
 			(effects
 				(font
@@
 	(global_label "SCK"
 		(shape input)
-		(at -160.02 152.4 180)
+		(at 200.66 140.97 180)
 		(fields_autoplaced yes)
 		(effects
@@
 		)
 		(property "Intersheetrefs" "${INTERSHEET_REFS}"
-			(at -166.7547 152.4 0)
+			(at 193.9253 140.97 0)
 			(effects
 				(font
@@
 	(global_label "SI"
 		(shape input)
-		(at -160.02 154.94 180)
+		(at 200.66 143.51 180)
 		(fields_autoplaced yes)
 		(effects
@@
 		)
 		(property "Intersheetrefs" "${INTERSHEET_REFS}"
-			(at -164.8195 154.94 0)
+			(at 195.8605 143.51 0)
 			(effects
 				(font
@@
 	(global_label "Low"
 		(shape input)
-		(at -127 157.48 0)
+		(at 233.68 146.05 0)
 		(fields_autoplaced yes)
 		(effects
@@
 		)
 		(property "Intersheetrefs" "${INTERSHEET_REFS}"
-			(at -120.5072 157.48 0)
+			(at 240.1728 146.05 0)
 			(effects
 				(font
@@
 	(global_label "+5V"
 		(shape input)
-		(at -143.51 140.97 90)
+		(at 217.17 129.54 90)
 		(fields_autoplaced yes)
 		(effects
@@
 		)
 		(property "Intersheetrefs" "${INTERSHEET_REFS}"
-			(at -143.51 134.1143 90)
+			(at 217.17 122.6843 90)
 			(effects
 				(font
@@
 	(symbol
 		(lib_id "0_Baja_Final:HiLetgo_CAN_BUS")
-		(at -143.51 154.94 0)
+		(at 217.17 143.51 0)
 		(unit 1)
 		(exclude_from_sim no)
@@
 		(fields_autoplaced yes)
 		(property "Reference" "UNIT_2"
-			(at -141.3159 138.43 0)
+			(at 219.3641 127 0)
 			(effects
 				(font
@@
 		)
 		(property "Value" "HiLetgo CAN Bus"
-			(at -141.3159 140.97 0)
+			(at 219.3641 129.54 0)
 			(effects
 				(font
@@
 			)
 		)
-		(property "Footprint" "BAJA SAE:HiLetgo CAN Bus"
-			(at -143.256 176.276 0)
+		(property "Footprint" "0_Baja_2025:CAN Bus (Feb 2025)"
+			(at 217.424 164.846 0)
 			(effects
 				(font
@@
 		)
 		(property "Datasheet" ""
-			(at -147.32 151.13 0)
+			(at 213.36 139.7 0)
 			(effects
 				(font
@@
 		)
 		(property "Description" ""
-			(at -147.32 151.13 0)
+			(at 213.36 139.7 0)
 			(effects
 				(font
@@
 	(symbol
 		(lib_id "Simulation_SPICE:0")
-		(at -143.51 170.18 0)
+		(at 217.17 158.75 0)
 		(unit 1)
 		(exclude_from_sim no)
@@
 		(fields_autoplaced yes)
 		(property "Reference" "#GND01"
-			(at -143.51 175.26 0)
+			(at 217.17 163.83 0)
 			(effects
 				(font
@@
 		)
 		(property "Value" "0"
-			(at -143.51 167.64 0)
+			(at 217.17 156.21 0)
 			(effects
 				(font
@@
 		)
 		(property "Footprint" ""
-			(at -143.51 170.18 0)
+			(at 217.17 158.75 0)
 			(effects
 				(font
@@
 		)
 		(property "Datasheet" "https://ngspice.sourceforge.io/docs/ngspice-html-manual/manual.xhtml#subsec_Circuit_elements__device"
-			(at -143.51 180.34 0)
+			(at 217.17 168.91 0)
 			(effects
 				(font
@@
 		)
 		(property "Description" "0V reference potential for simulation"
-			(at -143.51 177.8 0)
+			(at 217.17 166.37 0)
 			(effects
 				(font
