File: hardware/KICAD Projects/BAJE SAE/Main Computer/Main Computer.kicad_sch (KiCad schematic)
At the start: 6 parts, among them J1 Pi 5 GPIO HEADER, J2 Conn_01x06, J3 Conn_01x02, J4 CAN to outer connector, U1 NRF24L01_Breakout

Commit message: fnlsdnf
Parts:
- added RV1: R_Potentiometer_Trim, symbol Device:R_Potentiometer_Trim
Other:
- moved on the sheet: J1, J3, J4, U1
Changed lines of the file:
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@@
 	(wire
 		(pts
-			(xy 173.99 78.74) (xy 187.96 78.74)
+			(xy 163.83 76.2) (xy 171.45 76.2)
 		)
 		(stroke
@@
 	(wire
 		(pts
-			(xy 115.57 129.54) (xy 115.57 130.81)
+			(xy 177.8 121.92) (xy 177.8 123.19)
 		)
 		(stroke
@@
 	(wire
 		(pts
-			(xy 173.99 76.2) (xy 187.96 76.2)
+			(xy 163.83 73.66) (xy 171.45 73.66)
 		)
 		(stroke
@@
 	(wire
 		(pts
-			(xy 175.26 67.31) (xy 181.61 67.31)
+			(xy 165.1 64.77) (xy 171.45 64.77)
 		)
 		(stroke
@@
 	(wire
 		(pts
-			(xy 173.99 81.28) (xy 187.96 81.28)
+			(xy 163.83 78.74) (xy 171.45 78.74)
 		)
 		(stroke
@@
 	(wire
 		(pts
-			(xy 173.99 73.66) (xy 187.96 73.66)
+			(xy 163.83 71.12) (xy 171.45 71.12)
 		)
 		(stroke
@@
 	(wire
 		(pts
-			(xy 173.99 64.77) (xy 181.61 64.77)
+			(xy 163.83 62.23) (xy 171.45 62.23)
 		)
 		(stroke
@@
 	(rectangle
 		(start 154.0448 57.0384)
-		(end 219.71 86.7012)
+		(end 203.2 82.55)
+		(stroke
+			(width 0)
+			(type dot)
+		)
+		(fill
+			(type none)
+		)
+	)
+	(rectangle
+		(start 153.67 90.17)
+		(end 209.55 127)
 		(stroke
 			(width 0)
@@
 	(global_label "High"
 		(shape input)
-		(at 173.99 81.28 180)
+		(at 163.83 78.74 180)
 		(fields_autoplaced yes)
 		(effects
@@
 		)
 		(property "Intersheetrefs" "${INTERSHEET_REFS}"
-			(at 166.7715 81.28 0)
+			(at 156.6115 78.74 0)
 			(effects
 				(font
@@
 	(global_label "Low"
 		(shape input)
-		(at 173.99 73.66 180)
+		(at 163.83 71.12 180)
 		(fields_autoplaced yes)
 		(effects
@@
 		)
 		(property "Intersheetrefs" "${INTERSHEET_REFS}"
-			(at 167.4972 73.66 0)
+			(at 157.3372 71.12 0)
 			(effects
 				(font
@@
 	(global_label "+5v"
 		(shape output)
-		(at 173.99 64.77 180)
+		(at 163.83 62.23 180)
 		(fields_autoplaced yes)
 		(effects
@@
 		)
 		(property "Intersheetrefs" "${INTERSHEET_REFS}"
-			(at 167.2553 64.77 0)
+			(at 157.0953 62.23 0)
 			(effects
 				(font
@@
 	(global_label "SO"
 		(shape input)
-		(at 102.87 109.22 180)
+		(at 165.1 101.6 180)
 		(fields_autoplaced yes)
 		(effects
@@
 		)
 		(property "Intersheetrefs" "${INTERSHEET_REFS}"
-			(at 97.3448 109.22 0)
+			(at 159.5748 101.6 0)
 			(effects
 				(font
@@
 	(global_label "Low"
 		(shape input)
-		(at 173.99 78.74 180)
+		(at 163.83 76.2 180)
 		(fields_autoplaced yes)
 		(effects
@@
 		)
 		(property "Intersheetrefs" "${INTERSHEET_REFS}"
-			(at 167.4972 78.74 0)
+			(at 157.3372 76.2 0)
 			(effects
 				(font
@@
 	(global_label "High"
 		(shape input)
-		(at 173.99 76.2 180)
+		(at 163.83 73.66 180)
 		(fields_autoplaced yes)
 		(effects
@@
 		)
 		(property "Intersheetrefs" "${INTERSHEET_REFS}"
-			(at 166.7715 76.2 0)
+			(at 156.6115 73.66 0)
 			(effects
 				(font
@@
 	(global_label "SCK"
 		(shape input)
-		(at 102.87 111.76 180)
+		(at 165.1 104.14 180)
 		(fields_autoplaced yes)
 		(effects
@@
 		)
 		(property "Intersheetrefs" "${INTERSHEET_REFS}"
-			(at 96.1353 111.76 0)
+			(at 158.3653 104.14 0)
 			(effects
 				(font
@@
 	(global_label "GND"
 		(shape input)
-		(at 175.26 67.31 180)
+		(at 165.1 64.77 180)
 		(fields_autoplaced yes)
 		(effects
@@
 		)
 		(property "Intersheetrefs" "${INTERSHEET_REFS}"
-			(at 168.4043 67.31 0)
+			(at 158.2443 64.77 0)
 			(effects
 				(font
@@
 	(global_label "SI"
 		(shape input)
-		(at 102.87 106.68 180)
+		(at 165.1 99.06 180)
 		(fields_autoplaced yes)
 		(effects
@@
 		)
 		(property "Intersheetrefs" "${INTERSHEET_REFS}"
-			(at 98.0705 106.68 0)
+			(at 160.3005 99.06 0)
 			(effects
 				(font
@@
 	(symbol
 		(lib_id "Connector_Generic:Conn_01x02")
-		(at 186.69 64.77 0)
+		(at 176.53 62.23 0)
 		(unit 1)
 		(exclude_from_sim no)
@@
 		(fields_autoplaced yes)
 		(property "Reference" "J3"
-			(at 189.23 64.7699 0)
+			(at 179.07 62.2299 0)
 			(effects
 				(font
@@
 		)
 		(property "Value" "Conn_01x02"
-			(at 189.23 67.3099 0)
+			(at 179.07 64.7699 0)
 			(effects
 				(font
@@
 		)
 		(property "Footprint" "Connector_Wire:SolderWire-0.75sqmm_1x02_P4.8mm_D1.25mm_OD2.3mm"
-			(at 186.69 64.77 0)
+			(at 176.53 62.23 0)
 			(effects
 				(font
@@
 		)
 		(property "Datasheet" "~"
-			(at 186.69 64.77 0)
+			(at 176.53 62.23 0)
 			(effects
 				(font
@@
 		)
 		(property "Description" "Generic connector, single row, 01x02, script generated (kicad-library-utils/schlib/autogen/connector/)"
-			(at 186.69 64.77 0)
+			(at 176.53 62.23 0)
 			(effects
 				(font
@@
 	)
 	(symbol
+		(lib_id "Device:R_Potentiometer_Trim")
+		(at 123.19 106.68 0)
+		(unit 1)
+		(exclude_from_sim no)
+		(in_bom yes)
+		(on_board yes)
+		(dnp no)
+		(fields_autoplaced yes)
+		(property "Reference" "RV1"
+			(at 120.65 105.4099 0)
+			(effects
+				(font
+					(size 1.27 1.27)
+				)
+				(justify right)
+			)
+		)
+		(property "Value" "R_Potentiometer_Trim"
+			(at 120.65 107.9499 0)
+			(effects
+				(font
+					(size 1.27 1.27)
+				)
+				(justify right)
+			)
+		)
+		(property "Footprint" ""
+			(at 123.19 106.68 0)
+			(effects
+				(font
+					(size 1.27 1.27)
+				)
+				(hide yes)
+			)
+		)
+		(property "Datasheet" "~"
+			(at 123.19 106.68 0)
+			(effects
+				(font
+					(size 1.27 1.27)
+				)
+				(hide yes)
+			)
+		)
+		(property "Description" "Trim-potentiometer"
+			(at 123.19 106.68 0)
+			(effects
+				(font
+					(size 1.27 1.27)
+				)
+				(hide yes)
+			)
+		)
+		(pin "1"
+		)
+		(pin "2"
+		)
+		(pin "3"
+		)
+		(instances
+			(project ""
+				(path "/34ed1785-5142-4033-9af8-31e0ad1e0321"
+					(reference "RV1")
+					(unit 1)
+				)
+			)
+		)
+	)
+	(symbol
 		(lib_id "RF:NRF24L01_Breakout")
-		(at 115.57 114.3 0)
+		(at 177.8 106.68 0)
 		(unit 1)
 		(exclude_from_sim no)
@@
 		(fields_autoplaced yes)
 		(property "Reference" "U1"
-			(at 125.73 113.0299 0)
+			(at 187.96 105.4099 0)
 			(effects
 				(font
@@
 		)
 		(property "Value" "NRF24L01_Breakout"
-			(at 125.73 115.5699 0)
+			(at 187.96 107.9499 0)
 			(effects
 				(font
@@
 		)
 		(property "Footprint" "RF_Module:nRF24L01_Breakout"
-			(at 119.38 99.06 0)
+			(at 181.61 91.44 0)
 			(effects
 				(font
@@
 		)
 		(property "Datasheet" "http://www.nordicsemi.com/eng/content/download/2730/34105/file/nRF24L01_Product_Specification_v2_0.pdf"
-			(at 115.57 116.84 0)
+			(at 177.8 109.22 0)
 			(effects
 				(font
@@
 		)
 		(property "Description" "Ultra low power 2.4GHz RF Transceiver, Carrier PCB"
-			(at 115.57 114.3 0)
+			(at 177.8 106.68 0)
 			(effects
 				(font
@@
 	(symbol
 		(lib_id "Simulation_SPICE:0")
-		(at 115.57 130.81 0)
+		(at 177.8 123.19 0)
 		(unit 1)
 		(exclude_from_sim no)
@@
 		(fields_autoplaced yes)
 		(property "Reference" "#GND02"
-			(at 115.57 135.89 0)
+			(at 177.8 128.27 0)
 			(effects
 				(font
@@
 		)
 		(property "Value" "0"
-			(at 115.57 128.27 0)
+			(at 177.8 120.65 0)
 			(effects
 				(font
@@
 		)
 		(property "Footprint" ""
-			(at 115.57 130.81 0)
+			(at 177.8 123.19 0)
 			(effects
 				(font
@@
 		)
 		(property "Datasheet" "https://ngspice.sourceforge.io/docs/ngspice-html-manual/manual.xhtml#subsec_Circuit_elements__device"
-			(at 115.57 140.97 0)
+			(at 177.8 133.35 0)
 			(effects
 				(font
@@
 		)
 		(property "Description" "0V reference potential for simulation"
-			(at 115.57 138.43 0)
+			(at 177.8 130.81 0)
 			(effects
 				(font
@@
 	(symbol
 		(lib_id "Connector_Generic:Conn_01x04")
-		(at 193.04 76.2 0)
+		(at 176.53 73.66 0)
 		(unit 1)
 		(exclude_from_sim no)
@@
 		(fields_autoplaced yes)
 		(property "Reference" "J4"
-			(at 195.58 76.1999 0)
+			(at 179.07 73.6599 0)
 			(effects
 				(font
@@
 		)
 		(property "Value" "CAN to outer connector"
-			(at 195.58 78.7399 0)
+			(at 179.07 76.1999 0)
 			(effects
 				(font
@@
 		)
 		(property "Footprint" "Connector_Wire:SolderWire-0.1sqmm_1x04_P3.6mm_D0.4mm_OD1mm"
-			(at 193.04 76.2 0)
+			(at 176.53 73.66 0)
 			(effects
 				(font
@@
 		)
 		(property "Datasheet" "~"
-			(at 193.04 76.2 0)
+			(at 176.53 73.66 0)
 			(effects
 				(font
@@
 		)
 		(property "Description" "Generic connector, single row, 01x04, script generated (kicad-library-utils/schlib/autogen/connector/)"
-			(at 193.04 76.2 0)
+			(at 176.53 73.66 0)
 			(effects
 				(font

Commit message: Schematic cleanup for Main Computer
Parts:
- removed RV1: R_Potentiometer_Trim, symbol Device:R_Potentiometer_Trim
Connections:
- net +5v: now also U1.2 (VCC)
Other:
- note added: "GPIO Header (Custom Symbol)"
- note added: "Radio"
- moved on the sheet: J2, J3, J4, U1, UNIT_1

Commit message: finished pcbs yayyyy
Parts:
- removed U1: NRF24L01_Breakout, RF_Module:nRF24L01_Breakout, symbol RF:NRF24L01_Breakout
- added U2: E01-ML01DP5, 0_custom:Ebyte E01-ML01DP5, symbol 0_custom:Ebyte_E01-ML01DP5
Connections:
- net +5V is gone; now on net +5v: UNIT_1.7 (VCC)
- net 0: now also J1.9 (GND), U2.1 (GND)
- net CS: now also J1.24 (GPIO_8)
- net SCK: now also J1.23 (GPIO_11), U2.5 (SCK)
- net SI: now also J1.19 (GPIO_10), U2.6 (MOSI)
- net SO: now also J1.21 (GPIO_9), U2.7 (MISO)
- net INT: now reaches UNIT_1.1 (INT)
- net INT: now also J1.22 (GPIO_25)
- net 3V3: now reaches J1.1 (3V3)
- net 3V3: now also U2.2 (VCC)
- net CE: now reaches J1.15 (GPIO_22)
- net CE: now also U2.3 (CE)
- net CSN: now reaches J1.26 (GPIO_7)
- net CSN: now also U2.4 (CSN)
- no-connect marks 2 -> 4
