File: hardware/KICAD Projects/BAJE SAE/Main Computer/Main Computer.kicad_pcb (KiCad board)
At the start: 2 copper layers, 70.2 x 56.2 mm, 9 parts, among them J1 Pi 5 GPIO HEADER, J3 Conn_01x02, J4 CAN to outer connector, U1 NRF24L01_Breakout

Commit message: finished main computer rough outline
Parts:
- removed the REF** at (167.5, 70.0)
- removed the REF** at (107.2, 22.5)
- removed the REF** at (107.5, 70.0)
- removed the REF** at (167.5, 22.5)
- added REF**: MountingHole_3.2mm_M3, MountingHole:MountingHole_3.2mm_M3, F.Cu at (148.1, 91.3)
- added REF**: MountingHole_3.2mm_M3, MountingHole:MountingHole_3.2mm_M3, F.Cu at (99.6, 91.3)
- added REF**: MountingHole_3.2mm_M3, MountingHole:MountingHole_3.2mm_M3, F.Cu at (99.6, 149.8)
- added REF**: MountingHole_3.2mm_M3, MountingHole:MountingHole_3.2mm_M3, F.Cu at (148.1, 149.8)
- moved J3 107.4 mm to (100.0, 113.5)
- moved J4 107.2 mm to (100.0, 97.7)
- moved J1 79.7 mm to (146.9, 96.3), turned to 0 degrees
- moved U1 68.5 mm to (131.2, 131.1)
- moved UNIT_1 52.8 mm to (129.6, 100.6), turned to 180 degrees
Other:
- board size 70.2 x 56.2 mm -> 55.5 x 65.5 mm

Commit message: Update Main Computer.kicad_pcb
Parts:
- added G***: LOGO, BAJA SAE:Baja Logo, B.Cu at (122.9, 102.7)
- added G***: LOGO, BAJA SAE:Matthew Skate, B.Cu at (121.9, 128.3)

Commit message: Added 3D Model for IMU
Parts:
- removed the G*** at (121.9, 128.3)

Commit message: finished pcbs yayyyy
Parts:
- removed U1: NRF24L01_Breakout, RF_Module:nRF24L01_Breakout
- added U2: E01-ML01DP5, 0_custom:Ebyte E01-ML01DP5, F.Cu at (123.5, 116.5)
- J1: moved to B.Cu
- moved J3 10.0 mm to (100.3, 123.5)
- moved J4 10.0 mm to (100.3, 107.7)
- moved J1 2.38 mm to (149.3, 96.7), turned to 180 degrees
Connections:
- J1 pad 1: unconnected-(J1-3V3-Pad1) -> 3V3
- J1 pad 15: unconnected-(J1-GPIO_22-Pad15) -> CE
- J1 pad 19: unconnected-(J1-GPIO_10-Pad19) -> SI
- J1 pad 21: unconnected-(J1-GPIO_9-Pad21) -> SO
- J1 pad 22: unconnected-(J1-GPIO_25-Pad22) -> INT
- J1 pad 23: unconnected-(J1-GPIO_11-Pad23) -> SCK
- J1 pad 24: unconnected-(J1-GPIO_8-Pad24) -> CS
- J1 pad 26: unconnected-(J1-GPIO_7-Pad26) -> CSN
- J1 pad 9: unconnected-(J1-GND-Pad9) -> GND
- UNIT_1 pad 1: unconnected-(UNIT_1-INT-Pad1) -> INT
- UNIT_1 pad 7: +5V -> +5v
Routing:
- net GND: track 0.00 -> 129.2 mm
- net 3V3: track 0.00 -> 67.1 mm
- net +5v: track 0.00 -> 61.2 mm
- net SO: track 0.00 -> 54.5 mm, vias 0 -> 2
- net SCK: track 0.00 -> 53.1 mm
- net SI: track 0.00 -> 44.9 mm, vias 0 -> 1
- net CS: track 0.00 -> 31.5 mm, vias 0 -> 1
- net CE: track 0.00 -> 27.3 mm, vias 0 -> 2
- net CSN: track 0.00 -> 24.0 mm
- net Low: track 0.00 -> 21.3 mm
- net High: track 0.00 -> 19.4 mm
- net INT: track 0.00 -> 17.6 mm
Other:
- board text added: "+"
- board text added: "-"
- board text added: "Designed by Connor & Matthew Larson in Tucson, AZ"
- board text added: "H"
- board text added: "L"
- board text added: "MAIN COMPUTER"
- board text removed: "penis"

Commit message: temp sense worky now
Other:
- board text added: "This side up Matthew"
Changed lines of the file:
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@@
+		)
+	)
+	(gr_text "This side up Matthew"
+		(at 97.34 138.24 0)
+		(layer "F.SilkS")
+		(effects
+			(font
+				(size 1 1)
+				(thickness 0.15)
+			)
+			(justify left bottom)
 		)
 	)

Commit message: hardware updates
Routing:
- net 3V3: track 67.1 -> 74.0 mm, vias 0 -> 1
- net GND: track 129.2 -> 127.7 mm
Other:
- board text added: "REV 2"
