File: hardware/KICAD Projects/BAJE SAE/Sensor Projects/Speedometer/Speedometer.kicad_sch (KiCad schematic)
At the start: 31 parts, among them J1 Conn_01x02, J2 Conn_01x06, J3 Conn_01x02, J4 CAN to outer connector, Q1 NPN, U1 NE555P, U2 LM311

Commit message: Edit page settings for Speedometer.
Other:
- company: (none) -> University of Arizona
- title: (none) -> Baja Speedometer 
- moved on the sheet: C5, C6, D3, J1, R9
Changed lines of the file:
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@@
 	(generator_version "8.0")
 	(paper "A4")
+	(title_block
+		(title "Baja Speedometer ")
+		(date "2025-02-02")
+		(rev "v1")
+		(company "University of Arizona")
+		(comment 1 "Jack Tanner")
+	)
 	(junction
 		(at 201.93 38.1)
@@
 	(wire
 		(pts
-			(xy 31.75 54.61) (xy 27.94 54.61)
+			(xy 30.48 26.67) (xy 26.67 26.67)
 		)
 		(stroke
@@
 	(wire
 		(pts
-			(xy 27.94 57.15) (xy 35.56 57.15)
+			(xy 26.67 29.21) (xy 34.29 29.21)
 		)
 		(stroke
@@
 	(global_label "Possitive"
 		(shape input)
-		(at 31.75 54.61 0)
+		(at 30.48 26.67 0)
 		(fields_autoplaced yes)
 		(effects
@@
 		)
 		(property "Intersheetrefs" "${INTERSHEET_REFS}"
-			(at 43.2019 54.61 0)
+			(at 41.9319 26.67 0)
 			(effects
 				(font
@@
 	(global_label "GND"
 		(shape input)
-		(at 35.56 57.15 0)
+		(at 34.29 29.21 0)
 		(fields_autoplaced yes)
 		(effects
@@
 		)
 		(property "Intersheetrefs" "${INTERSHEET_REFS}"
-			(at 42.4157 57.15 0)
+			(at 41.1457 29.21 0)
 			(effects
 				(font
@@
 	(symbol
 		(lib_id "Device:R_US")
-		(at 95.25 34.29 0)
+		(at 100.33 26.67 0)
 		(unit 1)
 		(exclude_from_sim no)
@@
 		(fields_autoplaced yes)
 		(property "Reference" "R9"
-			(at 97.79 33.0199 0)
+			(at 102.87 25.3999 0)
 			(effects
 				(font
@@
 		)
 		(property "Value" "R_US"
-			(at 97.79 35.5599 0)
+			(at 102.87 27.9399 0)
 			(effects
 				(font
@@
 		)
 		(property "Footprint" ""
-			(at 96.266 34.544 90)
+			(at 101.346 26.924 90)
 			(effects
 				(font
@@
 		)
 		(property "Datasheet" "~"
-			(at 95.25 34.29 0)
+			(at 100.33 26.67 0)
 			(effects
 				(font
@@
 		)
 		(property "Description" "Resistor, US symbol"
-			(at 95.25 34.29 0)
+			(at 100.33 26.67 0)
 			(effects
 				(font
@@
 	(symbol
 		(lib_id "Device:C_Polarized_US")
-		(at 60.96 55.88 0)
+		(at 30.48 66.04 0)
 		(unit 1)
 		(exclude_from_sim no)
@@
 		(on_board yes)
 		(dnp no)
-		(fields_autoplaced yes)
 		(property "Reference" "C5"
-			(at 64.77 53.9749 0)
+			(at 34.29 64.1349 0)
 			(effects
 				(font
@@
 		)
 		(property "Value" "10uF"
-			(at 64.77 56.5149 0)
+			(at 34.29 66.6749 0)
 			(effects
 				(font
@@
 		)
 		(property "Footprint" ""
-			(at 60.96 55.88 0)
+			(at 30.48 66.04 0)
 			(effects
 				(font
@@
 		)
 		(property "Datasheet" "~"
-			(at 60.96 55.88 0)
+			(at 30.48 66.04 0)
 			(effects
 				(font
@@
 		)
 		(property "Description" "Polarized capacitor, US symbol"
-			(at 60.96 55.88 0)
+			(at 30.48 66.04 0)
 			(effects
 				(font
@@
 	(symbol
 		(lib_id "Connector_Generic:Conn_01x02")
-		(at 22.86 57.15 180)
+		(at 21.59 29.21 180)
 		(unit 1)
 		(exclude_from_sim no)
@@
 		(fields_autoplaced yes)
 		(property "Reference" "J1"
-			(at 22.86 48.26 0)
+			(at 21.59 20.32 0)
 			(effects
 				(font
@@
 		)
 		(property "Value" "Conn_01x02"
-			(at 22.86 50.8 0)
+			(at 21.59 22.86 0)
 			(effects
 				(font
@@
 		)
 		(property "Footprint" "Connector_Wire:SolderWire-0.75sqmm_1x02_P4.8mm_D1.25mm_OD2.3mm"
-			(at 22.86 57.15 0)
+			(at 21.59 29.21 0)
 			(effects
 				(font
@@
 		)
 		(property "Datasheet" "~"
-			(at 22.86 57.15 0)
+			(at 21.59 29.21 0)
 			(effects
 				(font
@@
 		)
 		(property "Description" "Generic connector, single row, 01x02, script generated (kicad-library-utils/schlib/autogen/connector/)"
-			(at 22.86 57.15 0)
+			(at 21.59 29.21 0)
 			(effects
 				(font
@@
 	(symbol
 		(lib_id "Device:LED")
-		(at 88.9 30.48 90)
+		(at 88.9 25.4 90)
 		(unit 1)
 		(exclude_from_sim no)
@@
 		(fields_autoplaced yes)
 		(property "Reference" "D3"
-			(at 92.71 30.7974 90)
+			(at 92.71 25.7174 90)
 			(effects
 				(font
@@
 		)
 		(property "Value" "LED"
-			(at 92.71 33.3374 90)
+			(at 92.71 28.2574 90)
 			(effects
 				(font
@@
 		)
 		(property "Footprint" ""
-			(at 88.9 30.48 0)
+			(at 88.9 25.4 0)
 			(effects
 				(font
@@
 		)
 		(property "Datasheet" "~"
-			(at 88.9 30.48 0)
+			(at 88.9 25.4 0)
 			(effects
 				(font
@@
 		)
 		(property "Description" "Light emitting diode"
-			(at 88.9 30.48 0)
+			(at 88.9 25.4 0)
 			(effects
 				(font
@@
 	(symbol
 		(lib_id "Device:C_Polarized_US")
-		(at 72.39 55.88 0)
+		(at 41.91 66.04 0)
 		(unit 1)
 		(exclude_from_sim no)
@@
 		(dnp no)
 		(property "Reference" "C6"
-			(at 76.2 53.086 0)
+			(at 45.72 63.246 0)
 			(effects
 				(font
@@
 		)
 		(property "Value" "10nF"
-			(at 76.2 56.5149 0)
+			(at 45.72 66.6749 0)
 			(effects
 				(font
@@
 		)
 		(property "Footprint" ""
-			(at 72.39 55.88 0)
+			(at 41.91 66.04 0)
 			(effects
 				(font
@@
 		)
 		(property "Datasheet" "~"
-			(at 72.39 55.88 0)
+			(at 41.91 66.04 0)
 			(effects
 				(font
@@
 		)
 		(property "Description" "Polarized capacitor, US symbol"
-			(at 72.39 55.88 0)
+			(at 41.91 66.04 0)
 			(effects
 				(font

Commit message: Add symbol for A3144 Hall Effect sensor, add to exist DT library file.
Parts:
- added U3: A3144, symbol DT13-6P:A3144
Changed lines of the file:
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@@
+	)
+	(symbol
+		(lib_id "DT13-6P:A3144")
+		(at 63.5 62.23 0)
+		(unit 1)
+		(exclude_from_sim no)
+		(in_bom yes)
+		(on_board yes)
+		(dnp no)
+		(fields_autoplaced yes)
+		(property "Reference" "U3"
+			(at 57.15 66.0399 0)
+			(effects
+				(font
+					(size 1.27 1.27)
+				)
+				(justify right)
+			)
+		)
+		(property "Value" "A3144"
+			(at 57.15 68.5799 0)
+			(effects
+				(font
+					(size 1.27 1.27)
+				)
+				(justify right)
+			)
+		)
+		(property "Footprint" ""
+			(at 63.5 62.23 0)
+			(effects
+				(font
+					(size 1.27 1.27)
+				)
+				(hide yes)
+			)
+		)
+		(property "Datasheet" "https://www.elecrow.com/download/A3141-2-3-4-Datasheet.pdf?srsltid=AfmBOorrsjBY2AmYjT58rnK_N69ih2Y2Co9rSXOYxEPPaNMpLUfjbq4q"
+			(at 63.5 62.23 0)
+			(effects
+				(font
+					(size 1.27 1.27)
+				)
+				(hide yes)
+			)
+		)
+		(property "Description" "A3144 Hall Effect Sensor switches from floating to GND when interacting with magnet."
+			(at 63.5 62.23 0)
+			(effects
+				(font
+					(size 1.27 1.27)
+				)
+				(hide yes)
+			)
+		)
+		(pin "3"
+		)
+		(pin "2"
+		)
+		(pin "1"
+		)
+		(instances
+			(project ""
+				(path "/d32b6a5f-c7f0-4229-a4f9-b1dde9133fa5"
+					(reference "U3")
+					(unit 1)
+				)
+			)
+		)
 	)
 	(symbol

Commit message: Add all symbols and wires for speedometer circuit.
Parts:
- removed C1, C2: 10u, Capacitor_THT:CP_Radial_D5.0mm_P2.50mm, symbol Device:C_Polarized
- removed D1: ~, Diode_THT:D_A-405_P7.62mm_Horizontal, symbol Device:D_Zener
- removed Q1: NPN, Package_TO_SOT_THT:TO-92L_Inline, symbol Simulation_SPICE:NPN
- removed R1: 10, Resistor_THT:R_Axial_DIN0411_L9.9mm_D3.6mm_P15.24mm_Horizontal, symbol Device:R_US
- removed R10: 10k, Resistor_THT:R_Axial_DIN0411_L9.9mm_D3.6mm_P15.24mm_Horizontal, symbol Device:R_US
- removed R2: 470, Resistor_THT:R_Axial_DIN0411_L9.9mm_D3.6mm_P15.24mm_Horizontal, symbol Device:R_US
- removed R7: 100k, Resistor_THT:R_Axial_DIN0411_L9.9mm_D3.6mm_P15.24mm_Horizontal, symbol Device:R_US
- removed R8: 10k, symbol Device:R_US
- removed U1: NE555P, Package_DIP:DIP-8_W7.62mm, symbol Timer:NE555P
- removed U2: LM311, Package_DIP:DIP-8_W7.62mm, symbol Comparator:LM311
- removed VR1: 3362P-1-103, 3362P-1-103:TRIM_3362P-1-103, symbol 0_3362P-1-103:3362P-1-103
- added C5: 220n, symbol Device:C_Polarized_US
- added C6, C7: 10µ, symbol Device:C_Polarized_US
- added R5: 22k, symbol Device:R_US
- added U2: NE555P, Package_DIP:DIP-8_W7.62mm, symbol Timer:NE555P
- C1: renamed from C5; value 10uF -> 10µ
- C2: renamed from C6; value 10nF -> 10n
- C3: value .22u -> 10n; footprint Capacitor_THT:CP_Radial_D5.0mm_P2.50mm -> (none)
- C4: value C -> 10n; footprint Capacitor_THT:C_Disc_D6.0mm_W4.4mm_P5.00mm -> (none)
- D2: footprint Diode_THT:D_A-405_P7.62mm_Horizontal -> (none)
- R1: renamed from R9; value R_US -> 300
- R2: renamed from R12; value R_US -> 10k
- R3: value 1k -> 10k; footprint Resistor_THT:R_Axial_DIN0411_L9.9mm_D3.6mm_P15.24mm_Horizontal -> (none)
- R4: value 100k -> 10k; footprint Resistor_THT:R_Axial_DIN0411_L9.9mm_D3.6mm_P15.24mm_Horizontal -> (none)
- R6: value 100k -> 33k; footprint Resistor_THT:R_Axial_DIN0411_L9.9mm_D3.6mm_P15.24mm_Horizontal -> (none)
- renumbered D3 to D1, J2 to J1, J3 to J2, J4 to J3, J1 to J4, R5 to R7, R11 to R8, U3 to U1, UNIT_2 to UNIT_1, UNIT_1 to UNIT_2
Connections:
- net Comparator input is gone; now on an unnamed net: R3.2
- net Possitive is gone; now on net 5V: J4.2 (Pin_2)
- net +5V: no longer UNIT_2.27 (+5V)
- net +5v: no longer R3.1
- net 0: no longer C3.1, C4.2, D2.2 (A), J2.2 (Pin_2), J4.1 (Pin_1), UNIT_2.29 (COM/GND), UNIT_2.4 (COM/GND)
- net at D2.1 (K): now also C3.2
- net at R1.1: now also D1.1 (K)
- net at R1.2: now also C3.1, R2.2, U1.3 (OUT)
- net at R7.2, R8.1: now also C6.1
- net 5V: now reaches C1.1
- net 5V: now also C2.1, D1.2 (A), R2.1, R3.1, R4.1, U1.1 (Vcc), UNIT_2.27 (+5V), R5.1, U2.4 (R), U2.8 (VCC)
- net GND: now reaches C1.2
- net GND: now also C2.2, C4.1, J2.2 (Pin_2), J4.1 (Pin_1), U1.2 (GND), UNIT_2.29 (COM/GND), UNIT_2.4 (COM/GND), C5.2, C6.2, C7.2, U2.1 (GND)
- net at R4.2: now also D2.2 (A), U2.2 (TR); no longer R6.1
- net at R6.2: now also C5.1, U2.6 (THR), U2.7 (DIS)
- net +3V renamed 3.3V
- net 555 output renamed NE555_Out
- net NE555_Out: now also U2.3 (Q)
- net arduino input renamed Nano_Input
- net Nano_Input: now also C7.1
- new net: C4.2, U2.5 (CV)
- new net: R5.2, R6.1
- no-connect marks 23 -> 21
Other:
- note added: "Can Connector Pins"
- note added: "Car Battery"
- note added: "Cascading Low-Pass Filters"
- note added: "Differentiator"
- note added: "Hall Effect Sensor; Pullup Resistor"
- note added: "NE555 Timer; Pulse Generator"
- note added: "Rectifier"
- note removed: "Nano socketed with HWS16130 http://www.peconnectors.com/sockets-sip-machined/ hws16130/?utm_source=googleads&vt_keyword=&gad_source= 1&gbraid=0AAAAAD-J6wRIeL1mScc81doEXt4u-oFxN&gclid=Cj0KC QiA4rK8BhD7ARIsAFe5LXJCXX4yoeMSgdYYrUZ8CYCOGg6YWjx-KireWWb9vicOqA-PgvhT3uIaAs8kEALw_wcB"
- note removed: "Socket"
- moved on the sheet: D1, J3, J4, R1, R2, R7, R8, U1, UNIT_1

Commit message: Add footprint for Hall Effect sensor, and assign all footprints.
Parts:
- C1, C6, C7: footprint (none) -> Capacitor_THT:CP_Radial_D4.0mm_P2.00mm
- C2, C3, C4: footprint (none) -> Capacitor_THT:C_Disc_D3.8mm_W2.6mm_P2.50mm
- C5: footprint (none) -> Capacitor_THT:CP_Radial_D6.3mm_P2.50mm
- D1: footprint (none) -> LED_THT:LED_D4.0mm
- D2: footprint (none) -> Diode_THT:D_DO-41_SOD81_P7.62mm_Horizontal
- R1, R2, R3, R4, R5, R6: footprint (none) -> Resistor_THT:R_Axial_DIN0207_L6.3mm_D2.5mm_P10.16mm_Horizontal
- U1: footprint (none) -> SS49E:TO92127P460H470-3
Changed lines of the file:
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@@
 			)
 		)
-		(property "Footprint" ""
+		(property "Footprint" "Resistor_THT:R_Axial_DIN0207_L6.3mm_D2.5mm_P10.16mm_Horizontal"
 			(at 83.566 57.404 90)
 			(effects
@@
 			)
 		)
-		(property "Footprint" ""
+		(property "Footprint" "Capacitor_THT:CP_Radial_D4.0mm_P2.00mm"
 			(at 30.48 66.04 0)
 			(effects
@@
 			)
 		)
-		(property "Footprint" ""
+		(property "Footprint" "Capacitor_THT:CP_Radial_D6.3mm_P2.50mm"
 			(at 191.77 81.28 0)
 			(effects
@@
 			)
 		)
-		(property "Footprint" ""
+		(property "Footprint" "Capacitor_THT:C_Disc_D3.8mm_W2.6mm_P2.50mm"
 			(at 150.1648 77.47 0)
 			(effects
@@
 			)
 		)
-		(property "Footprint" ""
+		(property "Footprint" "Capacitor_THT:CP_Radial_D4.0mm_P2.00mm"
 			(at 204.47 115.57 0)
 			(effects
@@
 			)
 		)
-		(property "Footprint" ""
+		(property "Footprint" "SS49E:TO92127P460H470-3"
 			(at 63.5 60.96 0)
 			(effects
@@
 			)
 		)
-		(property "Footprint" ""
+		(property "Footprint" "Resistor_THT:R_Axial_DIN0207_L6.3mm_D2.5mm_P10.16mm_Horizontal"
 			(at 114.046 49.784 90)
 			(effects
@@
 			)
 		)
-		(property "Footprint" ""
+		(property "Footprint" "Diode_THT:D_DO-41_SOD81_P7.62mm_Horizontal"
 			(at 133.35 66.04 0)
 			(effects
@@
 			)
 		)
-		(property "Footprint" ""
+		(property "Footprint" "Capacitor_THT:CP_Radial_D4.0mm_P2.00mm"
 			(at 232.41 115.57 0)
 			(effects
@@
 			)
 		)
-		(property "Footprint" ""
+		(property "Footprint" "LED_THT:LED_D4.0mm"
 			(at 82.55 49.53 0)
 			(effects
@@
 			)
 		)
-		(property "Footprint" ""
+		(property "Footprint" "Resistor_THT:R_Axial_DIN0207_L6.3mm_D2.5mm_P10.16mm_Horizontal"
 			(at 192.786 61.214 90)
 			(effects
@@
 			)
 		)
-		(property "Footprint" ""
+		(property "Footprint" "Capacitor_THT:C_Disc_D3.8mm_W2.6mm_P2.50mm"
 			(at 110.49 65.0748 0)
 			(effects
@@
 			)
 		)
-		(property "Footprint" ""
+		(property "Footprint" "Resistor_THT:R_Axial_DIN0207_L6.3mm_D2.5mm_P10.16mm_Horizontal"
 			(at 140.716 51.054 90)
 			(effects
@@
 			)
 		)
-		(property "Footprint" ""
+		(property "Footprint" "Capacitor_THT:C_Disc_D3.8mm_W2.6mm_P2.50mm"
 			(at 41.91 66.04 0)
 			(effects
@@
 			)
 		)
-		(property "Footprint" ""
+		(property "Footprint" "Resistor_THT:R_Axial_DIN0207_L6.3mm_D2.5mm_P10.16mm_Horizontal"
 			(at 192.786 51.054 90)
 			(effects
@@
 			)
 		)
-		(property "Footprint" ""
+		(property "Footprint" "Resistor_THT:R_Axial_DIN0207_L6.3mm_D2.5mm_P10.16mm_Horizontal"
 			(at 94.996 53.594 90)
 			(effects

Commit message: Add mounting holes with footprints to schematic.
Parts:
- added H1, H2, H3, H4: MountingHole, MountingHole:MountingHole_3.2mm_M3, symbol Mechanical:MountingHole
Other:
- note added: "Mounting Holes"
