File: hardware/KICAD Projects/BAJE SAE/Sensor Projects/Speedometer/Speedometer.kicad_sch (KiCad schematic)
At the start: 29 parts, among them J1 Conn_01x06, J2 Conn_01x02, J3 CAN to outer connector, J4 Conn_01x02, U1 A3144, U2 NE555P

Commit message: Change NANO footprint and add all net labels.
Parts:
- UNIT_2: footprint BAJA SAE:SHIELD_ARDUINO_NANO -> Module:Arduino_Nano
Connections:
- net DIS/THR renamed DIS_THR
- net Nano_Input renamed Filter2
Changed lines of the file:
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@@
 		)
 	)
-	(label "DIS{slash}THR"
+	(label "DIS_THR"
 		(at 191.77 73.66 0)
 		(effects
@@
 			)
 			(justify left bottom)
+		)
+	)
+	(label "Nano_Input"
+		(at 85.09 161.29 270)
+		(effects
+			(font
+				(size 1.27 1.27)
+			)
+			(justify right bottom)
 		)
 	)
@@
 		(property "Intersheetrefs" "${INTERSHEET_REFS}"
 			(at 63.5 93.2157 90)
-			(effects
-				(font
-					(size 1.27 1.27)
-				)
-				(justify right)
-				(hide yes)
-			)
-		)
-	)
-	(global_label "Nano_Input"
-		(shape input)
-		(at 85.09 161.29 270)
-		(fields_autoplaced yes)
-		(effects
-			(font
-				(size 1.27 1.27)
-			)
-			(justify right)
-		)
-		(property "Intersheetrefs" "${INTERSHEET_REFS}"
-			(at 85.09 174.7978 90)
 			(effects
 				(font
@@
 			)
 		)
-		(property "Footprint" "BAJA SAE:SHIELD_ARDUINO_NANO"
+		(property "Footprint" "Module:Arduino_Nano"
 			(at 108.712 194.056 0)
 			(effects

Commit message: Add CAN, Change 5V to Power Inut.
Parts:
- removed J1: Conn_01x06, symbol Connector_Generic:Conn_01x06
- removed J2: Conn_01x02, Connector_Wire:SolderWire-0.75sqmm_1x02_P4.8mm_D1.25mm_OD2.3mm, symbol Connector_Generic:Conn_01x02
- UNIT_1: footprint BAJA SAE:HiLetgo CAN Bus -> SS49E:CAN_MCP2515
Connections:
- net 0 is gone; now on net GND: UNIT_1.6 (GND)
- net 5V is gone; now on net +5V: C1.1, C2.1, D1.2 (A), J4.2 (Pin_2), R2.1, R3.1, R4.1, R5.1, U1.1 (Vcc), U2.4 (R), U2.8 (VCC), UNIT_2.27 (+5V)
- net CS: now also UNIT_2.13 (D10)
- net 3.3V: no longer names the net of UNIT_2.17 (3V3)
- net Filter2 renamed Nano_Input
- net SCL: no longer names the net of UNIT_2.24 (A5)
- net SDA: no longer names the net of UNIT_2.23 (A4)
- no-connect marks 21 -> 23
Other:
- note removed: "+5v"
- note removed: "Connector Pinout"
- note removed: "GND"
- note removed: "High"
- note removed: "I/O"
- note removed: "Low"
- moved on the sheet: H1, H2, H3, H4, J3, UNIT_1, UNIT_2

Commit message: Add power flags; ERC Checked.
Changed lines of the file:
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@@
 	)
 	(junction
+		(at 82.55 40.64)
+		(diameter 0)
+		(color 0 0 0 0)
+	)
+	(junction
 		(at 41.91 78.74)
 		(diameter 0)
@@
 	(wire
 		(pts
+			(xy 82.55 40.64) (xy 82.55 45.72)
+		)
+		(stroke
+			(width 0)
+			(type default)
+		)
+	)
+	(wire
+		(pts
 			(xy 184.15 71.12) (xy 191.77 71.12)
 		)
@@
 	(wire
 		(pts
-			(xy 82.55 34.29) (xy 82.55 45.72)
+			(xy 82.55 34.29) (xy 82.55 40.64)
 		)
 		(stroke
@@
 	)
 	(symbol
+		(lib_id "power:PWR_FLAG")
+		(at 63.5 78.74 270)
+		(unit 1)
+		(exclude_from_sim no)
+		(in_bom yes)
+		(on_board yes)
+		(dnp no)
+		(fields_autoplaced yes)
+		(property "Reference" "#FLG02"
+			(at 65.405 78.74 0)
+			(effects
+				(font
+					(size 1.27 1.27)
+				)
+				(hide yes)
+			)
+		)
+		(property "Value" "PWR_FLAG"
+			(at 67.31 78.7399 90)
+			(effects
+				(font
+					(size 1.27 1.27)
+				)
+				(justify left)
+			)
+		)
+		(property "Footprint" ""
+			(at 63.5 78.74 0)
+			(effects
+				(font
+					(size 1.27 1.27)
+				)
+				(hide yes)
+			)
+		)
+		(property "Datasheet" "~"
+			(at 63.5 78.74 0)
+			(effects
+				(font
+					(size 1.27 1.27)
+				)
+				(hide yes)
+			)
+		)
+		(property "Description" "Special symbol for telling ERC where power comes from"
+			(at 63.5 78.74 0)
+			(effects
+				(font
+					(size 1.27 1.27)
+				)
+				(hide yes)
+			)
+		)
+		(pin "1"
+		)
+		(instances
+			(project "Speedometer"
+				(path "/d32b6a5f-c7f0-4229-a4f9-b1dde9133fa5"
+					(reference "#FLG02")
+					(unit 1)
+				)
+			)
+		)
+	)
+	(symbol
 		(lib_id "Timer:NE555P")
 		(at 171.45 71.12 0)
@@
 					(unit 1)
 				)
+			)
+		)
+	)
+	(symbol
+		(lib_id "power:PWR_FLAG")
+		(at 82.55 40.64 90)
+		(unit 1)
+		(exclude_from_sim no)
+		(in_bom yes)
+		(on_board yes)
+		(dnp no)
+		(fields_autoplaced yes)
+		(property "Reference" "#FLG01"
+			(at 80.645 40.64 0)
+			(effects
+				(font
+					(size 1.27 1.27)
+				)
+				(hide yes)
+			)
+		)
+		(property "Value" "PWR_FLAG"
+			(at 78.74 40.6399 90)
+			(effects
+				(font
+					(size 1.27 1.27)
+				)
+				(justify left)
+			)
+		)
+		(property "Footprint" ""
+			(at 82.55 40.64 0)
+			(effects
+				(font
+					(size 1.27 1.27)
+				)
+				(hide yes)
+			)
+		)
+		(property "Datasheet" "~"
+			(at 82.55 40.64 0)
+			(effects
+				(font
+					(size 1.27 1.27)
+				)
+				(hide yes)
+			)
+		)
+		(property "Description" "Special symbol for telling ERC where power comes from"
+			(at 82.55 40.64 0)
+			(effects
+				(font
+					(size 1.27 1.27)
+				)
+				(hide yes)
+			)
+		)
+		(pin "1"
+		)
+		(instances
+			(project ""
+				(path "/d32b6a5f-c7f0-4229-a4f9-b1dde9133fa5"
+					(reference "#FLG01")
+					(unit 1)
+				)

Commit message: Add L/H connectors and adjust footprints.
Parts:
- removed J3: CAN to outer connector, Connector_Wire:SolderWire-0.1sqmm_1x04_P3.6mm_D0.4mm_OD1mm, symbol Connector_Generic:Conn_01x04
- removed J4: Conn_01x02, Connector_Wire:SolderWire-0.75sqmm_1x02_P4.8mm_D1.25mm_OD2.3mm, symbol Connector_Generic:Conn_01x02
- added J1: Conn_01x02, Connector_Wire:SolderWire-0.75sqmm_1x02_P4.8mm_D1.25mm_OD2.3mm, symbol Connector_Generic:Conn_01x02
- added J2: CAN to outer connector, Connector_Wire:SolderWire-0.1sqmm_1x04_P3.6mm_D0.4mm_OD1mm, symbol Connector_Generic:Conn_01x04
- R7, R8: footprint Resistor_THT:R_Axial_DIN0411_L9.9mm_D3.6mm_P15.24mm_Horizontal -> Resistor_THT:R_Axial_DIN0207_L6.3mm_D2.5mm_P10.16mm_Horizontal
- U1: footprint SS49E:TO92127P460H470-3 -> Connector_PinHeader_2.54mm:PinHeader_1x03_P2.54mm_Vertical
- UNIT_1: footprint SS49E:CAN_MCP2515 -> 0_Baja_Final:Can Bus (Correct)
Connections:
- net +5V: now also J1.1 (Pin_1)
- net GND: now also J1.2 (Pin_2)
- net High: now also J2.2 (Pin_2), J2.4 (Pin_4)
- net Low: now also J2.1 (Pin_1), J2.3 (Pin_3)
Other:
- note added: "I/O"
- note removed: "Can Connector Pins"
- note removed: "Car Battery"
- moved on the sheet: H1, H2, H3, H4

Commit message: New Gerber files with corrected pins, Vin, and dimensions.
Parts:
- UNIT_1: footprint 0_Baja_Final:Can Bus (Correct) -> 0_Baja_Final:Jack_CanBus
Connections:
- net +5V: now also UNIT_2.30 (VIN)
- no-connect marks 23 -> 22
Changed lines of the file:
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@@
-	)
-	(no_connect
-		(at 106.68 184.15)
 	)
 	(no_connect
@@
 				)
 				(justify left)
+				(hide yes)
+			)
+		)
+	)
+	(global_label "+5V"
+		(shape output)
+		(at 106.68 184.15 270)
+		(fields_autoplaced yes)
+		(effects
+			(font
+				(size 1.27 1.27)
+			)
+			(justify right)
+		)
+		(property "Intersheetrefs" "${INTERSHEET_REFS}"
+			(at 106.68 191.0057 90)
+			(effects
+				(font
+					(size 1.27 1.27)
+				)
+				(justify right)
 				(hide yes)
 			)
@@
 			)
 		)
-		(property "Footprint" "0_Baja_Final:Can Bus (Correct)"
+		(property "Footprint" "0_Baja_Final:Jack_CanBus"
 			(at 45.974 159.766 0)
 			(effects

Commit message: Add all speedometer hall effect sensors and CAD file.
Parts:
- added C10, C12, C15, C16, C7, C9: 10µ, Capacitor_THT:CP_Radial_D4.0mm_P2.00mm, symbol Device:C_Polarized_US
- added C11, C13: 10n, Capacitor_THT:C_Disc_D3.8mm_W2.6mm_P2.50mm, symbol Device:C_Polarized_US
- added C14, C17, C18, C20: 10n, Capacitor_THT:C_Disc_D3.8mm_W2.6mm_P2.50mm, symbol Device:C
- added C19, C21: 220n, Capacitor_THT:CP_Radial_D6.3mm_P2.50mm, symbol Device:C_Polarized_US
- added D3, D5: LED, LED_THT:LED_D4.0mm, symbol Device:LED
- added D4, D6: D, Diode_THT:D_DO-41_SOD81_P7.62mm_Horizontal, symbol Device:D
- added R10, R12, R13, R14, R15, R17, R18, R19, R22, R8: 10k, Resistor_THT:R_Axial_DIN0207_L6.3mm_D2.5mm_P10.16mm_Horizontal, symbol Device:R_US
- added R11, R16: 300, Resistor_THT:R_Axial_DIN0207_L6.3mm_D2.5mm_P10.16mm_Horizontal, symbol Device:R_US
- added R20, R23: 22k, Resistor_THT:R_Axial_DIN0207_L6.3mm_D2.5mm_P10.16mm_Horizontal, symbol Device:R_US
- added R21, R24: 33k, Resistor_THT:R_Axial_DIN0207_L6.3mm_D2.5mm_P10.16mm_Horizontal, symbol Device:R_US
- added U3, U4: A3144, Connector_PinHeader_2.54mm:PinHeader_1x03_P2.54mm_Vertical, symbol DT13-6P:A3144
- added U5, U6: NE555P, Package_DIP:DIP-8_W7.62mm, symbol Timer:NE555P
- renumbered C7 to C8, H3 to H2, H2 to H3, R8 to R9
Connections:
- net +5V: now also C10.1, C11.1, C12.1, C13.1, D3.2 (A), D5.2 (A), R12.1, R14.1, R17.1, R18.1, R19.1, R20.1, R22.1, R23.1, U3.1 (Vcc), U4.1 (Vcc), U5.4 (R), U5.8 (VCC), U6.4 (R), U6.8 (VCC)
- net GND: now also C10.2, C11.2, C12.2, C13.2, C15.2, C16.2, C17.1, C19.2, C20.1, C21.2, C7.2, C9.2, U3.2 (GND), U4.2 (GND), U5.1 (GND), U6.1 (GND)
- net Nano_Input1: now reaches UNIT_2.20 (A1)
- net Nano_Input1: now also C16.1, R15.2
- net Nano_Input2: now reaches UNIT_2.21 (A2)
- net Nano_Input2: now also C9.1, R10.2
- new net: R23.2, R24.1
- new net: R20.2, R21.1
- new net: D3.1 (K), R11.1
- new net: D5.1 (K), R16.1
- new net CV1: C17.2, U5.5 (CV)
- new net CV2: C20.2, U6.5 (CV)
- new net DIS_THR1: C19.1, R21.2, U5.6 (THR), U5.7 (DIS)
- new net DIS_THR2: C21.1, R24.2, U6.6 (THR), U6.7 (DIS)
- new net Diff1: C14.2, D4.1 (K), R14.2
- new net Diff2: C18.2, D6.1 (K), R19.2
- new net Filter1.1: C15.1, R13.2, R15.1
- new net Filter1.2: C7.1, R10.1, R8.2
- new net Hall_Out1: C14.1, R11.2, R12.2, U3.3 (OUT)
- new net Hall_Out2: C18.1, R16.2, R18.2, U4.3 (OUT)
- new net NE555_Out1: R13.1, U5.3 (Q)
- new net NE555_Out2: R8.1, U6.3 (Q)
- new net Rect1: D4.2 (A), R17.2, U5.2 (TR)
- new net Rect2: D6.2 (A), R22.2, U6.2 (TR)
- no-connect marks 22 -> 20
