File: hardware/KICAD Projects/BAJE SAE/Sensor Projects/Speedometer/Speedometer.kicad_pcb (KiCad board)
At the start: 2 copper layers, 81 x 89 mm, 26 parts, among them J1 Conn_01x02, J3 Conn_01x02, J4 CAN to outer connector, Q1 NPN, U1 NE555P, U2 LM311

Commit message: Add footprints to PCB Editor.
Parts:
- removed J1: Conn_01x02, Connector_Wire:SolderWire-0.75sqmm_1x02_P4.8mm_D1.25mm_OD2.3mm
- removed Q1: NPN, Package_TO_SOT_THT:TO-92L_Inline
- removed R10, R11: 10k, Resistor_THT:R_Axial_DIN0411_L9.9mm_D3.6mm_P15.24mm_Horizontal
- removed REF** (x2): MountingHole_3.2mm_M3, MountingHole:MountingHole_3.2mm_M3
- removed UNIT_1: ARDUINO_NANO, 0_nano:SHIELD_ARDUINO_NANO
- removed VR1: 3362P-1-103, 0_custom:TRIM_3362P-1-103
- added C5: 220n, Capacitor_THT:CP_Radial_D6.3mm_P2.50mm, F.Cu at (157.0, 105.5)
- added C6: 10µ, Capacitor_THT:CP_Radial_D4.0mm_P2.00mm, F.Cu at (156.0, 93.2)
- added C7: 10µ, Capacitor_THT:CP_Radial_D4.0mm_P2.00mm, F.Cu at (156.0, 98.8)
- added H1: MountingHole, MountingHole:MountingHole_3.2mm_M3, F.Cu at (150.2, 77.2)
- added H2: MountingHole, MountingHole:MountingHole_3.2mm_M3, F.Cu at (150.2, 85.1)
- added H3: MountingHole, MountingHole:MountingHole_3.2mm_M3, F.Cu at (150.2, 93.0)
- added H4: MountingHole, MountingHole:MountingHole_3.2mm_M3, F.Cu at (150.2, 101.0)
- added R8: 10k, Resistor_THT:R_Axial_DIN0411_L9.9mm_D3.6mm_P15.24mm_Horizontal, F.Cu at (188.5, 69.1)
- C1: value 10u -> 10µ; footprint Capacitor_THT:CP_Radial_D5.0mm_P2.50mm -> Capacitor_THT:CP_Radial_D4.0mm_P2.00mm
- C2, C3: value 10u -> 10n; footprint Capacitor_THT:CP_Radial_D5.0mm_P2.50mm -> Capacitor_THT:C_Disc_D3.8mm_W2.6mm_P2.50mm
- C4: value C -> 10n; footprint Capacitor_THT:C_Disc_D6.0mm_W4.4mm_P5.00mm -> Capacitor_THT:C_Disc_D3.8mm_W2.6mm_P2.50mm
- D1: value ~ -> LED; footprint Diode_THT:D_A-405_P7.62mm_Horizontal -> LED_THT:LED_D4.0mm
- D2: footprint Diode_THT:D_A-405_P7.62mm_Horizontal -> Diode_THT:D_DO-41_SOD81_P7.62mm_Horizontal
- J3: value Conn_01x02 -> CAN to outer connector; footprint Connector_Wire:SolderWire-0.75sqmm_1x02_P4.8mm_D1.25mm_OD2.3mm -> Connector_Wire:SolderWire-0.1sqmm_1x04_P3.6mm_D0.4mm_OD1mm
- J4: value CAN to outer connector -> Conn_01x02; footprint Connector_Wire:SolderWire-0.1sqmm_1x04_P3.6mm_D0.4mm_OD1mm -> Connector_Wire:SolderWire-0.75sqmm_1x02_P4.8mm_D1.25mm_OD2.3mm
- R1: value 10 -> 300; footprint Resistor_THT:R_Axial_DIN0411_L9.9mm_D3.6mm_P15.24mm_Horizontal -> Resistor_THT:R_Axial_DIN0207_L6.3mm_D2.5mm_P10.16mm_Horizontal
- R2: value 470 -> 10k; footprint Resistor_THT:R_Axial_DIN0411_L9.9mm_D3.6mm_P15.24mm_Horizontal -> Resistor_THT:R_Axial_DIN0207_L6.3mm_D2.5mm_P10.16mm_Horizontal
- R3: value 1k -> 10k; footprint Resistor_THT:R_Axial_DIN0411_L9.9mm_D3.6mm_P15.24mm_Horizontal -> Resistor_THT:R_Axial_DIN0207_L6.3mm_D2.5mm_P10.16mm_Horizontal
- R4: value 430 -> 10k; footprint Resistor_THT:R_Axial_DIN0411_L9.9mm_D3.6mm_P15.24mm_Horizontal -> Resistor_THT:R_Axial_DIN0207_L6.3mm_D2.5mm_P10.16mm_Horizontal
- R5: value 10k -> 22k; footprint Resistor_THT:R_Axial_DIN0411_L9.9mm_D3.6mm_P15.24mm_Horizontal -> Resistor_THT:R_Axial_DIN0207_L6.3mm_D2.5mm_P10.16mm_Horizontal
- R6: value 430 -> 33k; footprint Resistor_THT:R_Axial_DIN0411_L9.9mm_D3.6mm_P15.24mm_Horizontal -> Resistor_THT:R_Axial_DIN0207_L6.3mm_D2.5mm_P10.16mm_Horizontal
- R7: value 2k -> 10k
- U1: value NE555P -> A3144; footprint Package_DIP:DIP-8_W7.62mm -> SS49E:TO92127P460H470-3
- U2: value LM311 -> NE555P
- UNIT_2: value HiLetgo CAN Bus -> ARDUINO_NANO; footprint 0_Baja_Final:HiLetgo CAN Bus (Facing Up) -> Module:Arduino_Nano; moved to F.Cu
- moved J3 76.8 mm to (188.4, 73.5), turned to 0 degrees
- moved R7 68.2 mm to (188.5, 63.9), turned to 0 degrees
- moved R6 67.3 mm to (134.5, 95.5), turned to 0 degrees
- moved J4 66.9 mm to (189.0, 77.6), turned to 0 degrees
- moved D1 63.0 mm to (134.9, 105.0), turned to 0 degrees
- moved R4 60.1 mm to (134.5, 87.3)
- moved D2 56.4 mm to (134.8, 99.6), turned to 0 degrees
- moved R2 52.5 mm to (134.5, 79.2), turned to 0 degrees
- moved UNIT_2 33.8 mm to (169.3, 65.9), turned to 0 degrees
- moved C3 33.5 mm to (161.4, 91.2)
- moved C2 32.6 mm to (161.4, 87.0), turned to 0 degrees
- moved U1 32.3 mm to (150.2, 108.1), turned to 0 degrees
- moved C4 28.9 mm to (161.4, 95.3), turned to 0 degrees
- moved R1 27.7 mm to (134.5, 75.2), turned to 0 degrees
- moved R3 26.5 mm to (134.5, 83.3), turned to 0 degrees
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Connections:
- C1 pad 1: Net-(C1-Pad1) -> 5V
- C2 pad 1: arduino input -> 5V
- C3 pad 1: GND -> /Hall_Out
- C3 pad 2: Net-(U1-DIS) -> /Diff
- C4 pad 1: Net-(U1-CV) -> GND
- C4 pad 2: GND -> /CV
- D1 pad 2: GND -> 5V
- D2 pad 1: Net-(D1-K) -> /Diff
- D2 pad 2: GND -> /Rect
- J3 pad 1: +5v -> Low
- J3 pad 2: GND -> High
- J4 pad 1: Low -> GND
- J4 pad 2: High -> 5V
- R1 pad 1: Possitive -> Net-(D1-K)
- R1 pad 2: Net-(D1-K) -> /Hall_Out
- R2 pad 1: Net-(D1-K) -> 5V
- R2 pad 2: Net-(Q1-B) -> /Hall_Out
- R3 pad 1: +5v -> 5V
- R3 pad 2: Comparator input -> /Diff
- R4 pad 1: Net-(R4-Pad1) -> 5V
- R4 pad 2: Net-(R4-Pad2) -> /Rect
- R5 pad 1: 555 output -> 5V
- R5 pad 2: Net-(C1-Pad1) -> Net-(R5-Pad2)
- R6 pad 1: Net-(R4-Pad2) -> Net-(R5-Pad2)
- R6 pad 2: +5v -> /DIS_THR
- R7 pad 1: Net-(U1-DIS) -> /NE555_Out
- R7 pad 2: Net-(R4-Pad1) -> /Filter1
- U1 pad 1: GND -> 5V
- U1 pad 2: 555 input -> GND
- U1 pad 3: 555 output -> /Hall_Out
- U2 pad 2: Comparator input -> /Rect
- U2 pad 3: Net-(U2--) -> /NE555_Out
- U2 pad 4: GND -> 5V
- U2 pad 5: unconnected-(U2-BAL-Pad5) -> /CV
- U2 pad 6: unconnected-(U2-STRB-Pad6) -> /DIS_THR
- U2 pad 7: 555 input -> /DIS_THR
- U2 pad 8: +5v -> 5V
- UNIT_2 pad 2: SCK -> unconnected-(UNIT_2-D0/RX-Pad2)
- UNIT_2 pad 3: SI -> unconnected-(UNIT_2-RESET-Pad3)
- UNIT_2 pad 4: SO -> GND
- UNIT_2 pad 5: CS -> unconnected-(UNIT_2-D2-Pad5)
- UNIT_2 pad 6: GND -> unconnected-(UNIT_2-D3-Pad6)
- UNIT_2 pad 7: +5V -> unconnected-(UNIT_2-D4-Pad7)
- UNIT_2 pad 8: High -> unconnected-(UNIT_2-D5-Pad8)
- UNIT_2 pad 9: Low -> unconnected-(UNIT_2-D6-Pad9)
Routing:
- net GND: track 325.5 -> 0.00 mm
- net +5v: track 122.0 -> 0.00 mm
- net SI: track 55.6 -> 0.00 mm
- net SO: track 45.1 -> 0.00 mm
- net SCK: track 43.0 -> 0.00 mm
- net Low: track 39.1 -> 0.00 mm
- net 555 input: track 36.3 -> 0.00 mm
- net +5V: track 36.1 -> 0.00 mm
- net Net-(U1-DIS): track 33.9 -> 0.00 mm
- net 555 output: track 21.4 -> 0.00 mm
- net Net-(D1-K): track 20.7 -> 0.00 mm
- net arduino input: track 19.7 -> 0.00 mm
- net High: track 19.3 -> 0.00 mm
- net Comparator input: track 18.7 -> 0.00 mm
- net Net-(Q1-B): track 17.0 -> 0.00 mm
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Other:
- board outline removed

Commit message: Arange parts and add edge cuts around mounting holes.
Parts:
- moved J4 69.8 mm to (119.5, 71.0)
- moved J3 62.7 mm to (126.0, 66.5), turned to 180 degrees
- moved UNIT_2 56.4 mm to (119.3, 92.2), turned to 90 degrees
- moved U1 54.8 mm to (123.5, 60.2), turned to -90 degrees
- moved R7 54.8 mm to (133.9, 68.0)
- moved D1 51.2 mm to (126.0, 54.5), turned to 180 degrees
- moved R6 50.8 mm to (155.0, 48.9), turned to -90 degrees
- moved C2 49.8 mm to (118.0, 62.5)
- moved H1 49.5 mm to (111.0, 47.0)
- moved R5 48.5 mm to (158.0, 49.0), turned to -90 degrees
- moved C1 47.9 mm to (118.5, 58.0)
- moved C5 41.7 mm to (156.0, 63.8), turned to -90 degrees
- moved C3 41.4 mm to (132.0, 62.0), turned to -90 degrees
- moved H2 40.5 mm to (164.0, 47.0)
- moved R8 39.7 mm to (149.0, 72.5), turned to 180 degrees
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Other:
- board outline added: 66.1 x 62.6 mm

Commit message: Add routing; add GND copper field.
Parts:
- moved R5 10.5 mm to (158.5, 59.5), turned to 90 degrees
- moved R6 0.58 mm to (155.0, 49.5)
Routing:
- net 5V: track 0.00 -> 73.7 mm
- net /NE555_Out: track 0.00 -> 21.4 mm
- net /Filter2: track 0.00 -> 19.0 mm
- net /Rect: track 0.00 -> 14.0 mm
- net /DIS_THR: track 0.00 -> 12.3 mm
- net /Hall_Out: track 0.00 -> 11.7 mm
- net /Filter1: track 0.00 -> 8.97 mm
- net /Diff: track 0.00 -> 7.65 mm
- net Net-(D1-K): track 0.00 -> 6.31 mm
- net /CV: track 0.00 -> 6.14 mm
- net Net-(R5-Pad2): track 0.00 -> 3.57 mm
- added copper zone on B.Cu, net GND

Commit message: DRC Check, Edit Silkscreen.
Parts:
- removed J3: CAN to outer connector, Connector_Wire:SolderWire-0.1sqmm_1x04_P3.6mm_D0.4mm_OD1mm
- added UNIT_1: HiLetgo CAN Bus, SS49E:CAN_MCP2515, F.Cu at (94.7, 77.9)
- J4: value Conn_01x02 -> Battery
- moved H1 42.2 mm to (70.5, 59.0)
- moved H4 40.6 mm to (70.4, 96.5)
- moved J4 2.51 mm to (119.2, 68.5)
- moved R6 0.16 mm to (155.0, 49.3)
- moved R8 0.12 mm to (149.1, 72.5)
- moved R1 0.08 mm to (129.0, 49.3)
- moved R2 0.08 mm to (132.0, 49.3)
- moved R3 0.08 mm to (135.5, 49.3)
Connections:
- net /Filter2 renamed /Nano_Input
- net 5V renamed +5V
- UNIT_2 pad 13: unconnected-(UNIT_2-D10-Pad13) -> CS
- UNIT_2 pad 17: 3.3V -> unconnected-(UNIT_2-3V3-Pad17)
- UNIT_2 pad 23: SDA -> unconnected-(UNIT_2-A4-Pad23)
- UNIT_2 pad 24: SCL -> unconnected-(UNIT_2-A5-Pad24)
Routing:
- net SO: track 0.00 -> 49.2 mm
- net SI: track 0.00 -> 46.2 mm
- net SCK: track 0.00 -> 44.4 mm
- net +5V: track 73.7 -> 117.5 mm
- net CS: track 0.00 -> 41.6 mm
- net GND: track 0.00 -> 17.3 mm
Other:
- board size 66.1 x 62.6 mm -> 106.6 x 62.6 mm
- board text added: "CAN"
- board text added: "NANO"

Commit message: Add final silkscreen and page settings.
Other:
- board text added: "Jack Tanner Baja 2024-2025"
Changed lines of the file:
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@@
 	)
 	(paper "A4")
+	(title_block
+		(title "Baja Speedometer")
+		(date "2025-02-02")
+		(rev "v1")
+		(company "University of Arizona")
+		(comment 1 "Jack Tanner")
+	)
 	(layers
 		(0 "F.Cu" signal)
@@
 		(layer "Edge.Cuts")
 	)
+	(gr_text "Jack Tanner\nBaja 2024-2025\n"
+		(at 103.11 79.01 0)
+		(layer "B.SilkS")
+		(effects
+			(font
+				(size 2 2)
+				(thickness 0.5)
+				(bold yes)
+			)
+			(justify left bottom mirror)
+		)
+	)
 	(gr_text "NANO"
