File: hardware/KICAD Projects/BAJE SAE/Sensor Projects/Speedometer/Speedometer.kicad_pcb (KiCad board)
At the start: 2 copper layers, 106.6 x 62.6 mm, 26 parts, among them J4 Battery, U1 A3144, U2 NE555P

Commit message: Change edge cuts.
Parts:
- moved H1 7.50 mm to (68.6, 51.8)
- moved H4 6.69 mm to (69.0, 90.0)
- moved H3 6.69 mm to (165.4, 90.0)
- moved H2 4.99 mm to (165.5, 51.8)
Other:
- board size 106.6 x 62.6 mm -> 104.4 x 46.4 mm
Changed lines of the file:
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@@
 	(footprint "MountingHole:MountingHole_3.2mm_M3"
 		(layer "F.Cu")
-		(at 70.5 59)
+		(at 68.57 51.75)
 		(descr "Mounting Hole 3.2mm, no annular, M3")
 		(tags "mounting hole 3.2mm no annular m3")
@@
 	(footprint "MountingHole:MountingHole_3.2mm_M3"
 		(layer "F.Cu")
-		(at 164 96.5)
+		(at 165.39 89.96)
 		(descr "Mounting Hole 3.2mm, no annular, M3")
 		(tags "mounting hole 3.2mm no annular m3")
@@
 	(footprint "MountingHole:MountingHole_3.2mm_M3"
 		(layer "F.Cu")
-		(at 70.376361 96.5)
+		(at 68.98 89.96)
 		(descr "Mounting Hole 3.2mm, no annular, M3")
 		(tags "mounting hole 3.2mm no annular m3")
@@
 	(footprint "MountingHole:MountingHole_3.2mm_M3"
 		(layer "F.Cu")
-		(at 164 47)
+		(at 165.52 51.75)
 		(descr "Mounting Hole 3.2mm, no annular, M3")
 		(tags "mounting hole 3.2mm no annular m3")
@@
 		)
 		(fp_text user "${REFERENCE}"
-			(at 0 0 0)
+			(at -0.13 0.25 0)
 			(layer "F.Fab")
 			(effects
@@
 		)
 	)
-	(gr_line
-		(start 77.057559 59.893898)
-		(end 114 60)
-		(stroke
-			(width 0.05)
-			(type default)
-		)
-		(layer "Edge.Cuts")
-	)
-	(gr_line
-		(start 122 48)
-		(end 114 60)
-		(stroke
-			(width 0.05)
-			(type default)
-		)
-		(layer "Edge.Cuts")
-	)
-	(gr_line
-		(start 73.123639 90.582618)
-		(end 73 65)
-		(stroke
-			(width 0.05)
-			(type default)
-		)
-		(layer "Edge.Cuts")
-	)
-	(gr_line
-		(start 122 48)
-		(end 157.5 48)
-		(stroke
-			(width 0.05)
-			(type default)
-		)
-		(layer "Edge.Cuts")
-	)
-	(gr_arc
-		(start 76.43392 94)
-		(mid 65.765148 101.022452)
-		(end 73.123639 90.582618)
-		(stroke
-			(width 0.05)
-			(type default)
-		)
-		(layer "Edge.Cuts")
-	)
-	(gr_arc
-		(start 73 65)
-		(mid 65.408784 54.802429)
-		(end 77.057559 59.893898)
-		(stroke
-			(width 0.05)
-			(type default)
-		)
-		(layer "Edge.Cuts")
-	)
-	(gr_line
-		(start 158 94)
-		(end 76.43392 94)
-		(stroke
-			(width 0.05)
-			(type default)
-		)
-		(layer "Edge.Cuts")
-	)
-	(gr_line
-		(start 162.110264 53.299119)
-		(end 161.94452 90.333559)
-		(stroke
-			(width 0.05)
-			(type default)
-		)
-		(layer "Edge.Cuts")
-	)
-	(gr_arc
-		(start 157.5 48)
-		(mid 168.96156 42.683414)
-		(end 162.110264 53.299119)
-		(stroke
-			(width 0.05)
-			(type default)
-		)
-		(layer "Edge.Cuts")
-	)
-	(gr_arc
-		(start 161.94452 90.333559)
-		(mid 168.425312 101.260946)
-		(end 158 94)
+	(gr_rect
+		(start 65.03 47.97)
+		(end 169.44 94.34)
 		(stroke
 			(width 0.05)
 			(type default)
 		)
+		(fill none)
 		(layer "Edge.Cuts")
 	)

Commit message: Add L/H connectors and adjust footprints.
Parts:
- removed J4: Battery, Connector_Wire:SolderWire-0.75sqmm_1x02_P4.8mm_D1.25mm_OD2.3mm
- added J1: Conn_01x02, Connector_Wire:SolderWire-0.75sqmm_1x02_P4.8mm_D1.25mm_OD2.3mm, F.Cu at (101.7, 60.0)
- added J2: CAN to outer connector, Connector_Wire:SolderWire-0.1sqmm_1x04_P3.6mm_D0.4mm_OD1mm, F.Cu at (87.2, 54.0)
- R7, R8: footprint Resistor_THT:R_Axial_DIN0411_L9.9mm_D3.6mm_P15.24mm_Horizontal -> Resistor_THT:R_Axial_DIN0207_L6.3mm_D2.5mm_P10.16mm_Horizontal
- U1: footprint SS49E:TO92127P460H470-3 -> Connector_PinHeader_2.54mm:PinHeader_1x03_P2.54mm_Vertical
- UNIT_1: footprint SS49E:CAN_MCP2515 -> 0_Baja_Final:Can Bus (Correct); moved to B.Cu
- moved UNIT_1 24.2 mm to (71.8, 85.5), turned to -90 degrees
- moved U1 6.84 mm to (124.5, 67.0), turned to 180 degrees
- moved R8 3.04 mm to (146.1, 72.5)
- moved R7 1.96 mm to (135.8, 68.0)
Routing:
- net High: track 0.00 -> 42.0 mm
- net Low: track 0.00 -> 37.6 mm
- net CS: track 41.6 -> 57.3 mm
- net SCK: track 44.4 -> 48.1 mm
- net /Filter1: track 9.09 -> 11.8 mm
- net +5V: track 117.5 -> 115.0 mm
- net /NE555_Out: track 21.4 -> 19.4 mm
- net SO: track 49.2 -> 50.1 mm
- net /Hall_Out: track 11.7 -> 10.9 mm
- net GND: vias 0 -> 2
Other:
- board text added: "5V"
- board text added: "GND"
- board text added: "High"
- board text added: "Low"

Commit message: New Gerber files with corrected pins, Vin, and dimensions.
Changed lines of the file:
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@@
 			(at 2.4 -2.47 0)
 			(layer "F.SilkS")
+			(hide yes)
 			(effects
 				(font

Commit message: Gerber 3.0 added.
Parts:
- UNIT_1: footprint 0_Baja_Final:Can Bus (Correct) -> 0_Baja_Final:Jack_CanBus
Connections:
- UNIT_2 pad 30: unconnected-(UNIT_2-VIN-Pad30) -> +5V
Routing:
- net +5V: track 115.0 -> 120.9 mm
- net SI: track 46.6 -> 44.2 mm
- net SO: track 50.1 -> 48.0 mm
- net SCK: track 48.1 -> 45.9 mm
- net CS: track 57.3 -> 55.3 mm
- net Low: track 37.6 -> 39.2 mm
- net High: track 42.0 -> 42.6 mm
