File: hardware/KICAD Projects/BAJE SAE/Dash/Dash.kicad_sch (KiCad schematic)
At the start: 18 parts, among them U1 28-SOIC

Commit message: updated footprint for breakout
Parts:
- removed U$1, U$3: MOUNTINGHOLE2.5, Dash:MOUNTINGHOLE_2.5_PLATED, symbol Dash-eagle-import:MOUNTINGHOLE2.5
- removed U$2, U$4, U$5: FIDUCIAL, Dash:FIDUCIAL_1MM, symbol Dash-eagle-import:FIDUCIAL
- U1: footprint Dash:SOP28_300MIL -> BAJA SAE:Adafruit HT16K33 breakout
Other:
- moved on the sheet: A1, A2, A3, C1, D1, JP1, JP2, R1, R2, R3, R4, R5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

Commit message: dash <3
Parts:
- removed A1, A2, A3: SOLDERJUMPERREFLOW_NOPASTE, Dash:SOLDERJUMPER_REFLOW_NOPASTE, symbol Dash-eagle-import:SOLDERJUMPERREFLOW_NOPASTE
- removed C1: 10uF, Dash:C0805, symbol Dash-eagle-import:C-USC0805
- removed D1: 1N4148, Dash:SOD-323F, symbol Dash-eagle-import:DIODESOD-323F
- removed JP1, JP2: PINHD-1X14-CB, Dash:1X14-CB, symbol Dash-eagle-import:PINHD-1X14-CB
- removed R1, R2, R3: 47K, Dash:R0805, symbol Dash-eagle-import:R-US_R0805
- removed R4, R5: 10K, Dash:R0805, symbol Dash-eagle-import:R-US_R0805
- removed U1: 28-SOIC, BAJA SAE:Adafruit HT16K33 breakout, symbol Dash-eagle-import:HT16K33_SOP28
- added D1, D10, D11, D12, D13, D14, D15, D16, D17, D18, D19, D2, D20, D3, D4, D5, D6, D7, D8, D9: LED, LED_THT:LED_D5.0mm, symbol Device:LED
- added J1: Conn_01x02, Connector_Wire:SolderWire-0.75sqmm_1x02_P4.8mm_D1.25mm_OD2.3mm, symbol Connector_Generic:Conn_01x02
- added J10: 14 Segment (3), Connector_PinHeader_2.54mm:PinHeader_1x04_P2.54mm_Vertical, symbol Connector_Generic:Conn_01x04
- added J11: 14 Segment (4), Connector_PinHeader_2.54mm:PinHeader_1x04_P2.54mm_Vertical, symbol Connector_Generic:Conn_01x04
- added J2: CAN to outer connector, Connector_Wire:SolderWire-0.1sqmm_1x04_P3.6mm_D0.4mm_OD1mm, symbol Connector_Generic:Conn_01x04
- added J3: Conn_01x06, symbol Connector_Generic:Conn_01x06
- added J4: Servo 1 (RPM), Connector_PinHeader_2.54mm:PinHeader_1x03_P2.54mm_Vertical, symbol Connector_Generic:Conn_01x03
- added J5: Servo 2 (Speed), Connector_PinHeader_2.54mm:PinHeader_1x03_P2.54mm_Vertical, symbol Connector_Generic:Conn_01x03
- added J6: Button 1, Connector_PinHeader_2.54mm:PinHeader_1x02_P2.54mm_Vertical, symbol Connector_Generic:Conn_01x02
- added J7: Button 2, Connector_PinHeader_2.54mm:PinHeader_1x02_P2.54mm_Vertical, symbol Connector_Generic:Conn_01x02
- added J8: 14 Segment (1), Connector_PinHeader_2.54mm:PinHeader_1x04_P2.54mm_Vertical, symbol Connector_Generic:Conn_01x04
- added J9: 14 Segment (2), Connector_PinHeader_2.54mm:PinHeader_1x04_P2.54mm_Vertical, symbol Connector_Generic:Conn_01x04
- added U1: ~, BAJA SAE:LED Breakout, symbol 0_Custom:LED_Breakout
- added UNIT_1: ESP32-DEVKITC-32D, BAJA SAE:MODULE_ESP32-DEVKITC-32D, symbol BAJA SAE:ESP32-DEVKITC-32D
- added UNIT_3: CAN Bus, BAJA SAE:HiLetgo CAN Bus (Facing Up), symbol BAJA SAE:HiLetgo_CAN_BUS
Connections:
- net A0: now also D10.2 (A), D9.2 (A), U1.25 (A0)
- net A1: now also D11.2 (A), D12.2 (A), U1.24 (A1)
- net A2: now also D13.2 (A), D14.2 (A), U1.23 (A2)
- net GND: now also J1.2 (Pin_2), J10.4 (Pin_4), J11.4 (Pin_4), J4.1 (Pin_1), J5.1 (Pin_1), J6.2 (Pin_2), J7.2 (Pin_2), J8.4 (Pin_4), J9.4 (Pin_4), UNIT_1.J2-14 (GND1), UNIT_1.J3-1 (GND3), UNIT_1.J3-7 (GND2), UNIT_3.6 (GND)
- net SCL: now also J10.1 (Pin_1), J11.1 (Pin_1), J8.1 (Pin_1), J9.1 (Pin_1), UNIT_1.J3-3 (IO22)
- net SDA: now also J10.2 (Pin_2), J11.2 (Pin_2), J8.2 (Pin_2), J9.2 (Pin_2), UNIT_1.J3-6 (IO21)
- new net +5v: J1.1 (Pin_1), J4.2 (Pin_2), J5.2 (Pin_2), UNIT_1.J2-19 (EXT_5V), UNIT_3.7 (VCC)
- new net A3: D15.2 (A), D16.2 (A), U1.22 (A3)
- new net A4: D17.2 (A), D18.2 (A), U1.21 (A4)
- new net A5: D19.2 (A), D20.2 (A), U1.20 (A5)
- new net A6: D1.2 (A), D2.2 (A), U1.19 (A6)
- new net A7: D3.2 (A), D4.2 (A), U1.18 (A7)
- new net A8: D5.2 (A), D6.2 (A), U1.17 (A8)
- new net A9: D7.2 (A), D8.2 (A), U1.16 (A9)
- new net C0: D1.1 (K), D11.1 (K), D13.1 (K), D15.1 (K), D17.1 (K), D19.1 (K), D3.1 (K), D5.1 (K), D7.1 (K), D9.1 (K), U1.2 (C0)
- new net C1: D10.1 (K), D12.1 (K), D14.1 (K), D16.1 (K), D18.1 (K), D2.1 (K), D20.1 (K), D4.1 (K), D6.1 (K), D8.1 (K), U1.3 (C1)
- new net C2: U1.4 (C2)
- new net C3: U1.5 (C3)
- new net C4: U1.6 (C4)
- new net C5: U1.7 (C5)
- new net C6: U1.8 (C6)
- new net C7: U1.9 (C7)
- new net CS: UNIT_1.J3-10 (IO5), UNIT_3.5 (CS)
- new net High: J2.2 (Pin_2), J2.4 (Pin_4), UNIT_3.8 (High_CAN)
- new net IO12 Button 1: J6.1 (Pin_1), UNIT_1.J2-13 (IO12)
- new net IO14 Button 2: J7.1 (Pin_1), UNIT_1.J2-12 (IO14)
- new net IO32 Speed: J5.3 (Pin_3), UNIT_1.J2-7 (IO32)
- new net IO33 RPM: J4.3 (Pin_3), UNIT_1.J2-8 (IO33)
- new net Low: J2.1 (Pin_1), J2.3 (Pin_3), UNIT_3.9 (Low_CAN)
- new net Regulated 3v3: J10.3 (Pin_3), J11.3 (Pin_3), J8.3 (Pin_3), J9.3 (Pin_3)
- new net SCK: UNIT_1.J3-9 (IO18), UNIT_3.2 (SCK)
- new net SI: UNIT_1.J3-2 (IO23), UNIT_3.3 (SI)
- new net SO: UNIT_1.J3-8 (IO19), UNIT_3.4 (SO)
- no-connect marks 0 -> 31
Other:
- note added: "+5v"
- note added: "14 Segments"
- note added: "Buttons"
- note added: "CAN Bus"
- note added: "Connector Pinout"
- note added: "ESP-32 Socketed with ESS-119-T-03"
- note added: "ESP32"
- note added: "GND"
- note added: "High"
- note added: "I/O"
- note added: "LED Breakout"
- note added: "LEDs"
- note added: "Low"
- note added: "Servos"
- note added: "Socket"

Commit message: Added 3v3 voltage regulation
Parts:
- added R1: 1.7k, symbol Device:R
- added R2: 6.6k, symbol Device:R
- added RV1: 300 (3v3 tune), symbol Device:R_Potentiometer_Trim
- added TP1: 3v3, symbol Connector:TestPoint
Connections:
- net +5v: now also R1.1
- net GND: now also RV1.1
- net Regulated 3v3: now also RV1.2, TP1.1
- new net: R2.2, RV1.3
- new net: R1.2, R2.1
Other:
- note added: "Power Regulation"
- note removed: "I/O"
- moved on the sheet: J1, J2

Commit message: made schematic pretty
Connections:
- net GND: now also R2.2, U1.1 (GND)
- net Regulated 3v3: now also U1.28 (VDD)
- net at RV1.3: now also R1.2, R2.1; no longer R2.2
Other:
- moved on the sheet: D1, D10, D11, D12, D13, D14, D15, D16, D17, D18, D19, D2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

Commit message: dash updates
Parts:
- RV1: value 300 (3v3 tune) -> 1k (3v3 tune)
Changed lines of the file:
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@@
 			)
 		)
-		(property "Value" "300 (3v3 tune)"
+		(property "Value" "1k (3v3 tune)"
 			(at 145.034 80.01 0)
 			(effects
