File: hardware/KICAD Projects/BAJE SAE/Dash/Dash Master/Dash.kicad_sch (KiCad schematic)
At the start: 38 parts, among them J1 Conn_01x02, J10 14 Segment (3), J11 14 Segment (4), J2 CAN to outer connector, J3 Conn_01x06, J4 Servo 1 (RPM), J5 Servo 2 (Speed), J6 Button 1, J7 Button 2, J8 14 Segment (1), J9 14 Segment (2)

Commit message: Updates to dash
Parts:
- removed D5, D6, D7, D8: LED, LED_THT:LED_D5.0mm, symbol Device:LED
Other:
- moved on the sheet: D1, D10, D11, D12, D13, D14, D15, D16, D17, D18, D19, D2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
