File: hardware/KICAD Projects/BAJE SAE/Dash/Dash Indicators (Left)/Dash Indicators (Left).kicad_pcb (KiCad board)
At the start: 2 copper layers, 55.8 x 87 mm, 23 parts, among them J1-A1 Conn_01x05, J1-B1 Conn_01x05

Commit message: temp sense worky now
Parts:
- moved G*** 62.3 mm to (31.4, 66.9)
- moved J1-A1 1.16 mm to (98.0, 105.3)
Routing:
- net A9: track 60.8 -> 59.6 mm
- net A10: track 81.9 -> 80.7 mm
- net A12: track 72.9 -> 72.2 mm
- net A8: track 87.5 -> 87.0 mm
Changed lines of the file:
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@@
 			(outputformat 1)
 			(mirror no)
-			(drillshape 1)
+			(drillshape 0)
 			(scaleselection 1)
-			(outputdirectory "")
+			(outputdirectory "Gerbers/")
 		)
 	)
@@
 	(footprint "BAJA SAE:Untitled"
 		(layer "B.Cu")
-		(at 93.5 71.5 90)
+		(at 31.4 66.9 90)
 		(property "Reference" "G***"
 			(at 0 0 90)
@@
 	(footprint "Connector_PinHeader_2.54mm:PinHeader_1x05_P2.54mm_Vertical"
 		(layer "B.Cu")
-		(at 98.04 106.5 90)
+		(at 98.04 105.34 90)
 		(descr "Through hole straight pin header, 1x05, 2.54mm pitch, single row")
 		(tags "Through hole pin header THT 1x05 2.54mm single row")
@@
 	(dimension
 		(type aligned)
-		(layer "Edge.Cuts")
-		(pts
-			(xy 112.7 40.231088) (xy 114.5 42.031088)
-		)
-		(height -5.816149)
-		(gr_text "2.5456 mm"
-			(at 118.525811 36.205277 315)
-			(layer "Edge.Cuts")
-			(effects
-				(font
-					(size 1 1)
-					(thickness 0.15)
-				)
-			)
-		)
-		(format
-			(prefix "")
-			(suffix "")
-			(units 3)
-			(units_format 1)
-			(precision 4)
-		)
-		(style
-			(thickness 0.05)
-			(arrow_length 1.27)
-			(text_position_mode 0)
-			(extension_height 0.58642)
-			(extension_offset 0.5) keep_text_aligned)
-	)
-	(dimension
-		(type aligned)
-		(layer "Edge.Cuts")
-		(pts
-			(xy 112.7 96.828932) (xy 114.5 95.028932)
-		)
-		(height 12.052121)
-		(gr_text "2.5456 mm"
-			(at 121.308963 103.637895 45)
-			(layer "Edge.Cuts")
-			(effects
-				(font
-					(size 1 1)
-					(thickness 0.15)
-				)
-			)
-		)
-		(format
-			(prefix "")
-			(suffix "")
-			(units 3)
-			(units_format 1)
-			(precision 4)
-		)
-		(style
-			(thickness 0.05)
-			(arrow_length 1.27)
-			(text_position_mode 0)
-			(extension_height 0.58642)
-			(extension_offset 0.5) keep_text_aligned)
-	)
-	(dimension
-		(type aligned)
 		(layer "F.Fab")
 		(pts
@@
 	(segment
 		(start 107.1 97.4)
-		(end 107.1 46.1)
+		(end 99.16 105.34)
 		(width 0.2)
 		(layer "F.Cu")
@@
 	)
 	(segment
-		(start 107.1 46.1)
-		(end 103.35 42.35)
+		(start 99.16 105.34)
+		(end 98.04 105.34)
 		(width 0.2)
 		(layer "F.Cu")
@@
 	)
 	(segment
-		(start 105 99.54)
-		(end 105 99.5)
-		(width 0.2)
-		(layer "F.Cu")
-		(net 1)
-	)
-	(segment
-		(start 98.04 106.5)
-		(end 105 99.54)
+		(start 107.1 46.1)
+		(end 107.1 97.4)
 		(width 0.2)
 		(layer "F.Cu")
@@
 	(segment
 		(start 103.35 42.35)
-		(end 100.065 42.35)
+		(end 107.1 46.1)
 		(width 0.2)
 		(layer "F.Cu")
@@
 	)
 	(segment
-		(start 105 99.5)
-		(end 107.1 97.4)
+		(start 100.065 42.35)
+		(end 103.35 42.35)
 		(width 0.2)
 		(layer "F.Cu")
@@
 	)
 	(segment
-		(start 95.8 104.9)
-		(end 99.034314 104.9)
+		(start 106.617157 97.317157)
+		(end 99.984314 103.95)
 		(width 0.2)
 		(layer "F.Cu")
@@
 	)
 	(segment
-		(start 95.5 105.2)
-		(end 95.8 104.9)
+		(start 99.984314 103.95)
+		(end 96.89 103.95)
 		(width 0.2)
 		(layer "F.Cu")
@@
 	)
 	(segment
-		(start 105.65 72.35)
-		(end 100.065 72.35)
+		(start 96.89 103.95)
+		(end 95.5 105.34)
 		(width 0.2)
 		(layer "F.Cu")
@@
 	)
 	(segment
-		(start 106.617157 97.317157)
-		(end 106.617157 73.317157)
+		(start 105.65 72.35)
+		(end 100.065 72.35)
 		(width 0.2)
 		(layer "F.Cu")
@@
 	)
 	(segment
-		(start 95.5 106.5)
-		(end 95.5 105.2)
+		(start 106.617157 97.317157)
+		(end 106.617157 73.317157)
 		(width 0.2)
 		(layer "F.Cu")
@@
 	)
 	(segment
-		(start 99.034314 104.9)
-		(end 106.617157 97.317157)
-		(width 0.2)
-		(layer "F.Cu")
-		(net 4)
-	)
-	(segment
 		(start 100.065 71.065)
 		(end 99.4 70.4)
@@
 	)
 	(segment
-		(start 92.96 106.5)
-		(end 94.2 105.26)
-		(width 0.2)
-		(layer "B.Cu")
-		(net 5)
-	)
-	(segment
 		(start 100.065 48.565)
 		(end 98.7 47.2)
@@
 	)
 	(segment
-		(start 94.2 105.26)
-		(end 94.2 100.4)
+		(start 94.2 104.1)
+		(end 92.96 105.34)
 		(width 0.2)
 		(layer "B.Cu")
@@
 	(segment
 		(start 94.2 100.4)
+		(end 94.2 104.1)
+		(width 0.2)
+		(layer "B.Cu")
+		(net 5)
+	)
+	(segment
+		(start 94.2 100.4)
 		(end 95.1 99.5)
 		(width 0.2)
@@
 	)
 	(segment
-		(start 90.42 106.5)
-		(end 90.7 106.5)
+		(start 94.35 100.75)
+		(end 94.35 103.276346)
 		(width 0.2)
 		(layer "F.Cu")
@@
 	)
 	(segment
-		(start 93 104.7)
-		(end 94.2 103.5)
-		(width 0.2)
-		(layer "F.Cu")
-		(net 6)
-	)
-	(segment
-		(start 92.5 104.7)
-		(end 93 104.7)
+		(start 90.2 96.6)
+		(end 94.35 100.75)
 		(width 0.2)
 		(layer "F.Cu")
@@
 	)
 	(segment
-		(start 90.7 106.5)
-		(end 92.5 104.7)
+		(start 93.436346 104.19)
+		(end 91.57 104.19)
 		(width 0.2)
 		(layer "F.Cu")
@@
 	)
 	(segment
-		(start 94.2 100.6)
-		(end 90.2 96.6)
+		(start 94.35 103.276346)
+		(end 93.436346 104.19)
 		(width 0.2)
 		(layer "F.Cu")
@@
 	)
 	(segment
-		(start 94.2 103.5)
-		(end 94.2 100.6)
+		(start 91.57 104.19)
+		(end 90.42 105.34)
 		(width 0.2)
 		(layer "F.Cu")
@@
 	)
 	(segment
-		(start 100.065 57.35)
-		(end 100.065 55.365)
+		(start 88.265 60.035)
+		(end 88.265 57.35)
 		(width 0.2)
 		(layer "B.Cu")
@@
 	)
 	(segment
-		(start 82.1 100.72)
-		(end 82.1 61.4)
+		(start 100.065 57.35)
+		(end 100.065 55.365)
 		(width 0.2)
 		(layer "B.Cu")
@@
 	)
 	(segment
-		(start 87.88 106.5)
-		(end 82.1 100.72)
+		(start 91.7 53.9)
+		(end 91.7 53.915)
 		(width 0.2)
 		(layer "B.Cu")
@@
 	)
 	(segment
-		(start 91.7 53.9)
-		(end 91.7 53.915)
+		(start 81.61 99.07)
+		(end 81.61 61.89)
 		(width 0.2)
 		(layer "B.Cu")
@@
 	)
 	(segment
-		(start 88.265 60.035)
-		(end 88.265 57.35)
+		(start 81.61 61.89)
+		(end 82.4 61.1)
+		(width 0.2)
+		(layer "B.Cu")
+		(net 7)
+	)
+	(segment
+		(start 87.88 105.34)
+		(end 81.61 99.07)
 		(width 0.2)
 		(layer "B.Cu")
@@
 		(width 0.2)
 		(layer "B.Cu")
-		(net 7)
-	)
-	(segment
-		(start 82.1 61.4)
-		(end 82.4 61.1)
-		(width 0.2)
-		(layer "B.Cu")
