File: hardware/KICAD Projects/BAJE SAE/Dash/Dash Indicators (Right)/Dash Indicators (Right).kicad_sch (KiCad schematic)
At the start: 18 parts, among them J1-A1 Conn_01x05, J1-B1 Conn_01x05

Commit message: dash
Connections:
- net A10 renamed A2
- net A11 renamed A3
- net A12 renamed A4
- net A13 renamed A5
- net A14 renamed A6
- net A15 renamed A7
- net A8 renamed A0
- net A9 renamed A1
