File: hardware/KICAD Projects/BAJE SAE/Dash/Dash Indicators (Right)/Dash Indicators (Right).kicad_pcb (KiCad board)
At the start: 2 copper layers, 55.8 x 87 mm, 23 parts, among them J1-A1 Conn_01x05, J1-B1 Conn_01x05

Commit message: dash
Parts:
- moved G*** 0.28 mm to (93.7, 71.3)
Connections:
- net A10 renamed A2
- net A11 renamed A3
- net A12 renamed A4
- net A13 renamed A5
- net A14 renamed A6
- net A15 renamed A7
- net A8 renamed A0
- net A9 renamed A1
Other:
- board text added: "A0"
- board text added: "A4"
- board text added: "RIGHT"
- board text removed: "A12"
- board text removed: "A8"
- board text removed: "LEFT"

Commit message: temp sense worky now
Parts:
- moved J1-A1 1.12 mm to (98.0, 105.4)
Routing:
- net A1: track 60.8 -> 59.5 mm
- net A4: track 72.9 -> 71.8 mm
- net A2: track 81.9 -> 80.8 mm
Changed lines of the file:
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@@
 			(outputformat 1)
 			(mirror no)
-			(drillshape 1)
+			(drillshape 0)
 			(scaleselection 1)
-			(outputdirectory "")
+			(outputdirectory "Gerbers/")
 		)
 	)
@@
 	(footprint "Connector_PinHeader_2.54mm:PinHeader_1x05_P2.54mm_Vertical"
 		(layer "B.Cu")
-		(at 98.04 106.5 90)
+		(at 98.04 105.38 90)
 		(descr "Through hole straight pin header, 1x05, 2.54mm pitch, single row")
 		(tags "Through hole pin header THT 1x05 2.54mm single row")
@@
 	(dimension
 		(type aligned)
-		(layer "Edge.Cuts")
-		(pts
-			(xy 112.7 40.231088) (xy 114.5 42.031088)
-		)
-		(height -5.816149)
-		(gr_text "2.5456 mm"
-			(at 118.525811 36.205277 315)
-			(layer "Edge.Cuts")
-			(effects
-				(font
-					(size 1 1)
-					(thickness 0.15)
-				)
-			)
-		)
-		(format
-			(prefix "")
-			(suffix "")
-			(units 3)
-			(units_format 1)
-			(precision 4)
-		)
-		(style
-			(thickness 0.05)
-			(arrow_length 1.27)
-			(text_position_mode 0)
-			(extension_height 0.58642)
-			(extension_offset 0.5) keep_text_aligned)
-	)
-	(dimension
-		(type aligned)
-		(layer "Edge.Cuts")
-		(pts
-			(xy 112.7 96.828932) (xy 114.5 95.028932)
-		)
-		(height 12.052121)
-		(gr_text "2.5456 mm"
-			(at 121.308963 103.637895 45)
-			(layer "Edge.Cuts")
-			(effects
-				(font
-					(size 1 1)
-					(thickness 0.15)
-				)
-			)
-		)
-		(format
-			(prefix "")
-			(suffix "")
-			(units 3)
-			(units_format 1)
-			(precision 4)
-		)
-		(style
-			(thickness 0.05)
-			(arrow_length 1.27)
-			(text_position_mode 0)
-			(extension_height 0.58642)
-			(extension_offset 0.5) keep_text_aligned)
-	)
-	(dimension
-		(type aligned)
 		(layer "F.Fab")
 		(pts
@@
 	)
 	(segment
-		(start 105 99.54)
+		(start 103.35 42.35)
+		(end 100.065 42.35)
+		(width 0.2)
+		(layer "F.Cu")
+		(net 1)
+	)
+	(segment
+		(start 105 100.87)
 		(end 105 99.5)
 		(width 0.2)
@@
 	)
 	(segment
-		(start 98.04 106.5)
-		(end 105 99.54)
+		(start 105 99.5)
+		(end 107.1 97.4)
 		(width 0.2)
 		(layer "F.Cu")
@@
 	)
 	(segment
-		(start 103.35 42.35)
-		(end 100.065 42.35)
+		(start 100.49 105.38)
+		(end 105 100.87)
 		(width 0.2)
 		(layer "F.Cu")
@@
 	)
 	(segment
-		(start 105 99.5)
-		(end 107.1 97.4)
+		(start 98.04 105.38)
+		(end 100.49 105.38)
 		(width 0.2)
 		(layer "F.Cu")
@@
 	)
 	(segment
-		(start 95.8 104.9)
-		(end 99.034314 104.9)
-		(width 0.2)
-		(layer "F.Cu")
-		(net 4)
-	)
-	(segment
-		(start 95.5 105.2)
-		(end 95.8 104.9)
+		(start 105.65 72.35)
+		(end 100.065 72.35)
 		(width 0.2)
 		(layer "F.Cu")
@@
 	)
 	(segment
-		(start 105.65 72.35)
-		(end 100.065 72.35)
+		(start 106.617157 73.317157)
+		(end 105.65 72.35)
 		(width 0.2)
 		(layer "F.Cu")
@@
 	)
 	(segment
-		(start 106.617157 97.317157)
-		(end 106.617157 73.317157)
+		(start 99.764314 104.17)
+		(end 106.617157 97.317157)
 		(width 0.2)
 		(layer "F.Cu")
@@
 	)
 	(segment
-		(start 95.5 106.5)
-		(end 95.5 105.2)
+		(start 96.53 104.17)
+		(end 99.764314 104.17)
 		(width 0.2)
 		(layer "F.Cu")
@@
 	)
 	(segment
-		(start 106.617157 73.317157)
-		(end 105.65 72.35)
+		(start 106.617157 97.317157)
+		(end 106.617157 73.317157)
 		(width 0.2)
 		(layer "F.Cu")
@@
 	)
 	(segment
-		(start 99.034314 104.9)
-		(end 106.617157 97.317157)
+		(start 95.5 105.2)
+		(end 96.53 104.17)
 		(width 0.2)
 		(layer "F.Cu")
@@
 	)
 	(segment
-		(start 103.5 89.4)
-		(end 104.5 88.4)
+		(start 94.2 104.14)
+		(end 92.96 105.38)
 		(width 0.2)
 		(layer "B.Cu")
@@
 	)
 	(segment
-		(start 92.96 106.5)
-		(end 94.2 105.26)
+		(start 103.5 89.4)
+		(end 104.5 88.4)
 		(width 0.2)
 		(layer "B.Cu")
@@
 	)
 	(segment
-		(start 94.2 105.26)
-		(end 94.2 100.4)
+		(start 94.2 100.4)
+		(end 94.2 104.14)
 		(width 0.2)
 		(layer "B.Cu")
@@
 	)
 	(segment
-		(start 90.2 81.785)
-		(end 88.265 79.85)
-		(width 0.2)
-		(layer "F.Cu")
-		(net 6)
-	)
-	(segment
-		(start 90.42 106.5)
-		(end 90.7 106.5)
+		(start 91.85 103.95)
+		(end 90.42 105.38)
 		(width 0.2)
 		(layer "F.Cu")
@@
 	)
 	(segment
-		(start 93 104.7)
-		(end 94.2 103.5)
+		(start 90.2 81.785)
+		(end 88.265 79.85)
 		(width 0.2)
 		(layer "F.Cu")
@@
 	)
 	(segment
-		(start 92.5 104.7)
-		(end 93 104.7)
+		(start 93.75 103.95)
+		(end 91.85 103.95)
 		(width 0.2)
 		(layer "F.Cu")
@@
 	)
 	(segment
-		(start 90.7 106.5)
-		(end 92.5 104.7)
+		(start 94.2 103.5)
+		(end 93.75 103.95)
 		(width 0.2)
 		(layer "F.Cu")
@@
 	)
 	(segment
-		(start 82.4 61.1)
-		(end 87.2 61.1)
+		(start 88.265 57.35)
+		(end 88.265 60.035)
 		(width 0.2)
 		(layer "B.Cu")
@@
 	)
 	(segment
-		(start 100.065 57.35)
-		(end 100.065 55.365)
+		(start 82.11 61.39)
+		(end 82.11 99.61)
 		(width 0.2)
 		(layer "B.Cu")
@@
 	)
 	(segment
-		(start 82.1 100.72)
-		(end 82.1 61.4)
+		(start 100.065 57.35)
+		(end 100.065 55.365)
 		(width 0.2)
 		(layer "B.Cu")
@@
 	)
 	(segment
-		(start 87.88 106.5)
-		(end 82.1 100.72)
+		(start 82.4 61.1)
+		(end 82.11 61.39)
 		(width 0.2)
 		(layer "B.Cu")
@@
 	(segment
 		(start 88.265 60.035)
-		(end 88.265 57.35)
+		(end 87.2 61.1)
 		(width 0.2)
 		(layer "B.Cu")
@@
 	)
 	(segment
-		(start 87.2 61.1)
-		(end 88.265 60.035)
+		(start 98.4 53.7)
+		(end 91.9 53.7)
 		(width 0.2)
 		(layer "B.Cu")
@@
 	)
 	(segment
-		(start 98.4 53.7)
-		(end 91.9 53.7)
+		(start 100.065 55.365)
+		(end 98.4 53.7)
 		(width 0.2)
 		(layer "B.Cu")
@@
 	)
 	(segment
-		(start 100.065 55.365)
-		(end 98.4 53.7)
+		(start 82.11 99.61)
+		(end 87.88 105.38)
 		(width 0.2)
 		(layer "B.Cu")
@@
 	)
 	(segment
-		(start 82.1 61.4)
+		(start 87.2 61.1)
 		(end 82.4 61.1)
 		(width 0.2)
