File: hardware/KICAD Projects/BAJE SAE/Dash/Dash Main/Dash Main.kicad_pcb (KiCad board)
At the start: 2 copper layers, 137.9 x 76.2 mm, 26 parts, among them J1 CAN to outer connector, J1-A1 Conn_01x05, J1-B1 Conn_01x05, J10 Button 2, J11 14 Segment (2), J2 Servo 1 (RPM), J2-A1 Conn_01x05, J2-B1 Conn_01x05, J3 Button 1, J4 14 Segment (1), J5 14 Segment (3), J7 Conn_01x02, J8 Servo 2 (Speed), J9 14 Segment (4)

Commit message: dash traces done
Parts:
- UNIT_1: footprint BAJA SAE:HiLetgo CAN Bus (Facing Up) -> 0_Baja_Final:Can Bus (Correct)
- moved UNIT_1 20.6 mm to (176.6, 87.1), turned to -90 degrees
- moved REF** 1.50 mm to (128.8, 69.6)
Connections:
- J1 pad 1: Low -> High
- J1 pad 2: High -> Low
- J1 pad 3: Low -> High
- J1 pad 4: High -> Low
- U2 pad 2: (no net) -> GND
- U2 pad 5: (no net) -> 3v3 ground
Routing:
- net GND: track 0.00 -> 348.1 mm
- net Regulated 3v3: track 0.00 -> 294.6 mm, vias 0 -> 1
- net +5v: track 0.00 -> 207.0 mm, vias 0 -> 1
- net C1: track 0.00 -> 192.7 mm, vias 0 -> 1
- net C0: track 0.00 -> 173.4 mm
- net SI: track 0.00 -> 144.7 mm
- net SCL: track 0.00 -> 128.5 mm
- net 3v3 ground: track 0.00 -> 114.5 mm, vias 0 -> 2
- net A11: track 0.00 -> 110.9 mm, vias 0 -> 2
- net CS: track 0.00 -> 109.9 mm
- net SDA: track 0.00 -> 108.4 mm
- net A12: track 0.00 -> 107.1 mm
- net SCK: track 0.00 -> 104.9 mm
- net A15: track 0.00 -> 104.8 mm
- net IO33 RPM: track 0.00 -> 103.6 mm, vias 0 -> 1
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
Commit message: made project template
Parts:
- moved UNIT_1 2.06 mm to (178.4, 88.2)
Routing:
- net +5v: track 207.0 -> 239.0 mm, vias 1 -> 2
- net GND: track 348.1 -> 373.4 mm
- net High: track 66.5 -> 79.1 mm
- net SCK: track 104.9 -> 114.5 mm, vias 0 -> 1
- net SI: track 144.7 -> 154.1 mm
- net CS: track 109.9 -> 100.9 mm
- net Low: track 73.3 -> 69.9 mm
- net SO: track 100.9 -> 102.3 mm
Other:
- board text added: "+5V"
- board text added: "A0"
- board text added: "A13"
- board text added: "A4"
- board text added: "Button 1"
- board text added: "Button 2"
- board text added: "C1"
- board text added: "GND"
- board text added: "H"
- board text added: "J1"
- board text added: "J10"
- board text added: "J11"
- board text added: "J3"
- board text added: "J4"
- board text added: "J5"
- board text added: "J6"
- board text added: "J7"
- board text added: "J8"
- board text added: "J9"
- board text added: "L"
- board text added: "Left LED"
- board text added: "RPM Servo"
- board text added: "Right LED"
- board text added: "Solder Here!"
- board text added: "Speed Servo"

Commit message: dash
Parts:
- added G***: LOGO, BAJA SAE:Untitled, B.Cu at (135.4, 48.5)
Other:
- board text added: "Designed by Connor Larson, Karsten Yian and Julian m56 In Tucson, Arizona, on Febuary 23rd, 2025."

Commit message: temp sense worky now
Changed lines of the file:
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@@
 			(outputformat 1)
 			(mirror no)
-			(drillshape 1)
+			(drillshape 0)
 			(scaleselection 1)
-			(outputdirectory "")
+			(outputdirectory "Gerbers/")
 		)
 	)
@@
 	)
 	(gr_text "Designed by Connor Larson, Karsten Yian and Julian m56 \nIn Tucson, Arizona, on Febuary 23rd, 2025."
-		(at 70.43 81.245 90)
+		(at 67.98 87.09 90)
 		(layer "F.SilkS")
 		(effects

Commit message: Created Dash Gerbers
Parts:
- removed the J7 at (92.7, 94.5)
- added J12: Conn_01x02, Connector_Wire:SolderWire-0.75sqmm_1x02_P4.8mm_D1.25mm_OD2.3mm, F.Cu at (93.0, 94.3)
- U2: moved to B.Cu
- moved UNIT_1 34.0 mm to (181.2, 54.3)
- moved U1 33.3 mm to (148.9, 61.9), turned to 0 degrees
- moved U2 2.47 mm to (106.6, 61.0), turned to 180 degrees
- renumbered J2-A1 to J1-1, J2-B1 to J1-2, J2 to J10, J1-A1 to J11-1, J1-B1 to J11-2, J8 to J2, J3 to J4, J4 to J5, J11 to J6, J5 to J7, J9 to J8, J10 to J9
Connections:
- J5 pad 4: GND -> 3v3 ground
- J6 pad 4: GND -> 3v3 ground
- J7 pad 4: GND -> 3v3 ground
- J8 pad 4: GND -> 3v3 ground
- U1 pad 26: unconnected-(U1-SCL-Pad26) -> SCL
- U1 pad 27: unconnected-(U1-SDA-Pad27) -> SDA
Routing:
- net GND: track 373.4 -> 240.0 mm, vias 0 -> 1
- net SI: track 154.1 -> 25.5 mm, vias 0 -> 1
- net Regulated 3v3: track 294.6 -> 194.5 mm, vias 1 -> 0
- net SCK: track 114.5 -> 40.5 mm
- net CS: track 100.9 -> 38.6 mm
- net SO: track 102.3 -> 44.9 mm, vias 0 -> 2
- net SDA: track 108.4 -> 155.7 mm
- net Low: track 69.9 -> 114.6 mm
- net +5v: track 239.0 -> 198.6 mm
- net 3v3 ground: track 114.5 -> 154.6 mm, vias 2 -> 0
- net C1: track 192.7 -> 156.2 mm, vias 1 -> 0
- net A12: track 107.1 -> 74.7 mm
- net A11: track 110.9 -> 80.6 mm, vias 2 -> 0
- net SCL: track 128.5 -> 157.7 mm
- net High: track 79.1 -> 106.7 mm
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Other:
- board text added: "3V3 Converter"
- board text added: "CAN"
- board text added: "ESP 32"
- board text added: "J2"
- board text added: "LED Breakout"
- board text added: "REV. 2"
- board text added: "This side up Matthew"
- board text added: "Where is J3? dw about it"
- board text removed: "J3"
