File: hardware/KICAD Projects/BAJE SAE/Dash/Dash Main/Dash Main.kicad_sch (KiCad schematic)
At the start: 19 parts, among them J1 CAN to outer connector, J1-A1 Conn_01x05, J1-B1 Conn_01x05, J10 Button 2, J11 14 Segment (2), J2 Servo 1 (RPM), J2-A1 Conn_01x05, J2-B1 Conn_01x05, J3 Button 1, J4 14 Segment (1), J5 14 Segment (3), J6 Conn_01x06, J7 Conn_01x02, J8 Servo 2 (Speed), J9 14 Segment (4)

Commit message: dash traces done
Parts:
- UNIT_1: footprint BAJA SAE:HiLetgo CAN Bus (Facing Up) -> 0_Baja_Final:Can Bus (Correct)
Connections:
- net 3v3 ground: now also U2.5 (-Vout); no longer U2. (-Vout)
- net GND: now also U2.2 (GND); no longer U2.1 (Vin)
Changed lines of the file:
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@@
 		(pin "3"
 		)
-		(pin ""
+		(pin "5"
 		)
 		(pin "6"
@@
 		(pin "1"
 		)
-		(pin "1"
+		(pin "2"
 		)
 		(instances
@@
 			)
 		)
-		(property "Footprint" "BAJA SAE:HiLetgo CAN Bus (Facing Up)"
+		(property "Footprint" "0_Baja_Final:Can Bus (Correct)"
 			(at 51.054 145.796 0)
 			(effects

Commit message: made project template
Parts:
- renumbered J2-A1 to J1-1, J2-B1 to J1-2, J2 to J10, J1-A1 to J11-1, J1-B1 to J11-2, J8 to J2, J3 to J5, J4 to J5, J11 to J6, J5 to J7, J9 to J8, J10 to J9
Changed lines of the file:
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@@
 		(on_board yes)
 		(dnp no)
-		(property "Reference" "J9"
+		(property "Reference" "J8"
 			(at 160.02 132.0799 0)
 			(effects
@@
 			(project "Dash Main"
 				(path "/ce068e4e-d009-4dc1-a111-640e06c307fc"
-					(reference "J9")
+					(reference "J8")
 					(unit 1)
 				)
@@
 		(dnp no)
 		(fields_autoplaced yes)
-		(property "Reference" "J11"
+		(property "Reference" "J6"
 			(at 161.29 110.4899 0)
 			(effects
@@
 			(project "Dash Main"
 				(path "/ce068e4e-d009-4dc1-a111-640e06c307fc"
-					(reference "J11")
+					(reference "J6")
 					(unit 1)
 				)
@@
 		(dnp no)
 		(fields_autoplaced yes)
-		(property "Reference" "J8"
+		(property "Reference" "J2"
 			(at 247.65 111.7599 0)
 			(effects
@@
 			(project "Dash Main"
 				(path "/ce068e4e-d009-4dc1-a111-640e06c307fc"
-					(reference "J8")
+					(reference "J2")
 					(unit 1)
 				)
@@
 		(dnp no)
 		(fields_autoplaced yes)
-		(property "Reference" "J1-B1"
-			(at 147.32 175.2599 0)
+		(property "Reference" "J11-2"
+			(at 147.32 176.5299 0)
 			(effects
 				(font
@@
 			(project "Dash Main"
 				(path "/ce068e4e-d009-4dc1-a111-640e06c307fc"
-					(reference "J1-B1")
+					(reference "J11-2")
 					(unit 1)
 				)
@@
 		(dnp no)
 		(fields_autoplaced yes)
-		(property "Reference" "J2-B1"
+		(property "Reference" "J1-2"
 			(at 168.91 176.5299 0)
 			(effects
@@
 			(project "Dash Main"
 				(path "/ce068e4e-d009-4dc1-a111-640e06c307fc"
-					(reference "J2-B1")
+					(reference "J1-2")
 					(unit 1)
 				)
@@
 		(dnp no)
 		(fields_autoplaced yes)
-		(property "Reference" "J5"
+		(property "Reference" "J7"
 			(at 119.38 132.0799 0)
 			(effects
@@
 			(project "Dash Main"
 				(path "/ce068e4e-d009-4dc1-a111-640e06c307fc"
-					(reference "J5")
+					(reference "J7")
 					(unit 1)
 				)
@@
 		(dnp no)
 		(fields_autoplaced yes)
-		(property "Reference" "J2"
+		(property "Reference" "J10"
 			(at 208.28 111.7599 0)
 			(effects
@@
 			(project "Dash Main"
 				(path "/ce068e4e-d009-4dc1-a111-640e06c307fc"
-					(reference "J2")
+					(reference "J10")
 					(unit 1)
 				)
@@
 		(dnp no)
 		(fields_autoplaced yes)
-		(property "Reference" "J1-A1"
-			(at 147.32 162.5599 0)
+		(property "Reference" "J11-1"
+			(at 147.32 163.8299 0)
 			(effects
 				(font
@@
 			(project "Dash Main"
 				(path "/ce068e4e-d009-4dc1-a111-640e06c307fc"
-					(reference "J1-A1")
+					(reference "J11-1")
 					(unit 1)
 				)
@@
 		(dnp no)
 		(fields_autoplaced yes)
-		(property "Reference" "J2-A1"
+		(property "Reference" "J1-1"
 			(at 168.91 163.8299 0)
 			(effects
@@
 			(project "Dash Main"
 				(path "/ce068e4e-d009-4dc1-a111-640e06c307fc"
-					(reference "J2-A1")
+					(reference "J1-1")
 					(unit 1)
 				)
@@
 		(dnp no)
 		(fields_autoplaced yes)
-		(property "Reference" "J10"
+		(property "Reference" "J9"
 			(at 254 137.1599 0)
 			(effects
@@
 			(project "Dash Main"
 				(path "/ce068e4e-d009-4dc1-a111-640e06c307fc"
-					(reference "J10")
+					(reference "J9")
 					(unit 1)
 				)
@@
 		(dnp no)
 		(fields_autoplaced yes)
-		(property "Reference" "J3"
+		(property "Reference" "J5"
 			(at 212.09 135.8899 0)
 			(effects
@@
 			(project "Dash Main"
 				(path "/ce068e4e-d009-4dc1-a111-640e06c307fc"
-					(reference "J3")
+					(reference "J5")
 					(unit 1)
 				)
@@
 		(dnp no)
 		(fields_autoplaced yes)
-		(property "Reference" "J4"
+		(property "Reference" "J5"
 			(at 119.38 110.4899 0)
 			(effects
@@
 			(project "Dash Main"
 				(path "/ce068e4e-d009-4dc1-a111-640e06c307fc"
-					(reference "J4")
-					(unit 1)
-				)
+					(reference "J5")
+					(unit 1)
+				)

Commit message: Created Dash Gerbers
Parts:
- renumbered J7 to J12, J5 to J4, J6 to J999
Connections:
- net 3v3 ground: now also J5.4 (Pin_4), J6.4 (Pin_4), J7.4 (Pin_4), J8.4 (Pin_4)
- net GND: no longer J5.4 (Pin_4), J6.4 (Pin_4), J7.4 (Pin_4), J8.4 (Pin_4)
- net SCL: now also U1.26 (SCL)
- net SDA: now also U1.27 (SDA)
Changed lines of the file:
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@@
 		)
 	)
-	(global_label "GND"
+	(global_label "A10"
 		(shape input)
-		(at 153.67 115.57 180)
+		(at 241.3 82.55 0)
 		(fields_autoplaced yes)
 		(effects
@@
 				(size 1.27 1.27)
 			)
-			(justify right)
+			(justify left)
 		)
 		(property "Intersheetrefs" "${INTERSHEET_REFS}"
-			(at 146.8143 115.57 0)
+			(at 247.7928 82.55 0)
 			(effects
 				(font
 					(size 1.27 1.27)
 				)
-				(justify right)
+				(justify left)
 				(hide yes)
 			)
 		)
 	)
-	(global_label "A10"
+	(global_label "Regulated 3v3"
 		(shape input)
-		(at 241.3 82.55 0)
+		(at 111.76 113.03 180)
 		(fields_autoplaced yes)
 		(effects
@@
 				(size 1.27 1.27)
 			)
-			(justify left)
+			(justify right)
 		)
 		(property "Intersheetrefs" "${INTERSHEET_REFS}"
-			(at 247.7928 82.55 0)
+			(at 94.9865 113.03 0)
 			(effects
 				(font
 					(size 1.27 1.27)
 				)
-				(justify left)
+				(justify right)
 				(hide yes)
 			)
 		)
 	)
-	(global_label "Regulated 3v3"
+	(global_label "A8"
 		(shape input)
-		(at 111.76 113.03 180)
+		(at 161.29 158.75 180)
 		(fields_autoplaced yes)
 		(effects
@@
 		)
 		(property "Intersheetrefs" "${INTERSHEET_REFS}"
-			(at 94.9865 113.03 0)
+			(at 156.0067 158.75 0)
 			(effects
 				(font
@@
 		)
 	)
-	(global_label "A8"
+	(global_label "SDA"
 		(shape input)
-		(at 161.29 158.75 180)
+		(at 111.76 110.49 180)
 		(fields_autoplaced yes)
 		(effects
@@
 		)
 		(property "Intersheetrefs" "${INTERSHEET_REFS}"
-			(at 156.0067 158.75 0)
+			(at 105.2067 110.49 0)
 			(effects
 				(font
@@
 		)
 	)
-	(global_label "SDA"
+	(global_label "3v3 ground"
 		(shape input)
-		(at 111.76 110.49 180)
+		(at 111.76 137.16 180)
 		(fields_autoplaced yes)
 		(effects
@@
 		)
 		(property "Intersheetrefs" "${INTERSHEET_REFS}"
-			(at 105.2067 110.49 0)
+			(at 97.8894 137.16 0)
 			(effects
 				(font
@@
 		)
 	)
+	(global_label "SDA"
+		(shape input)
+		(at 241.3 36.83 0)
+		(fields_autoplaced yes)
+		(effects
+			(font
+				(size 1.27 1.27)
+			)
+			(justify left)
+		)
+		(property "Intersheetrefs" "${INTERSHEET_REFS}"
+			(at 247.8533 36.83 0)
+			(effects
+				(font
+					(size 1.27 1.27)
+				)
+				(justify left)
+				(hide yes)
+			)
+		)
+	)
 	(global_label "SCL"
 		(shape input)
@@
 		)
 	)
+	(global_label "3v3 ground"
+		(shape input)
+		(at 152.4 137.16 180)
+		(fields_autoplaced yes)
+		(effects
+			(font
+				(size 1.27 1.27)
+			)
+			(justify right)
+		)
+		(property "Intersheetrefs" "${INTERSHEET_REFS}"
+			(at 138.5294 137.16 0)
+			(effects
+				(font
+					(size 1.27 1.27)
+				)
+				(justify right)
+				(hide yes)
+			)
+		)
+	)
 	(global_label "C1"
 		(shape input)
@@
 		)
 	)
-	(global_label "GND"
+	(global_label "C5"
 		(shape input)
-		(at 152.4 137.16 180)
+		(at 210.82 55.88 180)
 		(fields_autoplaced yes)
 		(effects
@@
 		)
 		(property "Intersheetrefs" "${INTERSHEET_REFS}"
-			(at 145.5443 137.16 0)
+			(at 205.3553 55.88 0)
 			(effects
 				(font
@@
 		)
 	)
-	(global_label "C5"
+	(global_label "3v3 ground"
 		(shape input)
-		(at 210.82 55.88 180)
+		(at 111.76 115.57 180)
 		(fields_autoplaced yes)
 		(effects
@@
 		)
 		(property "Intersheetrefs" "${INTERSHEET_REFS}"
-			(at 205.3553 55.88 0)
+			(at 97.8894 115.57 0)
 			(effects
 				(font
@@
 		)
 	)
-	(global_label "GND"
-		(shape input)
-		(at 111.76 115.57 180)
-		(fields_autoplaced yes)
-		(effects
-			(font
-				(size 1.27 1.27)
-			)
-			(justify right)
-		)
-		(property "Intersheetrefs" "${INTERSHEET_REFS}"
-			(at 104.9043 115.57 0)
-			(effects
-				(font
-					(size 1.27 1.27)
-				)
-				(justify right)
-				(hide yes)
-			)
-		)
-	)
 	(global_label "SCL"
 		(shape input)
@@
 		)
 	)
-	(global_label "GND"
-		(shape input)
-		(at 111.76 137.16 180)
-		(fields_autoplaced yes)
-		(effects
-			(font
-				(size 1.27 1.27)
-			)
-			(justify right)
-		)
-		(property "Intersheetrefs" "${INTERSHEET_REFS}"
-			(at 104.9043 137.16 0)
-			(effects
-				(font
-					(size 1.27 1.27)
-				)
-				(justify right)
-				(hide yes)
-			)
-		)
-	)
 	(global_label "A1"
 		(shape input)
@@
 		)
 	)
+	(global_label "3v3 ground"
+		(shape input)
+		(at 153.67 115.57 180)
+		(fields_autoplaced yes)
+		(effects
+			(font
+				(size 1.27 1.27)
+			)
+			(justify right)
+		)
+		(property "Intersheetrefs" "${INTERSHEET_REFS}"
+			(at 139.7994 115.57 0)
+			(effects
+				(font
+					(size 1.27 1.27)
+				)
+				(justify right)
+				(hide yes)
+			)
+		)
+	)
 	(global_label "Regulated 3v3"
 		(shape input)
@@
 		)
 	)
+	(global_label "SCL"
+		(shape input)
+		(at 241.3 40.64 0)
+		(fields_autoplaced yes)
+		(effects
+			(font
+				(size 1.27 1.27)
+			)
+			(justify left)
+		)
+		(property "Intersheetrefs" "${INTERSHEET_REFS}"
+			(at 247.7928 40.64 0)
+			(effects
+				(font
+					(size 1.27 1.27)
+				)
+				(justify left)
+				(hide yes)
+			)
+		)
+	)
 	(global_label "A2"
 		(shape input)
@@
 		(dnp no)
 		(fields_autoplaced yes)
-		(property "Reference" "J7"
-			(at 151.13 60.9599 0)
+		(property "Reference" "J12"
+			(at 151.13 62.2299 0)
 			(effects
 				(font
@@
 			(project "Dash Main"
 				(path "/ce068e4e-d009-4dc1-a111-640e06c307fc"
-					(reference "J7")
+					(reference "J12")
 					(unit 1)
 				)
@@
 		(dnp no)
 		(fields_autoplaced yes)
-		(property "Reference" "J6"
+		(property "Reference" "J999"
 			(at 142.24 34.2899 0)
 			(effects
@@
 			(project "Dash Main"
 				(path "/ce068e4e-d009-4dc1-a111-640e06c307fc"
-					(reference "J6")
+					(reference "J999")
 					(unit 1)
 				)
@@
 		(dnp no)
 		(fields_autoplaced yes)
-		(property "Reference" "J5"
+		(property "Reference" "J4"
 			(at 212.09 135.8899 0)
 			(effects
@@
 			(project "Dash Main"
 				(path "/ce068e4e-d009-4dc1-a111-640e06c307fc"
-					(reference "J5")
+					(reference "J4")
 					(unit 1)
 				)
