File: hardware/KICAD Projects/BAJE SAE/12 to 5 with Trimmer/12 to 5 with Trimmer.kicad_sch (KiCad schematic)
At the start: 6 parts

Commit message: Update 12 to 5 with Trimmer.kicad_sch
Parts:
- RV1: value ? -> 3.95k
Other:
- note added: "2.5 x 2.32 X(2.43 + 0) RV1= (5.5-5) X 2.32 - 8.2"
- note added: "= 3.95k"
Changed lines of the file:
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@@
+		)
+	)
+	(text "= 3.95k"
+		(exclude_from_sim no)
+		(at 228.6 102.616 0)
+		(effects
+			(font
+				(size 1.27 1.27)
+			)
+		)
+	)
+	(text "    2.5 x 2.32 X(2.43 + 0)\nRV1=              (5.5-5) X 2.32      - 8.2"
+		(exclude_from_sim no)
+		(at 228.092 97.028 0)
+		(effects
+			(font
+				(size 1.27 1.27)
+			)
 		)
 	)
@@
 			)
 		)
-		(property "Value" "?"
+		(property "Value" "3.95k"
 			(at 165.1 110.4899 0)
 			(effects

Commit message: trimmer
Parts:
- removed H1: 12V In, symbol Mechanical:MountingHole_Pad
- removed H2: GND, symbol Mechanical:MountingHole_Pad
- removed H3: 5V GND, symbol Mechanical:MountingHole_Pad
- removed H4: 5V Out, symbol Mechanical:MountingHole_Pad
- added J1: Conn_01x04, TerminalBlock_Phoenix:TerminalBlock_Phoenix_MKDS-3-4-5.08_1x04_P5.08mm_Horizontal, symbol Connector_Generic:Conn_01x04
- RV1: value 3.95k -> 3.3k; footprint (none) -> Potentiometer_THT:Potentiometer_Bourns_3296W_Vertical
- U1: footprint (none) -> 0_Baja_2025:SKM10E-03
Connections:
- net at RV1.1: now also U1.4 (Trim); no longer U1. (-Vout)
- net VOUT: now reaches U1.3 (Vout)
- net VOUT: now also J1.4 (Pin_4)
- net VIN: now reaches U1.1 (Vin)
- net VIN: now also J1.1 (Pin_1)
- net GND renamed VOUT-
- net VOUT-: now also U1.5 (-Vout), J1.3 (Pin_3); no longer U1.1 (Vin)
- net trim: no longer names the net of RV1.3
- net trim: no longer U1.4 (Trim)
- new net V-: J1.2 (Pin_2), U1.2 (GND)
- no-connect marks 0 -> 2
Other:
- moved on the sheet: RV1
